Commit message: multi-uavs spawning but not moving

File: urdf/multi_uavs.urdf.xacro (robot description, xacro)
@@ -2,22 +2,4 @@
 <robot xmlns:xacro="http://www.ros.org/wiki/xacro" name="multi_crazy2fly">
     <xacro:include filename="$(find acts_simulator)/urdf/crazy2fly.urdf.xacro" />
-    <link name="world" />
-    <xacro:crazy2fly prefix="drone1_" />
-    <joint name="world_to_drone1" type="fixed">
-        <parent link="world" />
-        <child link="drone1_base_link" />
-        <origin xyz="1.0 1.0 1.0" rpy="0 0 0"/>
-    </joint>
-    <xacro:crazy2fly prefix="drone2_" />
-    <joint name="world_to_drone2" type="fixed">
-        <parent link="world" />
-        <child link="drone2_base_link" />
-        <origin xyz="2.0 2.0 2.0" rpy="0 0 0"/>
-    </joint>
-    <xacro:crazy2fly prefix="drone3_" />
-    <joint name="world_to_drone3" type="fixed">
-        <parent link="world" />
-        <child link="drone3_base_link" />
-        <origin xyz="3.0 3.0 3.0" rpy="0 0 0"/>
-    </joint>
+    <xacro:crazy2fly prefix="" />
 </robot>
