Commit message: multi uav control with cable working

File: urdf/uav_cable_assembly.urdf.xacro (robot description, xacro)
@@ -3,19 +3,33 @@
   <xacro:include filename="$(find acts_simulator)/urdf/crazy2fly.urdf.xacro" />
   <xacro:include filename="$(find acts_simulator)/urdf/components/cable_component.xacro" />
-  <xacro:macro name="add_drone" params="id segments length panel_link x_off y_off z_off">
+  <xacro:macro name="add_drone" params="id segments length x_off y_off z_off panel_link:=''">
     <xacro:property name="prefix" value="drone${id}_" />
     <xacro:crazy2fly prefix="${prefix}" />
+    <!-- When no panel_link, create a free-floating root link for the cable top -->
+    <xacro:if value="${panel_link == ''}">
+        <link name="${prefix}cable_root_link">
+            <inertial>
+                <mass value="0.0001"/>
+                <inertia ixx="1e-6" ixy="0" ixz="0" iyy="1e-6" iyz="0" izz="1e-6"/>
+            </inertial>
+        </link>
+        <xacro:property name="cable_parent" value="${prefix}cable_root_link" />
+    </xacro:if>
+    <xacro:unless value="${panel_link == ''}">
+        <xacro:property name="cable_parent" value="${panel_link}" />
+    </xacro:unless>
     <xacro:uav_cable
-      prefix="${prefix}"
-      parent_link="${panel_link}"
-      is_flexible="true"
-      segments="${segments}"
-      length="${length}"
-      radius="0.005" mass="0.01" />
+        prefix="${prefix}"
+        parent_link="${cable_parent}"
+        is_flexible="true"
+        segments="${segments}"
+        length="${length}"
+        radius="0.005" mass="0.01" />
+    <!-- Cable tip attaches to drone base -->
     <joint name="${prefix}cable_to_drone_joint" type="fixed">
-      <parent link="${prefix}link_${segments}"/>
-      <child link="${prefix}base_link"/>
-      <origin xyz="${x_off} ${y_off} ${float(z_off)}" rpy="0 0 0"/>
+        <parent link="${prefix}link_${segments}"/>
+        <child link="${prefix}base_link"/>
+        <origin xyz="${x_off} ${y_off} ${float(z_off)}" rpy="0 0 0"/>
     </joint>
-  </xacro:macro>
+</xacro:macro>
 </robot>

File: urdf/uav_usable.urdf.xacro (robot description, xacro)
@@ -1,4 +1,4 @@
 <?xml version="1.0"?>
-<robot xmlns:xacro="http://www.ros.org/wiki/xacro" name="multi_crazy2fly">
+<robot xmlns:xacro="http://www.ros.org/wiki/xacro" name="crazy2fly_usable">
     <xacro:include filename="$(find acts_simulator)/urdf/crazy2fly.urdf.xacro" />
     <xacro:arg name="prefix" default="drone1_"/>
@@ -6,5 +6,4 @@
     <xacro:arg name="y" default="0.0"/>
     <xacro:arg name="z" default="0.0"/>
-    <xacro:arg name="prefix" default="drone1"/>
     <xacro:crazy2fly prefix="$(arg prefix)" />
 </robot>
