Commit message: added uav model and rigid cable working

File: urdf/acts.urdf.xacro (robot description, xacro)
@@ -3,4 +3,5 @@
   <xacro:include filename="panel.urdf.xacro" />
   <xacro:include filename="uav_cable_assembly.xacro" />
+  <xacro:include filename="components/cable_component.xacro" />
   <!-- <xacro:include filename="physics_macros.xacro" /> -->
   <xacro:panel_platform prefix="main_panel_" />

File: urdf/cable.urdf.xacro (robot description, xacro)
@@ -7,5 +7,5 @@
   </inertial>
 </xacro:macro>
-<xacro:macro name="cable_segment" params="name m r h color">
+<xacro:macro name="cable_segment" parent_xyz:='0 0 0' params="name m r h color">
   <link name="${name}">
     <xacro:cylinder_inertia m="${m}" r="${r}" h="${h}" />

File: urdf/panel.urdf.xacro (robot description, xacro)
@@ -1,4 +1,10 @@
 <?xml version="1.0"?>
 <robot xmlns:xacro="http://www.ros.org/wiki/xacro">
+<!-- PARAMETERS -->
+  <xacro:property name="p_mass" value="1.0" />
+  <xacro:property name="p_width" value="1" />
+  <xacro:property name="p_depth" value="1" />
+  <xacro:property name="p_height" value="0.1" />
+    <!-- inertia -->
   <xacro:macro name="panel_box_inertia" params="m w d h">
     <inertial>
@@ -11,11 +17,15 @@
   <xacro:macro name="panel_platform" params="prefix">
     <link name="${prefix}base_link">
-      <xacro:panel_box_inertia m="1.0" w="0.4" d="0.4" h="0.1" />
+      <xacro:panel_box_inertia m="${p_mass}" w="${p_width}" d="${p_depth}" h="${p_height}" />
       <visual>
-        <geometry><box size="0.4 0.4 0.1"/></geometry>
+        <geometry>
+          <box size="${p_width} ${p_depth} ${p_height}"/>
+        </geometry>
         <material name="grey"><color rgba="0.5 0.5 0.5 1"/></material>
       </visual>
       <collision>
-        <geometry><box size="0.4 0.4 0.1"/></geometry>
+        <geometry>
+          <box size="${p_width} ${p_depth} ${p_height}"/>
+        </geometry>
       </collision>
     </link>

File: urdf/uav_cable_assembly.xacro (robot description, xacro)
@@ -2,5 +2,5 @@
 <robot xmlns:xacro="http://www.ros.org/wiki/xacro">
   <xacro:include filename="uav_component.xacro" />
-  <xacro:include filename="cable_component.xacro" />
+  <xacro:include filename="components/cable_component.xacro" />
   <xacro:macro name="uav_plus_cable" params="prefix parent_link x y z">
     <xacro:uav_platform prefix="${prefix}" />
@@ -10,5 +10,12 @@
       <origin xyz="${x} ${y} ${z}" rpy="0 0 0"/>
     </joint>
-    <xacro:cable_tether prefix="${prefix}cable_" parent_link="${prefix}base_link" />
+    <xacro:uav_cable
+      prefix="${prefix}cable_"
+      parent_link="${prefix}base_link"
+      is_flexible="True"
+      segments="10"
+      length="1.0"
+      radius="0.01"
+      mass="0.1" />
   </xacro:macro>
 </robot>

Commit message: real uav model imported correctly and uav-cable assembly created

File: urdf/acts.urdf.xacro (robot description, xacro)
@@ -4,13 +4,26 @@
   <xacro:include filename="uav_cable_assembly.xacro" />
   <xacro:include filename="components/cable_component.xacro" />
-  <!-- <xacro:include filename="physics_macros.xacro" /> -->
-  <xacro:panel_platform prefix="main_panel_" />
-  <xacro:uav_plus_cable
-    prefix="uav_left_"
-    parent_link="main_panel_base_link"
-    x="1.0" y="0.0" z="0.5" />
-  <xacro:uav_plus_cable
-    prefix="uav_right_"
-    parent_link="main_panel_base_link"
-    x="-1.0" y="0.0" z="0.5" />
+  <xacro:panel_platform
+  prefix="main_panel_"
+  mass="2.5"
+  width="2.0"
+  depth="2.0"
+  height="0.2" />
+  <link name="panel_corner_link" />
+  <joint name="panel_to_corner" type="fixed">
+    <parent link="main_panel_base_link"/>
+    <child link="panel_corner_link"/>
+    <origin xyz="0.8 0.8 0.1" rpy="0 3.14159 0"/>  <!-- the cable is directed upwards-->
+    <gazebo reference="panel_to_corner">
+    <disableFixedJointLumping>true</disableFixedJointLumping>
+  </gazebo>
+  </joint>
+  <xacro:uav_cable
+    prefix="upward_cable_"
+    parent_link="panel_corner_link"
+    is_flexible="${True}"
+    segments="10"
+    length="1.5"
+    radius="0.01"
+    mass="0.2" />
 </robot>

File: urdf/components/cable_component.xacro (robot description, xacro)
@@ -21,5 +21,5 @@
       </collision>
     </link>
-    <joint name="${prefix}rigid_joint" type="fixed">
+    <joint name="${prefix}rigid_joint" type="universal">
       <parent link="${parent_link}"/>
       <child link="${prefix}rigid_link"/>
@@ -28,45 +28,55 @@
   </xacro:macro>
   <xacro:macro name="flexible_chain_generator" params="prefix parent current_num total_num len rad m">
-    <link name="${prefix}link_${current_num}">
-      <xacro:cylinder_inertia m="${m}" r="${rad}" h="${len}" />
-      <visual>
-        <origin xyz="0 0 ${-len/2.0}"/>
-        <geometry><cylinder radius="${rad}" length="${len}"/></geometry>
-      </visual>
-      <collision>
-        <origin xyz="0 0 ${-len/2.0}"/>
-        <geometry><cylinder radius="${rad}" length="${len}"/></geometry>
-      </collision>
-    </link>
-    <joint name="${prefix}joint_${current_num}" type="continuous">
-      <parent link="${parent}"/>
-      <child link="${prefix}link_${current_num}"/>
-      <xacro:if value="${current_num == 1}">
-        <origin xyz="0 0 -0.05" rpy="0 0 0"/>
-      </xacro:if>
-      <xacro:unless value="${current_num == 1}">
-        <origin xyz="0 0 ${-len}" rpy="0 0 0"/>
-      </xacro:unless>
-      <axis xyz="1 1 0"/>
-      <dynamics damping="0.1" friction="0.02"/>
-    </joint>
-    <xacro:if value="${current_num &lt; total_num}">
-      <xacro:flexible_chain_generator
-        prefix="${prefix}"
-        parent="${prefix}link_${current_num}"
-        current_num="${current_num + 1}"
-        total_num="${total_num}"
-        len="${len}"
-        rad="${rad}"
-        m="${m}" />
-    </xacro:if>
-  </xacro:macro>
+  <link name="${prefix}virtual_${current_num}">
+    <inertial>
+      <mass value="0.0001"/> <inertia ixx="1e-8" ixy="0" ixz="0" iyy="1e-8" iyz="0" izz="1e-8"/>
+    </inertial>
+  </link>
+  <joint name="${prefix}joint_x_${current_num}" type="continuous">
+    <parent link="${parent}"/>
+    <child link="${prefix}virtual_${current_num}"/>
+    <xacro:if value="${current_num == 1}">
+      <origin xyz="0 0 0" rpy="0 0 0"/> </xacro:if>
+    <xacro:unless value="${current_num == 1}">
+      <origin xyz="0 0 ${-len}" rpy="0 0 0"/>
+    </xacro:unless>
+    <axis xyz="1 0 0"/>
+    <dynamics damping="0.01" friction="0.001"/>
+  </joint>
+  <link name="${prefix}link_${current_num}">
+    <xacro:cylinder_inertia m="${m}" r="${rad}" h="${len}" />
+    <visual>
+      <origin xyz="0 0 ${-len/2.0}"/>
+      <geometry><cylinder radius="${rad}" length="${len}"/></geometry>
+    </visual>
+    <collision>
+      <origin xyz="0 0 ${-len/2.0}"/>
+      <geometry><cylinder radius="${rad}" length="${len}"/></geometry>
+    </collision>
+    <self_collide>false</self_collide>
+  </link>
+  <joint name="${prefix}joint_y_${current_num}" type="continuous">
+    <parent link="${prefix}virtual_${current_num}"/>
+    <child link="${prefix}link_${current_num}"/>
+    <origin xyz="0 0 0" rpy="0 0 0"/>
+    <axis xyz="0 1 0"/>
+    <dynamics damping="0.01" friction="0.001"/>
+  </joint>
+  <xacro:if value="${current_num &lt; total_num}">
+    <xacro:flexible_chain_generator
+      prefix="${prefix}"
+      parent="${prefix}link_${current_num}"
+      current_num="${current_num + 1}"
+      total_num="${total_num}"
+      len="${len}" rad="${rad}" m="${m}" />
+  </xacro:if>
+</xacro:macro>
   <xacro:macro name="uav_cable" params="prefix parent_link is_flexible segments length radius mass">
-    <xacro:if value="${is_flexible == 'True'}">
+    <xacro:if value="${is_flexible}">
       <xacro:flexible_chain_generator
         prefix="${prefix}" parent="${parent_link}" current_num="1"
         total_num="${segments}" len="${length/segments}" rad="${radius}" m="${mass/segments}" />
     </xacro:if>
-    <xacro:unless value="${is_flexible == 'True'}">
+    <xacro:unless value="${is_flexible}">
       <xacro:rigid_cable prefix="${prefix}" parent_link="${parent_link}"
         length="${length}" radius="${radius}" mass="${mass}" />

File: urdf/crazy2fly.urdf.xacro (robot description, xacro)
@@ -19,5 +19,5 @@
 	<xacro:arg name="fixed" default="false" />
 	<!-- CONSTANTS -->
-	<xacro:property name="QCL_PACKAGE_NAME" value="quadrotor_control_lab" />
+	<xacro:property name="QCL_PACKAGE_NAME" value="acts_simulator" />
 	<xacro:property name="BASE_MESH_PATH" value="package://${QCL_PACKAGE_NAME}/meshes" />
 	<xacro:property name="BASE_CONFIG_PATH" value="$(find ${QCL_PACKAGE_NAME})/config" />

File: urdf/fake-uav_cable_assembly.xacro (robot description, xacro)
@@ -1,5 +1,5 @@
 <?xml version="1.0"?>
 <robot xmlns:xacro="http://www.ros.org/wiki/xacro">
-  <xacro:include filename="uav_component.xacro" />
+  <xacro:include filename="components/uav_component.xacro" />
   <xacro:include filename="components/cable_component.xacro" />
   <xacro:macro name="uav_plus_cable" params="prefix parent_link x y z">
@@ -13,5 +13,5 @@
       prefix="${prefix}cable_"
       parent_link="${prefix}base_link"
-      is_flexible="True"
+      is_flexible="${True}"
       segments="10"
       length="1.0"

File: urdf/panel.urdf.xacro (robot description, xacro)
@@ -1,10 +1,4 @@
 <?xml version="1.0"?>
 <robot xmlns:xacro="http://www.ros.org/wiki/xacro">
-<!-- PARAMETERS -->
-  <xacro:property name="p_mass" value="1.0" />
-  <xacro:property name="p_width" value="1" />
-  <xacro:property name="p_depth" value="1" />
-  <xacro:property name="p_height" value="0.1" />
-    <!-- inertia -->
   <xacro:macro name="panel_box_inertia" params="m w d h">
     <inertial>
@@ -15,10 +9,10 @@
     </inertial>
   </xacro:macro>
-  <xacro:macro name="panel_platform" params="prefix">
+  <xacro:macro name="panel_platform" params="prefix mass:=1.0 width:=1.0 depth:=1.0 height:=0.1">
     <link name="${prefix}base_link">
-      <xacro:panel_box_inertia m="${p_mass}" w="${p_width}" d="${p_depth}" h="${p_height}" />
+      <xacro:panel_box_inertia m="${mass}" w="${width}" d="${depth}" h="${height}" />
       <visual>
         <geometry>
-          <box size="${p_width} ${p_depth} ${p_height}"/>
+          <box size="${width} ${depth} ${height}"/>
         </geometry>
         <material name="grey"><color rgba="0.5 0.5 0.5 1"/></material>
@@ -26,8 +20,11 @@
       <collision>
         <geometry>
-          <box size="${p_width} ${p_depth} ${p_height}"/>
+          <box size="${width} ${depth} ${height}"/>
         </geometry>
       </collision>
     </link>
+    <gazebo reference="${prefix}base_link">
+      <selfCollide>true</selfCollide>
+    </gazebo>
   </xacro:macro>
 </robot>

Commit message: one drone correctly connected to the panel

File: urdf/acts.urdf.xacro (robot description, xacro)
@@ -2,28 +2,24 @@
 <robot xmlns:xacro="http://www.ros.org/wiki/xacro" name="acts_system">
   <xacro:include filename="panel.urdf.xacro" />
-  <xacro:include filename="uav_cable_assembly.xacro" />
-  <xacro:include filename="components/cable_component.xacro" />
+  <xacro:include filename="uav_cable_assembly.urdf.xacro" />
   <xacro:panel_platform
-  prefix="main_panel_"
-  mass="2.5"
-  width="2.0"
-  depth="2.0"
-  height="0.2" />
-  <link name="panel_corner_link" />
-  <joint name="panel_to_corner" type="fixed">
-    <parent link="main_panel_base_link"/>
-    <child link="panel_corner_link"/>
-    <origin xyz="0.8 0.8 0.1" rpy="0 3.14159 0"/>  <!-- the cable is directed upwards-->
-    <gazebo reference="panel_to_corner">
-    <disableFixedJointLumping>true</disableFixedJointLumping>
-  </gazebo>
+    prefix="main_panel_"
+    mass="2.5"
+    width="2.0"
+    depth="2.0"
+    height="0.2" />
+  <xacro:uav_towing_unit
+    prefix="drone1_"
+    panel_link="main_panel_base_link"
+    x="0" y="0" z="-0.1"
+    segments="30"
+    length="1.0"
+    radius="0.005"
+    mass="0.05" />
+  <link name="world"/>
+  <joint name="world_fixed" type="fixed">
+    <parent link="world"/>
+    <child link="base_link"/>
+    <origin xyz="0 0 2.0" rpy="0 0 0"/>
   </joint>
-  <xacro:uav_cable
-    prefix="upward_cable_"
-    parent_link="panel_corner_link"
-    is_flexible="${True}"
-    segments="10"
-    length="1.5"
-    radius="0.01"
-    mass="0.2" />
 </robot>

File: urdf/uav_cable_assembly.urdf.xacro (robot description, xacro)
@@ -1,20 +1,29 @@
 <?xml version="1.0"?>
-<robot xmlns:xacro="http://www.ros.org/wiki/xacro" name="uav_cable_assembly">
-<xacro:include filename="$(find acts_simulator)/urdf/crazy2fly.urdf.xacro" />
+<robot xmlns:xacro="http://www.ros.org/wiki/xacro">
+  <xacro:include filename="$(find acts_simulator)/urdf/crazy2fly.urdf.xacro" />
+  <xacro:include filename="$(find acts_simulator)/urdf/components/cable_component.xacro" />
+  <xacro:macro name="uav_towing_unit" params="prefix panel_link x y z segments length radius mass">
+    <xacro:uav_cable
+      prefix="${prefix}"
+      parent_link="base_link"
+      is_flexible="true"
+      segments="${segments}"
+      length="${length}"
+      radius="${radius}"
+      mass="${mass}" />
+    <joint name="${prefix}cable_to_panel_joint" type="continuous">
+      <parent link="${prefix}link_${segments}"/>
+      <child link="${panel_link}"/>
+      <origin xyz="${x} ${y} ${z}" rpy="0 0 0"/>
+      <axis xyz="1 0 0"/>
+      <dynamics damping="0.1" friction="0.01"/>
+    </joint>
+  </xacro:macro>
+</robot>
 <!-- # TODO: delete these lines to allow the uav to follow gravity-->
-<link name="world"/>
+<!-- <link name="world"/>
 <joint name="world_fixed" type="fixed">
   <parent link="world"/>
   <child link="base_link"/>
   <origin xyz="0 0 0" rpy="0 0 0"/>
-</joint>
-<xacro:include filename="$(find acts_simulator)/urdf/components/cable_component.xacro" />
-  <xacro:uav_cable
-    prefix="uav1_"
-    parent_link="base_link"
-    is_flexible="true"
-    segments="30"
-    length="1.0"
-    radius="0.005"
-    mass="0.05" />
-</robot>
+</joint> -->
