Commit message: multiple UAV but they are hanging out from the panel

File: urdf/acts.urdf.xacro (robot description, xacro)
@@ -3,23 +3,30 @@
   <xacro:include filename="panel.urdf.xacro" />
   <xacro:include filename="uav_cable_assembly.urdf.xacro" />
+  <link name="world"/>
   <xacro:panel_platform
     prefix="main_panel_"
     mass="2.5"
-    width="2.0"
-    depth="2.0"
+    width="1.0"
+    depth="1.0"
     height="0.2" />
+  <joint name="world_to_panel" type="fixed">
+    <parent link="world"/>
+    <child link="main_panel_base_link"/>
+    <origin xyz="0 0 1.0" rpy="0 0 0"/> </joint>
   <xacro:uav_towing_unit
     prefix="drone1_"
     panel_link="main_panel_base_link"
-    x="0" y="0" z="-0.1"
-    segments="30"
+    x="1.0" y="1.0" z="1"
+    segments="3"
     length="1.0"
     radius="0.005"
     mass="0.05" />
-  <link name="world"/>
-  <joint name="world_fixed" type="fixed">
-    <parent link="world"/>
-    <child link="base_link"/>
-    <origin xyz="0 0 2.0" rpy="0 0 0"/>
-  </joint>
+  <xacro:uav_towing_unit
+    prefix="drone2_"
+    panel_link="main_panel_base_link"
+    x="-1.0" y="-1.0" z="1"
+    segments="3"
+    length="1.0"
+    radius="0.005"
+    mass="0.05" />
 </robot>

File: urdf/components/core.xacro (robot description, xacro)
@@ -1,27 +1,17 @@
 <?xml version="1.0" encoding="utf-8"?>
-<!--
-File: core.xacro
-Project: Quadrotor Control Lab
-File Created: Tuesday, 25th November 2025 9:31:43 AM
-Author: nknab
-Email: kojo.anyinam-boateng@ls2n.fr
-Version: 1.0.0
-Brief: Core components for crazy2fly drone
-~~~~~
-Last Modified: Tuesday, 25th November 2025 10:44:59 AM
-Modified By: nknab
-~~~~~
-Copyright ©2025 nknab
--->
 <robot xmlns:xacro="http://www.ros.org/wiki/xacro">
-	<!-- VARIABLES -->
-	<xacro:property name="core_mesh_path" value="${BASE_MESH_PATH}/core" />
-	<xacro:macro name="core" params="parent_link *joint_pose">
-		<xacro:box_properties width="0.399681" length="0.399681" height="0.162643" />
-		<xacro:com mass="0.99" x="0.000847" y="-0.000015" z="-0.001832" />
-		<xacro:child_macro name="c2f" parent_link="${parent_link}"
-			file="core" shape="box" mesh_path="${core_mesh_path}">
-			<xacro:insert_block name="joint_pose" />
-		</xacro:child_macro>
-	</xacro:macro>
+    <xacro:property name="core_mesh_path" value="${BASE_MESH_PATH}/core" />
+    <xacro:macro name="core" params="parent_link prefix *joint_pose">
+        <xacro:box_properties width="0.399681" length="0.399681" height="0.162643" />
+        <xacro:com mass="0.99" x="0.000847" y="-0.000015" z="-0.001832" />
+        <xacro:child_macro
+            name="c2f"
+            parent_link="${parent_link}"
+            prefix="${prefix}"
+            file="core"
+            shape="box"
+            mesh_path="${core_mesh_path}">
+            <xacro:insert_block name="joint_pose" />
+        </xacro:child_macro>
+    </xacro:macro>
 </robot>

File: urdf/components/propeller.xacro (robot description, xacro)
@@ -1,56 +1,43 @@
 <?xml version="1.0" encoding="utf-8"?>
-<!--
-File: propeller.xacro
-Project: Quadrotor Control Lab
-File Created: Tuesday, 25th November 2025 10:09:57 AM
-Author: nknab
-Email: kojo.anyinam-boateng@ls2n.fr
-Version: 1.0.0
-Brief: Propeller macro to be used to create the propeller of the drone.
-~~~~~
-Last Modified: Tuesday, 25th November 2025 10:38:12 AM
-Modified By: nknab
-~~~~~
-Copyright ©2025 nknab
--->
 <robot xmlns:xacro="http://www.ros.org/wiki/xacro">
-	<xacro:macro name="prop"
-		params="parent_link prefix:='' motor_number prop_type:=cw *joint_pose">
-		<xacro:property name="propeller_mesh_path"
-			value="${BASE_MESH_PATH}/propellers/${prop_type}" />
-		<xacro:hollow_cylinder_properties inner_radius="0.0025" outer_radius="0.101608"
-			height="0.012855" />
-		<xacro:com mass="0.005" x="0.0" y="0.0" z="0.001409" />
-		<xacro:child_macro name="${prop_type}_propeller" parent_link="${parent_link}"
-			prefix="${prefix}" file="${prop_type}" shape="hollow" mesh_path="${propeller_mesh_path}"
-			joint_type="continuous">
-			<xacro:insert_block name="joint_pose" />
-		</xacro:child_macro>
-		<xacro:if value="${prefix != ''}">
-			<xacro:property name="resolved_prefix" value="${prefix}_${prop_type}_propeller" />
-		</xacro:if>
-		<xacro:unless value="${prefix != ''}">
-			<xacro:property name="resolved_prefix" value="${prop_type}_propeller" />
-		</xacro:unless>
-		<gazebo>
-			<plugin filename="gz-sim-multicopter-motor-model-system"
-				name="gz::sim::systems::MulticopterMotorModel">
-				<robotNamespace>$(arg namespace)</robotNamespace>
-				<jointName>${resolved_prefix}_joint</jointName>
-				<linkName>${resolved_prefix}_link</linkName>
-				<turningDirection>${prop_type}</turningDirection>
-				<timeConstantUp>0.000001</timeConstantUp>
-				<timeConstantDown>0.000001</timeConstantDown>
-				<maxRotVelocity>1466</maxRotVelocity>
-				<motorConstant>5.5e-06</motorConstant>
-				<momentConstant>0.06</momentConstant>
-				<commandSubTopic>command/motor_speed</commandSubTopic>
-				<actuator_number>${motor_number}</actuator_number>
-				<rotorDragCoefficient>0.00000175</rotorDragCoefficient>
-				<rollingMomentCoefficient>1e-08</rollingMomentCoefficient>
-				<rotorVelocitySlowdownSim>10</rotorVelocitySlowdownSim>
-				<motorType>velocity</motorType>
-			</plugin>
-		</gazebo>
-	</xacro:macro>
+    <xacro:macro name="prop"
+        params="parent_link drone_prefix:='' prefix:='' motor_number prop_type:=cw *joint_pose">
+        <xacro:property name="propeller_mesh_path"
+            value="${BASE_MESH_PATH}/propellers/${prop_type}" />
+        <xacro:hollow_cylinder_properties inner_radius="0.0025" outer_radius="0.101608"
+            height="0.012855" />
+        <xacro:com mass="0.005" x="0.0" y="0.0" z="0.001409" />
+        <xacro:if value="${prefix != ''}">
+            <xacro:property name="resolved_prefix" value="${drone_prefix}${prefix}_${prop_type}_propeller" />
+        </xacro:if>
+        <xacro:unless value="${prefix != ''}">
+            <xacro:property name="resolved_prefix" value="${drone_prefix}${prop_type}_propeller" />
+        </xacro:unless>
+        <xacro:child_macro name="${resolved_prefix}" parent_link="${parent_link}"
+            prefix="" file="${prop_type}" shape="hollow" mesh_path="${propeller_mesh_path}"
+            joint_type="continuous">
+            <xacro:insert_block name="joint_pose" />
+        </xacro:child_macro>
+        <gazebo>
+            <plugin filename="gz-sim-multicopter-motor-model-system"
+                name="gz::sim::systems::MulticopterMotorModel">
+                <robotNamespace>${ns}${drone_prefix}</robotNamespace>
+                <jointName>${resolved_prefix}_joint</jointName>
+                <linkName>${resolved_prefix}_link</linkName>
+                <turningDirection>${prop_type}</turningDirection>
+                <timeConstantUp>0.000001</timeConstantUp>
+                <timeConstantDown>0.000001</timeConstantDown>
+                <maxRotVelocity>1466</maxRotVelocity>
+                <motorConstant>5.5e-06</motorConstant>
+                <motorConstant>5.5e-06</motorConstant>
+                <momentConstant>0.06</momentConstant>
+                <commandSubTopic>command/motor_speed</commandSubTopic>
+                <actuator_number>${motor_number}</actuator_number>
+                <rotorDragCoefficient>0.00000175</rotorDragCoefficient>
+                <rollingMomentCoefficient>1e-08</rollingMomentCoefficient>
+                <rotorVelocitySlowdownSim>10</rotorVelocitySlowdownSim>
+                <motorType>velocity</motorType>
+            </plugin>
+        </gazebo>
+    </xacro:macro>
 </robot>

File: urdf/crazy2fly.urdf.xacro (robot description, xacro)
@@ -36,12 +36,13 @@
 	<xacro:include filename="components/propeller.xacro" />
 	<xacro:include filename="sensors/imu.xacro" />
+	<xacro:macro name="crazy2fly" params="prefix">
 	<!-- BASE LINK -->
-	<link name="base_link" />
+	<link name="${prefix}base_link" />
 	<!-- CORE -->
-	<xacro:core parent_link="base">
+	<xacro:core parent_link="${prefix}base_link" prefix="${prefix}">
 		<origin xyz="0 0 0" rpy="0 0 0" />
 	</xacro:core>
 	<!-- IMU SENSOR -->
-	<xacro:imu parent_link="c2f" sensor="px4">
+	<xacro:imu parent_link="${prefix}c2f" drone_prefix="${prefix}" sensor="px4">
 		<origin xyz="0 0 0.0315" rpy="0 0 0" />
 	</xacro:imu>
@@ -50,14 +51,14 @@
 	<xacro:property name="prop_z_offset" value="0.017" />
 	<xacro:property name="prop_Y" value="${radians(90)}" />
-	<xacro:prop parent_link="base" prefix="front" motor_number="2">
+	<xacro:prop parent_link="${prefix}base_link" drone_prefix="${prefix}" prefix="front" motor_number="2">
 		<origin xyz="${prop_xy_offset} 0 ${prop_z_offset}" rpy="0 0 0" />
 	</xacro:prop>
-	<xacro:prop parent_link="base" prefix="back" motor_number="3">
+	<xacro:prop parent_link="${prefix}base_link" drone_prefix="${prefix}" prefix="back" motor_number="3">
 		<origin xyz="-${prop_xy_offset} 0 ${prop_z_offset}" rpy="0 0 0" />
 	</xacro:prop>
-	<xacro:prop parent_link="base" prefix="right" prop_type="ccw" motor_number="0">
+	<xacro:prop parent_link="${prefix}base_link" drone_prefix="${prefix}" prefix="right" prop_type="ccw" motor_number="0">
 		<origin xyz="0 -${prop_xy_offset} ${prop_z_offset}" rpy="0 0 ${prop_Y}" />
 	</xacro:prop>
-	<xacro:prop parent_link="base" prefix="left" prop_type="ccw" motor_number="1">
+	<xacro:prop parent_link="${prefix}base_link" drone_prefix="${prefix}" prefix="left" prop_type="ccw" motor_number="1">
 		<origin xyz="0 ${prop_xy_offset} ${prop_z_offset}" rpy="0 0 ${prop_Y}" />
 	</xacro:prop>
@@ -66,36 +67,30 @@
 		<!-- JOINT STATES -->
 		<plugin filename="gz-sim-joint-state-publisher-system"
-			name="gz::sim::systems::JointStatePublisher">
-			<topic>${ns}joint_states</topic>
-			<joint_name>front_cw_propeller_joint</joint_name>
-			<joint_name>back_cw_propeller_joint</joint_name>
-			<joint_name>right_ccw_propeller_joint</joint_name>
-			<joint_name>left_ccw_propeller_joint</joint_name>
-		</plugin>
+		name="gz::sim::systems::JointStatePublisher">
+		<topic>${ns}${prefix}joint_states</topic>
+		<joint_name>${prefix}front_cw_propeller_joint</joint_name>
+		<joint_name>${prefix}back_cw_propeller_joint</joint_name>
+		<joint_name>${prefix}right_ccw_propeller_joint</joint_name>
+		<joint_name>${prefix}left_ccw_propeller_joint</joint_name>
+	</plugin>
 		<!-- ODOMETRY PUBLISHER -->
-		<plugin name="gz::sim::systems::OdometryPublisher"
-			filename="gz-sim-odometry-publisher-system">
+		<plugin name="gz::sim::systems::OdometryPublisher" filename="gz-sim-odometry-publisher-system">
 			<odom_publish_frequency>100</odom_publish_frequency>
 			<dimensions>3</dimensions>
-			<xacro:if value="${'$(arg namespace)' != ''}">
-				<odom_frame>$(arg namespace)</odom_frame>
-			</xacro:if>
-			<xacro:unless value="${'$(arg namespace)' != ''}">
-				<odom_frame>crazy2fly</odom_frame>
-			</xacro:unless>
-			<odom_topic>${ns}mocap/odom</odom_topic>
+			<odom_frame>${prefix}crazy2fly</odom_frame>
+			<odom_topic>${ns}${prefix}mocap/odom</odom_topic>
 			<odom_covariance_topic>${ns}mocap/odometry_with_covariance</odom_covariance_topic>
-			<tf_topic>${ns}mocap/pose</tf_topic>
-			<robot_base_frame>px4_imu_link</robot_base_frame>
+			<tf_topic>${ns}${prefix}mocap/pose</tf_topic>
+			<robot_base_frame>${prefix}px4_imu_link</robot_base_frame>
 		</plugin>
 		<!-- DETACHABLE JOINT -->
 		<xacro:if value="$(arg fixed)">
-			<plugin filename="gz-sim-detachable-joint-system"
-				name="gz::sim::systems::DetachableJoint">
-				<parent_link>base_link</parent_link>
-				<child_model>fixed_support</child_model>
-				<child_link>fixed_support_link</child_link>
-			</plugin>
+		<plugin filename="gz-sim-detachable-joint-system" name="gz::sim::systems::DetachableJoint">
+			<parent_link>${prefix}base_link</parent_link>
+			<child_model>${prefix}fixed_support</child_model>
+			<child_link>${prefix}fixed_support_link</child_link>
+		</plugin>
 		</xacro:if>
 	</gazebo>
+</xacro:macro>
 </robot>

File: urdf/macros/child.xacro (robot description, xacro)
@@ -1,67 +1,46 @@
 <?xml version="1.0" encoding="utf-8"?>
-<!--
-File: child.xacro
-Project: Quadrotor Control Lab
-File Created: Tuesday, 25th November 2025 9:30:48 AM
-Author: nknab
-Email: kojo.anyinam-boateng@ls2n.fr
-Version: 1.0.0
-Brief:  Macro for creating child links and joints.
-~~~~~
-Last Modified: Tuesday, 25th November 2025 10:15:27 AM
-Modified By: nknab
-~~~~~
-Copyright ©2025 nknab
--->
 <robot xmlns:xacro="http://www.ros.org/wiki/xacro">
-	<xacro:macro name="child_macro"
-		params="name parent_link mesh_path file prefix:='' shape:='' joint_type:=fixed *joint_pose">
-		<xacro:if value="${prefix != ''}">
-			<xacro:property name="resolved_prefix" value="${prefix}_${name}" />
-		</xacro:if>
-		<xacro:unless value="${prefix != ''}">
-			<xacro:property name="resolved_prefix" value="${name}" />
-		</xacro:unless>
-		<!-- Joint -->
-		<joint name="${resolved_prefix}_joint" type="${joint_type}">
-			<parent link="${parent_link}_link" />
-			<child link="${resolved_prefix}_link" />
-			<xacro:insert_block name="joint_pose" />
-			<xacro:if value="${joint_type == 'continuous' or joint_type == 'revolute'}">
-				<axis xyz="0 0 1" />
-			</xacro:if>
-			<xacro:if value="${joint_type == 'revolute'}">
-				<limit lower="${lower}" upper="${upper}" velocity="${velocity}" effort="${effort}" />
-				<dynamics damping="${damping}" friction="${friction}" />
-			</xacro:if>
-		</joint>
-		<!-- Link -->
-		<link name="${resolved_prefix}_link">
-			<visual name="${resolved_prefix}_link_visual">
-				<origin xyz="0 0 0" rpy="0 0 0" />
-				<geometry>
-					<mesh filename="${mesh_path}/${file}.dae" />
-				</geometry>
-			</visual>
-			<collision name="${resolved_prefix}_link_collision">
-				<origin xyz="0 0 0" rpy="0 0 0" />
-				<geometry>
-					<mesh filename="${mesh_path}/${file}.stl" />
-				</geometry>
-			</collision>
-			<xacro:if value="${shape == 'hollow'}">
-				<xacro:hollow_cylinder_inertial prefix="${resolved_prefix}_link" mass="${mass}"
-					inner_radius="${inner_radius}" outer_radius="${outer_radius}"
-					height="${height}">
-					<origin xyz="${com_x} ${com_y} ${com_z}" rpy="0 0 0" />
-				</xacro:hollow_cylinder_inertial>
-			</xacro:if>
-			<xacro:if value="${shape == 'box'}">
-				<xacro:box_inertial prefix="${resolved_prefix}_link" mass="${mass}"
-					x="${width}" y="${length}" z="${height}">
-					<origin xyz="${com_x} ${com_y} ${com_z}" rpy="0 0 0" />
-				</xacro:box_inertial>
-			</xacro:if>
-		</link>
-	</xacro:macro>
+    <xacro:macro name="child_macro"
+        params="name parent_link mesh_path file prefix:='' shape:='' joint_type:=fixed *joint_pose">
+        <xacro:property name="resolved_prefix" value="${prefix}${name}" />
+        <joint name="${resolved_prefix}_joint" type="${joint_type}">
+            <parent link="${parent_link}" />
+            <child link="${resolved_prefix}_link" />
+            <xacro:insert_block name="joint_pose" />
+            <xacro:if value="${joint_type == 'continuous' or joint_type == 'revolute'}">
+                <axis xyz="0 0 1" />
+            </xacro:if>
+            <xacro:if value="${joint_type == 'revolute'}">
+                <limit lower="${lower}" upper="${upper}" velocity="${velocity}" effort="${effort}" />
+                <dynamics damping="${damping}" friction="${friction}" />
+            </xacro:if>
+        </joint>
+        <link name="${resolved_prefix}_link">
+            <visual name="${resolved_prefix}_link_visual">
+                <origin xyz="0 0 0" rpy="0 0 0" />
+                <geometry>
+                    <mesh filename="${mesh_path}/${file}.dae" />
+                </geometry>
+            </visual>
+            <collision name="${resolved_prefix}_link_collision">
+                <origin xyz="0 0 0" rpy="0 0 0" />
+                <geometry>
+                    <mesh filename="${mesh_path}/${file}.stl" />
+                </geometry>
+            </collision>
+            <xacro:if value="${shape == 'hollow'}">
+                <xacro:hollow_cylinder_inertial prefix="${resolved_prefix}_link" mass="${mass}"
+                    inner_radius="${inner_radius}" outer_radius="${outer_radius}"
+                    height="${height}">
+                    <origin xyz="${com_x} ${com_y} ${com_z}" rpy="0 0 0" />
+                </xacro:hollow_cylinder_inertial>
+            </xacro:if>
+            <xacro:if value="${shape == 'box'}">
+                <xacro:box_inertial prefix="${resolved_prefix}_link" mass="${mass}"
+                    x="${width}" y="${length}" z="${height}">
+                    <origin xyz="${com_x} ${com_y} ${com_z}" rpy="0 0 0" />
+                </xacro:box_inertial>
+            </xacro:if>
+        </link>
+    </xacro:macro>
 </robot>

File: urdf/sensors/imu.xacro (robot description, xacro)
@@ -15,12 +15,12 @@
 -->
 <robot xmlns:xacro="http://www.ros.org/wiki/xacro">
-	<xacro:macro name="imu" params="parent_link prefix:='' sensor *joint_pose">
+	<xacro:macro name="imu" params="parent_link drone_prefix:='' prefix:='' sensor *joint_pose">
 		<xacro:property name="imu_yaml_file" value="${BASE_CONFIG_PATH}/sensors/imu.yaml" />
 		<xacro:property name="props" value="${xacro.load_yaml(imu_yaml_file)}" />
 		<xacro:if value="${prefix != ''}">
-			<xacro:property name="resolved_prefix" value="${prefix}_${sensor}_imu" />
+			<xacro:property name="resolved_prefix" value="${drone_prefix}${prefix}_${sensor}_imu" />
 		</xacro:if>
 		<xacro:unless value="${prefix != ''}">
-			<xacro:property name="resolved_prefix" value="${sensor}_imu" />
+			<xacro:property name="resolved_prefix" value="${drone_prefix}${sensor}_imu" />
 		</xacro:unless>
 		<!-- Joint -->
@@ -43,5 +43,5 @@
 		</link>
 		<gazebo reference="${resolved_prefix}_link">
-			<sensor name="imu_sensor" type="imu">
+			<sensor name="${resolved_prefix}_sensor" type="imu">
 				<always_on>true</always_on>
 				<update_rate>${props.update_rate}</update_rate>
@@ -113,5 +113,5 @@
 					</linear_acceleration>
 				</imu>
-				<topic>${ns}${props.topic}</topic>
+				<topic>${ns}${drone_prefix}${props.topic}</topic>
 				<gz_frame_id>${resolved_prefix}_link</gz_frame_id>
 			</sensor>

File: urdf/uav_cable_assembly.urdf.xacro (robot description, xacro)
@@ -4,7 +4,8 @@
   <xacro:include filename="$(find acts_simulator)/urdf/components/cable_component.xacro" />
   <xacro:macro name="uav_towing_unit" params="prefix panel_link x y z segments length radius mass">
+    <xacro:crazy2fly prefix="${prefix}" />
     <xacro:uav_cable
       prefix="${prefix}"
-      parent_link="base_link"
+      parent_link="${panel_link}"
       is_flexible="true"
       segments="${segments}"
@@ -12,18 +13,9 @@
       radius="${radius}"
       mass="${mass}" />
-    <joint name="${prefix}cable_to_panel_joint" type="continuous">
-      <parent link="${prefix}link_${segments}"/>
-      <child link="${panel_link}"/>
-      <origin xyz="${x} ${y} ${z}" rpy="0 0 0"/>
-      <axis xyz="1 0 0"/>
-      <dynamics damping="0.1" friction="0.01"/>
-    </joint>
-  </xacro:macro>
+   <joint name="${prefix}cable_to_drone_joint" type="fixed">
+    <parent link="${prefix}link_${segments}"/>
+    <child link="${prefix}base_link"/>
+    <origin xyz="0 0 ${-length/segments}" rpy="0 0 0"/>
+  </joint>
+</xacro:macro>
 </robot>
-<!-- # TODO: delete these lines to allow the uav to follow gravity-->
-<!-- <link name="world"/>
-<joint name="world_fixed" type="fixed">
-  <parent link="world"/>
-  <child link="base_link"/>
-  <origin xyz="0 0 0" rpy="0 0 0"/>
-</joint> -->
