Commit message: Multible uav connected to the panel

File: urdf/acts.urdf.xacro (robot description, xacro)
@@ -6,27 +6,8 @@
   <xacro:panel_platform
     prefix="main_panel_"
-    mass="2.5"
-    width="1.0"
-    depth="1.0"
-    height="0.2" />
-  <joint name="world_to_panel" type="fixed">
-    <parent link="world"/>
-    <child link="main_panel_base_link"/>
-    <origin xyz="0 0 1.0" rpy="0 0 0"/> </joint>
-  <xacro:uav_towing_unit
-    prefix="drone1_"
-    panel_link="main_panel_base_link"
-    x="1.0" y="1.0" z="1"
-    segments="3"
-    length="1.0"
-    radius="0.005"
-    mass="0.05" />
-  <xacro:uav_towing_unit
-    prefix="drone2_"
-    panel_link="main_panel_base_link"
-    x="-1.0" y="-1.0" z="1"
-    segments="3"
-    length="1.0"
-    radius="0.005"
-    mass="0.05" />
+    mass="2.5" width="5.0" depth="5.0" height="0.2" />
+  <xacro:add_drone id="1" x="1"  y="2"  z="1.2" segments="10" length="1" primary="true" />
+  <xacro:add_drone id="2" x="2"  y="2" z="1.2" segments="10"  length="1" handle_id="2" />
+  <xacro:add_drone id="3" x="1" y="3" z="1.2" segments="10"  length="1" handle_id="3" />
+  <xacro:add_drone id="4" x="2" y="3"  z="1.2" segments="10"  length="1" handle_id="4" />
 </robot>

File: urdf/components/cable_component.xacro (robot description, xacro)
@@ -9,4 +9,5 @@
     </inertial>
   </xacro:macro>
+<!-- ____________   Rigid cable  _______________________-->
   <xacro:macro name="rigid_cable" params="prefix parent_link length radius mass">
     <link name="${prefix}rigid_link">
@@ -27,4 +28,5 @@
     </joint>
   </xacro:macro>
+<!-- ____________   Flexible cable  _______________________-->
   <xacro:macro name="flexible_chain_generator" params="prefix parent current_num total_num len rad m">
   <link name="${prefix}virtual_${current_num}">
@@ -72,4 +74,5 @@
   </xacro:if>
 </xacro:macro>
+<!-- ____________   Cable macro  _______________________-->
   <xacro:macro name="uav_cable" params="prefix parent_link is_flexible segments length radius mass">
     <xacro:if value="${is_flexible}">

File: urdf/panel.urdf.xacro (robot description, xacro)
@@ -9,22 +9,32 @@
     </inertial>
   </xacro:macro>
-  <xacro:macro name="panel_platform" params="prefix mass:=1.0 width:=1.0 depth:=1.0 height:=0.1">
+  <xacro:macro name="handle" params="prefix suffix x y z">
+    <link name="${prefix}handle_${suffix}">
+      <inertial>
+        <mass value="0.001"/>
+        <inertia ixx="1e-9" ixy="0" ixz="0" iyy="1e-9" iyz="0" izz="1e-9"/>
+      </inertial>
+    </link>
+    <joint name="${prefix}handle_${suffix}_joint" type="fixed">
+      <parent link="${prefix}base_link"/>
+      <child link="${prefix}handle_${suffix}"/>
+      <origin xyz="${x} ${y} ${z}" rpy="0 0 0"/>
+    </joint>
+  </xacro:macro>
+  <xacro:macro name="panel_platform" params="prefix mass width depth height">
     <link name="${prefix}base_link">
       <xacro:panel_box_inertia m="${mass}" w="${width}" d="${depth}" h="${height}" />
       <visual>
-        <geometry>
-          <box size="${width} ${depth} ${height}"/>
-        </geometry>
+        <geometry><box size="${width} ${depth} ${height}"/></geometry>
         <material name="grey"><color rgba="0.5 0.5 0.5 1"/></material>
       </visual>
       <collision>
-        <geometry>
-          <box size="${width} ${depth} ${height}"/>
-        </geometry>
+        <geometry><box size="${width} ${depth} ${height}"/></geometry>
       </collision>
     </link>
-    <gazebo reference="${prefix}base_link">
-      <selfCollide>true</selfCollide>
-    </gazebo>
+    <xacro:handle prefix="${prefix}" suffix="1" x="0.2"  y="0.2"  z="${height/2}" />
+    <xacro:handle prefix="${prefix}" suffix="2" x="0.2"  y="-0.2" z="${height/2}" />
+    <xacro:handle prefix="${prefix}" suffix="3" x="-0.2" y="-0.2" z="${height/2}" />
+    <xacro:handle prefix="${prefix}" suffix="4" x="-0.2" y="0.2"  z="${height/2}" />
   </xacro:macro>
 </robot>

File: urdf/uav_cable_assembly.urdf.xacro (robot description, xacro)
@@ -3,9 +3,14 @@
   <xacro:include filename="$(find acts_simulator)/urdf/crazy2fly.urdf.xacro" />
   <xacro:include filename="$(find acts_simulator)/urdf/components/cable_component.xacro" />
-  <xacro:macro name="uav_towing_unit" params="prefix panel_link x y z segments length radius mass">
+  <xacro:macro name="uav_towing_unit" params="prefix panel_link x y z segments length radius mass attach_to_panel">
+    <joint name="world_to_${prefix}_joint" type="fixed">
+      <parent link="world"/>
+      <child link="${prefix}base_link"/>
+      <origin xyz="${x} ${y} ${z}" rpy="0 0 0"/>
+    </joint>
     <xacro:crazy2fly prefix="${prefix}" />
     <xacro:uav_cable
       prefix="${prefix}"
-      parent_link="${panel_link}"
+      parent_link="${prefix}base_link"
       is_flexible="true"
       segments="${segments}"
@@ -13,9 +18,40 @@
       radius="${radius}"
       mass="${mass}" />
-   <joint name="${prefix}cable_to_drone_joint" type="fixed">
-    <parent link="${prefix}link_${segments}"/>
-    <child link="${prefix}base_link"/>
-    <origin xyz="0 0 ${-length/segments}" rpy="0 0 0"/>
-  </joint>
-</xacro:macro>
+    <link name="${prefix}hook_link">
+      <inertial>
+        <mass value="0.01"/>
+        <inertia ixx="1e-8" ixy="0" ixz="0" iyy="1e-8" iyz="0" izz="1e-8"/>
+      </inertial>
+    </link>
+    <joint name="${prefix}cable_to_hook_joint" type="fixed">
+      <parent link="${prefix}link_${segments}"/>
+      <child link="${prefix}hook_link"/>
+      <origin xyz="0 0 ${-length/segments}" rpy="0 0 0"/>
+    </joint>
+    <xacro:if value="${attach_to_panel}">
+      <joint name="${prefix}hook_to_panel_joint" type="continuous">
+        <parent link="${prefix}hook_link"/>
+        <child link="${panel_link}"/>
+        <axis xyz="1 0 0"/>
+        <origin xyz="0 0 -0.1" rpy="0 0 0"/>
+      </joint>
+    </xacro:if>
+  </xacro:macro>
+  <xacro:macro name="add_drone" params="id x y z segments length handle_id:=1 primary:=false">
+    <xacro:uav_towing_unit
+      prefix="drone${id}_"
+      panel_link="main_panel_base_link"
+      x="${x}" y="${y}" z="${z}"
+      segments="${segments}"
+      length="${length}" radius="0.01" mass="0.1"
+      attach_to_panel="${primary}" />
+    <xacro:unless value="${primary}">
+      <gazebo>
+        <joint name="drone${id}_loop_closure" type="fixed">
+          <parent>main_panel_handle_${handle_id}</parent>
+          <child>drone${id}_hook_link</child>
+        </joint>
+      </gazebo>
+    </xacro:unless>
+  </xacro:macro>
 </robot>

Commit message: solved some errors

File: urdf/acts.urdf.xacro (robot description, xacro)
@@ -6,8 +6,8 @@
   <xacro:panel_platform
     prefix="main_panel_"
-    mass="2.5" width="5.0" depth="5.0" height="0.2" />
-  <xacro:add_drone id="1" x="1"  y="2"  z="1.2" segments="10" length="1" primary="true" />
-  <xacro:add_drone id="2" x="2"  y="2" z="1.2" segments="10"  length="1" handle_id="2" />
-  <xacro:add_drone id="3" x="1" y="3" z="1.2" segments="10"  length="1" handle_id="3" />
-  <xacro:add_drone id="4" x="2" y="3"  z="1.2" segments="10"  length="1" handle_id="4" />
+    mass="2.5" width="2.0" depth="2.0" height="0.2" />
+  <xacro:add_drone id="1" x="0"  y="1"  z="1.2" segments="10" length="1" primary="true" />
+  <xacro:add_drone id="2" x="0"  y="0" z="1.2" segments="10"  length="1" handle_id="2" />
+  <!--<xacro:add_drone id="3" x="1" y="3" z="1.2" segments="10"  length="1" handle_id="3" />
+  <xacro:add_drone id="4" x="2" y="3"  z="1.2" segments="10"  length="1" handle_id="4" /> -->
 </robot>

File: urdf/components/cable_component.xacro (robot description, xacro)
@@ -29,5 +29,5 @@
   </xacro:macro>
 <!-- ____________   Flexible cable  _______________________-->
-  <xacro:macro name="flexible_chain_generator" params="prefix parent current_num total_num len rad m">
+  <xacro:macro name="flexible_chain_generator" params="prefix parent current_num total_num cable_len rad m">
   <link name="${prefix}virtual_${current_num}">
     <inertial>
@@ -41,5 +41,5 @@
       <origin xyz="0 0 0" rpy="0 0 0"/> </xacro:if>
     <xacro:unless value="${current_num == 1}">
-      <origin xyz="0 0 ${-len}" rpy="0 0 0"/>
+      <origin xyz="0 0 ${-cable_len}" rpy="0 0 0"/>
     </xacro:unless>
     <axis xyz="1 0 0"/>
@@ -47,12 +47,12 @@
   </joint>
   <link name="${prefix}link_${current_num}">
-    <xacro:cylinder_inertia m="${m}" r="${rad}" h="${len}" />
+    <xacro:cylinder_inertia m="${m}" r="${rad}" h="${cable_len}" />
     <visual>
-      <origin xyz="0 0 ${-len/2.0}"/>
-      <geometry><cylinder radius="${rad}" length="${len}"/></geometry>
+      <origin xyz="0 0 ${-cable_len/2.0}"/>
+      <geometry><cylinder radius="${rad}" length="${cable_len}"/></geometry>
     </visual>
     <collision>
-      <origin xyz="0 0 ${-len/2.0}"/>
-      <geometry><cylinder radius="${rad}" length="${len}"/></geometry>
+      <origin xyz="0 0 ${-cable_len/2.0}"/>
+      <geometry><cylinder radius="${rad}" length="${cable_len}"/></geometry>
     </collision>
     <self_collide>false</self_collide>
@@ -71,5 +71,5 @@
       current_num="${current_num + 1}"
       total_num="${total_num}"
-      len="${len}" rad="${rad}" m="${m}" />
+      cable_len="${cable_len}" rad="${rad}" m="${m}" />
   </xacro:if>
 </xacro:macro>
@@ -79,5 +79,5 @@
       <xacro:flexible_chain_generator
         prefix="${prefix}" parent="${parent_link}" current_num="1"
-        total_num="${segments}" len="${length/segments}" rad="${radius}" m="${mass/segments}" />
+        total_num="${segments}" cable_len="${length/segments}" rad="${radius}" m="${mass/segments}" />
     </xacro:if>
     <xacro:unless value="${is_flexible}">

File: urdf/panel.urdf.xacro (robot description, xacro)
@@ -33,8 +33,9 @@
       </collision>
     </link>
-    <xacro:handle prefix="${prefix}" suffix="1" x="0.2"  y="0.2"  z="${height/2}" />
+    <xacro:handle prefix="${prefix}" suffix="1" x="1"  y="1"  z="${height/2}" />
     <xacro:handle prefix="${prefix}" suffix="2" x="0.2"  y="-0.2" z="${height/2}" />
+    <!--
     <xacro:handle prefix="${prefix}" suffix="3" x="-0.2" y="-0.2" z="${height/2}" />
-    <xacro:handle prefix="${prefix}" suffix="4" x="-0.2" y="0.2"  z="${height/2}" />
+    <xacro:handle prefix="${prefix}" suffix="4" x="-0.2" y="0.2"  z="${height/2}" /> -->
   </xacro:macro>
 </robot>

File: urdf/uav_cable_assembly.urdf.xacro (robot description, xacro)
@@ -18,15 +18,20 @@
       radius="${radius}"
       mass="${mass}" />
-    <link name="${prefix}hook_link">
-      <inertial>
-        <mass value="0.01"/>
-        <inertia ixx="1e-8" ixy="0" ixz="0" iyy="1e-8" iyz="0" izz="1e-8"/>
-      </inertial>
-    </link>
-    <joint name="${prefix}cable_to_hook_joint" type="fixed">
-      <parent link="${prefix}link_${segments}"/>
-      <child link="${prefix}hook_link"/>
-      <origin xyz="0 0 ${-length/segments}" rpy="0 0 0"/>
-    </joint>
+  <link name="${prefix}hook_link">
+    <inertial>
+      <mass value="0.01"/>
+      <inertia ixx="1e-6" ixy="0" ixz="0" iyy="1e-6" iyz="0" izz="1e-6"/>
+    </inertial>
+    <visual>
+      <geometry><sphere radius="0.005"/></geometry>
+      <material name="red"/>
+    </visual>
+  </link>
+  <joint name="${prefix}cable_to_hook_joint" type="revolute">
+    <parent link="${prefix}link_${segments}"/>
+    <child link="${prefix}hook_link"/>
+    <origin xyz="0 0 ${-length/segments}" rpy="0 0 0"/>
+    <limit effort="0" lower="0" upper="0" velocity="0"/>
+  </joint>
     <xacro:if value="${attach_to_panel}">
       <joint name="${prefix}hook_to_panel_joint" type="continuous">
@@ -48,8 +53,11 @@
     <xacro:unless value="${primary}">
       <gazebo>
-        <joint name="drone${id}_loop_closure" type="fixed">
-          <parent>main_panel_handle_${handle_id}</parent>
-          <child>drone${id}_hook_link</child>
-        </joint>
+        <plugin filename="gz-sim-detachable-joint-system" name="gz::sim::systems::DetachableJoint">
+          <parent_link>drone${id}_hook_link</parent_link>
+          <child_model>acts_system</child_model>
+          <child_link>main_panel_handle_${handle_id}</child_link>
+          <attach_topic>/drone${id}/attach</attach_topic>
+          <detach_topic>/drone${id}/detach</detach_topic>
+        </plugin>
       </gazebo>
     </xacro:unless>

Commit message: Inverted tree structure panel is the parent

File: urdf/acts.urdf.xacro (robot description, xacro)
@@ -7,7 +7,9 @@
     prefix="main_panel_"
     mass="2.5" width="2.0" depth="2.0" height="0.2" />
-  <xacro:add_drone id="1" x="0"  y="1"  z="1.2" segments="10" length="1" primary="true" />
-  <xacro:add_drone id="2" x="0"  y="0" z="1.2" segments="10"  length="1" handle_id="2" />
-  <!--<xacro:add_drone id="3" x="1" y="3" z="1.2" segments="10"  length="1" handle_id="3" />
-  <xacro:add_drone id="4" x="2" y="3"  z="1.2" segments="10"  length="1" handle_id="4" /> -->
+  <joint name="world_to_panel_joint" type="fixed">
+    <parent link="world"/>
+    <child link="main_panel_base_link"/>
+    <origin xyz="0 0 0" rpy="0 0 0"/> </joint>
+  <xacro:add_drone id="1" handle_id="1" segments="10" length="1.0" />
+  <xacro:add_drone id="2" handle_id="2" segments="10" length="1.0" />
 </robot>

File: urdf/panel.urdf.xacro (robot description, xacro)
@@ -33,5 +33,5 @@
       </collision>
     </link>
-    <xacro:handle prefix="${prefix}" suffix="1" x="1"  y="1"  z="${height/2}" />
+    <xacro:handle prefix="${prefix}" suffix="1" x="0"  y="0"  z="${height/2}" />
     <xacro:handle prefix="${prefix}" suffix="2" x="0.2"  y="-0.2" z="${height/2}" />
     <!--

File: urdf/uav_cable_assembly.urdf.xacro (robot description, xacro)
@@ -3,63 +3,29 @@
   <xacro:include filename="$(find acts_simulator)/urdf/crazy2fly.urdf.xacro" />
   <xacro:include filename="$(find acts_simulator)/urdf/components/cable_component.xacro" />
-  <xacro:macro name="uav_towing_unit" params="prefix panel_link x y z segments length radius mass attach_to_panel">
-    <joint name="world_to_${prefix}_joint" type="fixed">
-      <parent link="world"/>
-      <child link="${prefix}base_link"/>
-      <origin xyz="${x} ${y} ${z}" rpy="0 0 0"/>
-    </joint>
-    <xacro:crazy2fly prefix="${prefix}" />
-    <xacro:uav_cable
-      prefix="${prefix}"
-      parent_link="${prefix}base_link"
-      is_flexible="true"
-      segments="${segments}"
-      length="${length}"
-      radius="${radius}"
-      mass="${mass}" />
+<xacro:macro name="add_drone" params="id handle_id segments length">
+  <xacro:property name="prefix" value="drone${id}_" />
+  <joint name="${prefix}attachment_joint" type="continuous">
+    <parent link="main_panel_handle_${handle_id}"/>
+    <child link="${prefix}hook_link"/>
+    <axis xyz="1 0 0"/>
+    <origin xyz="0 0 0" rpy="0 0 0"/>
+  </joint>
   <link name="${prefix}hook_link">
-    <inertial>
-      <mass value="0.01"/>
-      <inertia ixx="1e-6" ixy="0" ixz="0" iyy="1e-6" iyz="0" izz="1e-6"/>
-    </inertial>
-    <visual>
-      <geometry><sphere radius="0.005"/></geometry>
-      <material name="red"/>
-    </visual>
+    <inertial><mass value="0.01"/><inertia ixx="1e-6" iyy="1e-6" izz="1e-6" ixy="0" ixz="0" iyz="0"/></inertial>
+    <visual><geometry><sphere radius="0.01"/></geometry></visual>
   </link>
-  <joint name="${prefix}cable_to_hook_joint" type="revolute">
+  <xacro:uav_cable
+    prefix="${prefix}"
+    parent_link="${prefix}hook_link"
+    is_flexible="true"
+    segments="${segments}"
+    length="${length}"
+    radius="0.01" mass="0.1" />
+  <xacro:crazy2fly prefix="${prefix}" />
+  <joint name="${prefix}cable_to_uav_joint" type="fixed">
     <parent link="${prefix}link_${segments}"/>
-    <child link="${prefix}hook_link"/>
-    <origin xyz="0 0 ${-length/segments}" rpy="0 0 0"/>
-    <limit effort="0" lower="0" upper="0" velocity="0"/>
+    <child link="${prefix}base_link"/>
+    <origin xyz="0 0 0" rpy="0 0 0"/>
   </joint>
-    <xacro:if value="${attach_to_panel}">
-      <joint name="${prefix}hook_to_panel_joint" type="continuous">
-        <parent link="${prefix}hook_link"/>
-        <child link="${panel_link}"/>
-        <axis xyz="1 0 0"/>
-        <origin xyz="0 0 -0.1" rpy="0 0 0"/>
-      </joint>
-    </xacro:if>
-  </xacro:macro>
-  <xacro:macro name="add_drone" params="id x y z segments length handle_id:=1 primary:=false">
-    <xacro:uav_towing_unit
-      prefix="drone${id}_"
-      panel_link="main_panel_base_link"
-      x="${x}" y="${y}" z="${z}"
-      segments="${segments}"
-      length="${length}" radius="0.01" mass="0.1"
-      attach_to_panel="${primary}" />
-    <xacro:unless value="${primary}">
-      <gazebo>
-        <plugin filename="gz-sim-detachable-joint-system" name="gz::sim::systems::DetachableJoint">
-          <parent_link>drone${id}_hook_link</parent_link>
-          <child_model>acts_system</child_model>
-          <child_link>main_panel_handle_${handle_id}</child_link>
-          <attach_topic>/drone${id}/attach</attach_topic>
-          <detach_topic>/drone${id}/detach</detach_topic>
-        </plugin>
-      </gazebo>
-    </xacro:unless>
-  </xacro:macro>
+</xacro:macro>
 </robot>

Commit message: simplified tree structure

File: urdf/acts.urdf.xacro (robot description, xacro)
@@ -4,12 +4,13 @@
   <xacro:include filename="uav_cable_assembly.urdf.xacro" />
   <link name="world"/>
+  <joint name="world_to_panel_joint" type="fixed">
+    <parent link="world"/>
+    <child link="main_panel_base_link"/>
+    <origin xyz="0 0 2.0" rpy="0 0 0"/>
+  </joint>
   <xacro:panel_platform
     prefix="main_panel_"
     mass="2.5" width="2.0" depth="2.0" height="0.2" />
-  <joint name="world_to_panel_joint" type="fixed">
-    <parent link="world"/>
-    <child link="main_panel_base_link"/>
-    <origin xyz="0 0 0" rpy="0 0 0"/> </joint>
-  <xacro:add_drone id="1" handle_id="1" segments="10" length="1.0" />
-  <xacro:add_drone id="2" handle_id="2" segments="10" length="1.0" />
+  <xacro:add_drone id="1" handle_id="1" segments="30" length="1.0" panel_link="main_panel_base_link"/>
+  <xacro:add_drone id="2" handle_id="2" segments="30" length="1.0" panel_link="main_panel_base_link"/>
 </robot>

File: urdf/components/cable_component.xacro (robot description, xacro)
@@ -41,5 +41,5 @@
       <origin xyz="0 0 0" rpy="0 0 0"/> </xacro:if>
     <xacro:unless value="${current_num == 1}">
-      <origin xyz="0 0 ${-cable_len}" rpy="0 0 0"/>
+      <origin xyz="0 0 ${cable_len}" rpy="0 0 0"/>
     </xacro:unless>
     <axis xyz="1 0 0"/>
@@ -49,9 +49,9 @@
     <xacro:cylinder_inertia m="${m}" r="${rad}" h="${cable_len}" />
     <visual>
-      <origin xyz="0 0 ${-cable_len/2.0}"/>
+      <origin xyz="0 0 ${cable_len/2.0}"/>
       <geometry><cylinder radius="${rad}" length="${cable_len}"/></geometry>
     </visual>
     <collision>
-      <origin xyz="0 0 ${-cable_len/2.0}"/>
+      <origin xyz="0 0 ${cable_len/2.0}"/>
       <geometry><cylinder radius="${rad}" length="${cable_len}"/></geometry>
     </collision>

File: urdf/uav_cable_assembly.urdf.xacro (robot description, xacro)
@@ -3,28 +3,18 @@
   <xacro:include filename="$(find acts_simulator)/urdf/crazy2fly.urdf.xacro" />
   <xacro:include filename="$(find acts_simulator)/urdf/components/cable_component.xacro" />
-<xacro:macro name="add_drone" params="id handle_id segments length">
+<xacro:macro name="add_drone" params="id handle_id segments length panel_link">
   <xacro:property name="prefix" value="drone${id}_" />
-  <joint name="${prefix}attachment_joint" type="continuous">
-    <parent link="main_panel_handle_${handle_id}"/>
-    <child link="${prefix}hook_link"/>
-    <axis xyz="1 0 0"/>
-    <origin xyz="0 0 0" rpy="0 0 0"/>
-  </joint>
-  <link name="${prefix}hook_link">
-    <inertial><mass value="0.01"/><inertia ixx="1e-6" iyy="1e-6" izz="1e-6" ixy="0" ixz="0" iyz="0"/></inertial>
-    <visual><geometry><sphere radius="0.01"/></geometry></visual>
-  </link>
+  <xacro:crazy2fly prefix="${prefix}" />
   <xacro:uav_cable
     prefix="${prefix}"
-    parent_link="${prefix}hook_link"
+    parent_link="${panel_link}"
     is_flexible="true"
     segments="${segments}"
     length="${length}"
-    radius="0.01" mass="0.1" />
-  <xacro:crazy2fly prefix="${prefix}" />
-  <joint name="${prefix}cable_to_uav_joint" type="fixed">
+    radius="0.01" mass="0001" />
+  <joint name="${prefix}cable_to_drone_joint" type="fixed">
     <parent link="${prefix}link_${segments}"/>
     <child link="${prefix}base_link"/>
-    <origin xyz="0 0 0" rpy="0 0 0"/>
+    <origin xyz="0 0 ${length/segments}" rpy="0 0 0"/>
   </joint>
 </xacro:macro>
