Commit message: drone is able to fly but not change position

File: urdf/acts.urdf.xacro (robot description, xacro)
@@ -7,10 +7,54 @@
     <parent link="world"/>
     <child link="main_panel_base_link"/>
-    <origin xyz="0 0 2.0" rpy="0 0 0"/>
+    <origin xyz="0 0 0.0" rpy="0 0 0"/>
   </joint>
   <xacro:panel_platform
     prefix="main_panel_"
-    mass="2.5" width="2.0" depth="2.0" height="0.2" />
-  <xacro:add_drone id="1" handle_id="1" segments="30" length="1.0" panel_link="main_panel_base_link"/>
-  <xacro:add_drone id="2" handle_id="2" segments="30" length="1.0" panel_link="main_panel_base_link"/>
+    mass="100.0" width="3.0" depth="3.0" height="0.2" />
+  <xacro:add_drone
+    id="1"
+    segments="10"
+    length="1.0"
+    panel_link="main_panel_base_link"
+    x_off="0.0"
+    y_off="0.0"
+    z_off="0.1"/>
+  <gazebo>
+    <self_collide>true</self_collide>
+  </gazebo>
+  <gazebo reference="drone1_base_link">
+    <self_collide>true</self_collide>
+    <collision name="drone1_total_collision">
+      <geometry>
+        <box size="0.3 0.3 0.1"/>
+      </geometry>
+      <surface>
+        <contact>
+          <collide_bitmask>0x01</collide_bitmask>
+        </contact>
+        <friction>
+          <ode>
+            <mu>1.0</mu>
+            <mu2>1.0</mu2>
+          </ode>
+        </friction>
+      </surface>
+    </collision>
+  </gazebo>
+  <gazebo reference="main_panel_base_link">
+    <collision name="panel_surface_collision">
+      <geometry>
+        <box size="3.0 3.0 0.2"/>
+      </geometry>
+      <surface>
+        <contact>
+          <collide_bitmask>0x01</collide_bitmask>
+        </contact>
+      </surface>
+    </collision>
+  </gazebo>
+  <gazebo reference="drone1_cable_to_drone_joint">
+    <preserveFixedJoint>true</preserveFixedJoint>
+    <disableFixedJointLumping>true</disableFixedJointLumping>
+  </gazebo>
 </robot>

File: urdf/crazy2fly.urdf.xacro (robot description, xacro)
@@ -38,5 +38,21 @@
 	<xacro:macro name="crazy2fly" params="prefix">
 	<!-- BASE LINK -->
-	<link name="${prefix}base_link" />
+	<link name="${prefix}base_link">
+		<inertial>
+			<mass value="1.0" />
+			<origin xyz="0 0 0" rpy="0 0 0" />
+			<inertia ixx="0.01" ixy="0" ixz="0" iyy="0.01" iyz="0" izz="0.02" />
+		</inertial>
+		<visual>
+			<geometry>
+			<box size="0.2 0.2 0.1"/>
+			</geometry>
+		</visual>
+		<collision name="${prefix}base_collision">
+			<geometry>
+			<box size="0.3 0.3 0.15"/>
+			</geometry>
+		</collision>
+	</link>
 	<!-- CORE -->
 	<xacro:core parent_link="${prefix}base_link" prefix="${prefix}">

File: urdf/panel.urdf.xacro (robot description, xacro)
@@ -29,13 +29,20 @@
         <material name="grey"><color rgba="0.5 0.5 0.5 1"/></material>
       </visual>
-      <collision>
-        <geometry><box size="${width} ${depth} ${height}"/></geometry>
+      <collision name="panel_collision">
+        <origin xyz="0 0 0" rpy="0 0 0"/>
+        <geometry> <box size="${width} ${depth} ${height}"/> </geometry>
       </collision>
     </link>
     <xacro:handle prefix="${prefix}" suffix="1" x="0"  y="0"  z="${height/2}" />
-    <xacro:handle prefix="${prefix}" suffix="2" x="0.2"  y="-0.2" z="${height/2}" />
+    <!-- <xacro:handle prefix="${prefix}" suffix="2" x="1"  y="1" z="${height/2}" /> -->
     <!--
     <xacro:handle prefix="${prefix}" suffix="3" x="-0.2" y="-0.2" z="${height/2}" />
     <xacro:handle prefix="${prefix}" suffix="4" x="-0.2" y="0.2"  z="${height/2}" /> -->
+  <gazebo reference="main_panel_base_link">
+    <mu1>1.0</mu1>
+    <mu2>1.0</mu2>
+    <self_collide>true</self_collide>
+    <kp>1000000.0</kp> <kd>1.0</kd>
+  </gazebo>
   </xacro:macro>
 </robot>

File: urdf/uav_cable_assembly.urdf.xacro (robot description, xacro)
@@ -3,19 +3,26 @@
   <xacro:include filename="$(find acts_simulator)/urdf/crazy2fly.urdf.xacro" />
   <xacro:include filename="$(find acts_simulator)/urdf/components/cable_component.xacro" />
-<xacro:macro name="add_drone" params="id handle_id segments length panel_link">
-  <xacro:property name="prefix" value="drone${id}_" />
-  <xacro:crazy2fly prefix="${prefix}" />
-  <xacro:uav_cable
-    prefix="${prefix}"
-    parent_link="${panel_link}"
-    is_flexible="true"
-    segments="${segments}"
-    length="${length}"
-    radius="0.01" mass="0001" />
-  <joint name="${prefix}cable_to_drone_joint" type="fixed">
-    <parent link="${prefix}link_${segments}"/>
-    <child link="${prefix}base_link"/>
-    <origin xyz="0 0 ${length/segments}" rpy="0 0 0"/>
-  </joint>
-</xacro:macro>
+  <xacro:macro name="add_drone" params="id segments length panel_link x_off y_off z_off">
+    <xacro:property name="prefix" value="drone${id}_" />
+    <xacro:crazy2fly prefix="${prefix}" />
+    <xacro:uav_cable
+      prefix="${prefix}"
+      parent_link="${panel_link}"
+      is_flexible="true"
+      segments="${segments}"
+      length="${length}"
+      radius="0.005" mass="0.01" />
+    <joint name="${prefix}cable_to_drone_joint" type="fixed">
+      <parent link="${prefix}link_${segments}"/>
+      <child link="${prefix}base_link"/>
+      <origin xyz="${x_off} ${y_off} ${float(z_off)}" rpy="0 0 0"/>
+    </joint>
+    <gazebo reference="${prefix}cable_to_drone_joint">
+      <preserveFixedJoint>true</preserveFixedJoint>
+      <disableFixedJointLumping>true</disableFixedJointLumping>
+    </gazebo>
+    <gazebo reference="${prefix}base_link">
+      <self_collide>true</self_collide>
+    </gazebo>
+  </xacro:macro>
 </robot>

Commit message: One drone able to fly and move the platform

File: urdf/acts.urdf.xacro (robot description, xacro)
@@ -3,13 +3,7 @@
   <xacro:include filename="panel.urdf.xacro" />
   <xacro:include filename="uav_cable_assembly.urdf.xacro" />
-  <link name="world"/>
-  <joint name="world_to_panel_joint" type="fixed">
-    <parent link="world"/>
-    <child link="main_panel_base_link"/>
-    <origin xyz="0 0 0.0" rpy="0 0 0"/>
-  </joint>
   <xacro:panel_platform
     prefix="main_panel_"
-    mass="100.0" width="3.0" depth="3.0" height="0.2" />
+    mass="10.0" width="3.0" depth="3.0" height="0.2" />
   <xacro:add_drone
     id="1"
@@ -23,38 +17,3 @@
     <self_collide>true</self_collide>
   </gazebo>
-  <gazebo reference="drone1_base_link">
-    <self_collide>true</self_collide>
-    <collision name="drone1_total_collision">
-      <geometry>
-        <box size="0.3 0.3 0.1"/>
-      </geometry>
-      <surface>
-        <contact>
-          <collide_bitmask>0x01</collide_bitmask>
-        </contact>
-        <friction>
-          <ode>
-            <mu>1.0</mu>
-            <mu2>1.0</mu2>
-          </ode>
-        </friction>
-      </surface>
-    </collision>
-  </gazebo>
-  <gazebo reference="main_panel_base_link">
-    <collision name="panel_surface_collision">
-      <geometry>
-        <box size="3.0 3.0 0.2"/>
-      </geometry>
-      <surface>
-        <contact>
-          <collide_bitmask>0x01</collide_bitmask>
-        </contact>
-      </surface>
-    </collision>
-  </gazebo>
-  <gazebo reference="drone1_cable_to_drone_joint">
-    <preserveFixedJoint>true</preserveFixedJoint>
-    <disableFixedJointLumping>true</disableFixedJointLumping>
-  </gazebo>
 </robot>

File: urdf/components/cable_component.xacro (robot description, xacro)
@@ -32,5 +32,6 @@
   <link name="${prefix}virtual_${current_num}">
     <inertial>
-      <mass value="0.0001"/> <inertia ixx="1e-8" ixy="0" ixz="0" iyy="1e-8" iyz="0" izz="1e-8"/>
+      <mass value="0.0001"/>
+      <inertia ixx="1e-6" ixy="0" ixz="0" iyy="1e-6" iyz="0" izz="1e-6"/>
     </inertial>
   </link>
@@ -38,11 +39,7 @@
     <parent link="${parent}"/>
     <child link="${prefix}virtual_${current_num}"/>
-    <xacro:if value="${current_num == 1}">
-      <origin xyz="0 0 0" rpy="0 0 0"/> </xacro:if>
-    <xacro:unless value="${current_num == 1}">
-      <origin xyz="0 0 ${cable_len}" rpy="0 0 0"/>
-    </xacro:unless>
+    <origin xyz="0 0 ${current_num == 1 and 0 or cable_len}" rpy="0 0 0"/>
     <axis xyz="1 0 0"/>
-    <dynamics damping="0.01" friction="0.001"/>
+    <dynamics damping="0.05" friction="0.01"/>
   </joint>
   <link name="${prefix}link_${current_num}">
@@ -52,17 +49,17 @@
       <geometry><cylinder radius="${rad}" length="${cable_len}"/></geometry>
     </visual>
-    <collision>
-      <origin xyz="0 0 ${cable_len/2.0}"/>
-      <geometry><cylinder radius="${rad}" length="${cable_len}"/></geometry>
-    </collision>
-    <self_collide>false</self_collide>
-  </link>
+    </link>
   <joint name="${prefix}joint_y_${current_num}" type="continuous">
     <parent link="${prefix}virtual_${current_num}"/>
     <child link="${prefix}link_${current_num}"/>
-    <origin xyz="0 0 0" rpy="0 0 0"/>
     <axis xyz="0 1 0"/>
-    <dynamics damping="0.01" friction="0.001"/>
+    <dynamics damping="0.05" friction="0.01"/>
   </joint>
+  <gazebo reference="${prefix}joint_x_${current_num}">
+    <implicitSpringDamper>true</implicitSpringDamper>
+  </gazebo>
+  <gazebo reference="${prefix}joint_y_${current_num}">
+    <implicitSpringDamper>true</implicitSpringDamper>
+  </gazebo>
   <xacro:if value="${current_num &lt; total_num}">
     <xacro:flexible_chain_generator

File: urdf/crazy2fly.urdf.xacro (robot description, xacro)
@@ -1,4 +1,5 @@
 <?xml version="1.0" encoding="utf-8"?>
 <!--
+This files has been modified starting from:
 File: crazy2fly.urdf.xacro
 Project: Quadrotor Control Lab
@@ -44,9 +45,9 @@
 			<inertia ixx="0.01" ixy="0" ixz="0" iyy="0.01" iyz="0" izz="0.02" />
 		</inertial>
-		<visual>
+		<!-- <visual>
 			<geometry>
 			<box size="0.2 0.2 0.1"/>
 			</geometry>
-		</visual>
+		</visual> -->
 		<collision name="${prefix}base_collision">
 			<geometry>

File: urdf/panel.urdf.xacro (robot description, xacro)
@@ -34,4 +34,8 @@
       </collision>
     </link>
+    <gazebo reference="${prefix}base_link">
+      <static>false</static>
+      <self_collide>true</self_collide>
+    </gazebo>
     <xacro:handle prefix="${prefix}" suffix="1" x="0"  y="0"  z="${height/2}" />
     <!-- <xacro:handle prefix="${prefix}" suffix="2" x="1"  y="1" z="${height/2}" /> -->
@@ -39,10 +43,4 @@
     <xacro:handle prefix="${prefix}" suffix="3" x="-0.2" y="-0.2" z="${height/2}" />
     <xacro:handle prefix="${prefix}" suffix="4" x="-0.2" y="0.2"  z="${height/2}" /> -->
-  <gazebo reference="main_panel_base_link">
-    <mu1>1.0</mu1>
-    <mu2>1.0</mu2>
-    <self_collide>true</self_collide>
-    <kp>1000000.0</kp> <kd>1.0</kd>
-  </gazebo>
   </xacro:macro>
 </robot>

File: urdf/uav_cable_assembly.urdf.xacro (robot description, xacro)
@@ -18,11 +18,4 @@
       <origin xyz="${x_off} ${y_off} ${float(z_off)}" rpy="0 0 0"/>
     </joint>
-    <gazebo reference="${prefix}cable_to_drone_joint">
-      <preserveFixedJoint>true</preserveFixedJoint>
-      <disableFixedJointLumping>true</disableFixedJointLumping>
-    </gazebo>
-    <gazebo reference="${prefix}base_link">
-      <self_collide>true</self_collide>
-    </gazebo>
   </xacro:macro>
 </robot>

Commit message: minor changes on uav controller

File: urdf/acts.urdf.xacro (robot description, xacro)
@@ -5,5 +5,5 @@
   <xacro:panel_platform
     prefix="main_panel_"
-    mass="10.0" width="3.0" depth="3.0" height="0.2" />
+    mass="0.1" width="3.0" depth="3.0" height="0.2" />
   <xacro:add_drone
     id="1"

File: urdf/components/ugv_component.xacro (robot description, xacro)
@@ -1,5 +1,5 @@
 <?xml version="1.0"?>
 <robot xmlns:xacro="http://www.ros.org/wiki/xacro">
-  <xacro:macro name="ugv_platform" params="prefix">
+  <xacro:macro name="ugv_component" params="prefix x y z">
     <link name="${prefix}base_link">
       <inertial>
@@ -8,15 +8,13 @@
       </inertial>
       <visual>
-        <geometry>
-          <box size="0.5 0.5 0.2"/> </geometry>
-        <material name="blue">
-            <color rgba="0 0 1 1"/>
-        </material>
+        <origin xyz="${x} ${y} ${z}" rpy="0 0 0"/>
+        <geometry><box size="0.5 0.5 0.2"/></geometry>
+        <material name="blue"><color rgba="0 0 1 1"/></material>
       </visual>
-      <collision>
+      <!-- <collision>
         <geometry>
           <box size="0.5 0.5 0.2"/>
         </geometry>
-      </collision>
+      </collision> -->
     </link>
   </xacro:macro>

Commit message: Minor fixes

File: urdf/acts.urdf.xacro (robot description, xacro)
@@ -5,5 +5,5 @@
   <xacro:panel_platform
     prefix="main_panel_"
-    mass="0.1" width="3.0" depth="3.0" height="0.2" />
+    mass="0.0001" width="3.0" depth="3.0" height="0.2" />
   <xacro:add_drone
     id="1"
@@ -13,5 +13,5 @@
     x_off="0.0"
     y_off="0.0"
-    z_off="0.1"/>
+    z_off="0.0"/>
   <gazebo>
     <self_collide>true</self_collide>

File: urdf/components/cable_component.xacro (robot description, xacro)
@@ -46,5 +46,5 @@
     <xacro:cylinder_inertia m="${m}" r="${rad}" h="${cable_len}" />
     <visual>
-      <origin xyz="0 0 ${cable_len/2.0}"/>
+      <origin xyz="0 0 ${-cable_len/2.0}"/>
       <geometry><cylinder radius="${rad}" length="${cable_len}"/></geometry>
     </visual>

Commit message: Payload motion with one drone working, but oscillates at point reached

File: urdf/acts.urdf.xacro (robot description, xacro)
@@ -5,10 +5,12 @@
   <xacro:panel_platform
     prefix="main_panel_"
-    mass="0.0001" width="3.0" depth="3.0" height="0.2" />
+    mass="0.001"
+    radius="0.5"
+    height="0.2" />
   <xacro:add_drone
     id="1"
     segments="10"
     length="1.0"
-    panel_link="main_panel_base_link"
+    panel_link="main_panel_handle_1"
     x_off="0.0"
     y_off="0.0"

File: urdf/components/cable_component.xacro (robot description, xacro)
@@ -8,23 +8,4 @@
                izz="${(m/2) * (r*r)}"/>
     </inertial>
-  </xacro:macro>
-<!-- ____________   Rigid cable  _______________________-->
-  <xacro:macro name="rigid_cable" params="prefix parent_link length radius mass">
-    <link name="${prefix}rigid_link">
-      <xacro:cylinder_inertia m="${mass}" r="${radius}" h="${length}" />
-      <visual>
-        <origin xyz="0 0 ${-length/2.0}"/>
-        <geometry><cylinder radius="${radius}" length="${length}"/></geometry>
-      </visual>
-      <collision>
-        <origin xyz="0 0 ${-length/2.0}"/>
-        <geometry><cylinder radius="${radius}" length="${length}"/></geometry>
-      </collision>
-    </link>
-    <joint name="${prefix}rigid_joint" type="universal">
-      <parent link="${parent_link}"/>
-      <child link="${prefix}rigid_link"/>
-      <origin xyz="0 0 -0.05" rpy="0 0 0"/>
-    </joint>
   </xacro:macro>
 <!-- ____________   Flexible cable  _______________________-->
@@ -79,6 +60,7 @@
     </xacro:if>
     <xacro:unless value="${is_flexible}">
-      <xacro:rigid_cable prefix="${prefix}" parent_link="${parent_link}"
-        length="${length}" radius="${radius}" mass="${mass}" />
+      <xacro:flexible_chain_generator
+      prefix="${prefix}" parent="${parent_link}" current_num="1"
+      total_num="1" cable_len="${length}" rad="${radius}" m="${mass}" />
     </xacro:unless>
   </xacro:macro>

File: urdf/panel.urdf.xacro (robot description, xacro)
@@ -1,4 +1,5 @@
 <?xml version="1.0"?>
 <robot xmlns:xacro="http://www.ros.org/wiki/xacro">
+    <xacro:include filename="$(find acts_simulator)/urdf/components/cable_component.xacro" />
   <xacro:macro name="panel_box_inertia" params="m w d h">
     <inertial>
@@ -8,34 +9,49 @@
                izz="${(m/12) * (w*w + d*d)}"/>
     </inertial>
-  </xacro:macro>
-  <xacro:macro name="handle" params="prefix suffix x y z">
-    <link name="${prefix}handle_${suffix}">
-      <inertial>
-        <mass value="0.001"/>
-        <inertia ixx="1e-9" ixy="0" ixz="0" iyy="1e-9" iyz="0" izz="1e-9"/>
-      </inertial>
-    </link>
-    <joint name="${prefix}handle_${suffix}_joint" type="fixed">
-      <parent link="${prefix}base_link"/>
-      <child link="${prefix}handle_${suffix}"/>
-      <origin xyz="${x} ${y} ${z}" rpy="0 0 0"/>
-    </joint>
-  </xacro:macro>
-  <xacro:macro name="panel_platform" params="prefix mass width depth height">
-    <link name="${prefix}base_link">
-      <xacro:panel_box_inertia m="${mass}" w="${width}" d="${depth}" h="${height}" />
-      <visual>
-        <geometry><box size="${width} ${depth} ${height}"/></geometry>
-        <material name="grey"><color rgba="0.5 0.5 0.5 1"/></material>
-      </visual>
-      <collision name="panel_collision">
-        <origin xyz="0 0 0" rpy="0 0 0"/>
-        <geometry> <box size="${width} ${depth} ${height}"/> </geometry>
-      </collision>
-    </link>
-    <gazebo reference="${prefix}base_link">
-      <static>false</static>
-      <self_collide>true</self_collide>
-    </gazebo>
+    </xacro:macro>
+  <xacro:macro name="panel_cylinder_inertia" params="m r h">
+        <inertial>
+            <mass value="${m}"/>
+            <inertia ixx="${(m/12) * (3*r*r + h*h)}" ixy="0.0" ixz="0.0"
+                     iyy="${(m/12) * (3*r*r + h*h)}" iyz="0.0"
+                     izz="${(m/2) * (r*r)}"/>
+    </inertial>
+    </xacro:macro>
+    <xacro:macro name="handle" params="prefix suffix x y z">
+      <!-- Handle sits on top of link_1 — drone cable attaches here  -->
+        <link name="${prefix}handle_${suffix}">
+            <inertial>
+                <mass value="0.0001"/>
+                <inertia ixx="1e-9" ixy="0" ixz="0" iyy="1e-9" iyz="0" izz="1e-9"/>
+            </inertial>
+        </link>
+        <joint name="${prefix}handle_${suffix}_joint" type="fixed">
+            <parent link="${prefix}link_1"/>
+            <child link="${prefix}handle_${suffix}"/>
+            <origin xyz="${x} ${y} ${z}" rpy="0 0 0"/>
+        </joint>
+    </xacro:macro>
+    <xacro:macro name="panel_platform" params="prefix mass radius height">
+        <!-- Free-floating root — exactly like PDF1's main_panel_cable_root_link -->
+        <link name="${prefix}cable_root_link">
+            <inertial>
+                <mass value="0.0001"/>
+                <inertia ixx="1e-6" ixy="0" ixz="0" iyy="1e-6" iyz="0" izz="1e-6"/>
+            </inertial>
+        </link>
+        <!-- Panel body as a single cable segment — gives it the flexible joint -->
+        <xacro:uav_cable
+            prefix="${prefix}"
+            parent_link="${prefix}cable_root_link"
+            is_flexible="true"
+            segments="1"
+            length="${height}"
+            radius="${radius}"
+            mass="${mass}" />
+        <!-- link_1 is now the panel body, add visual/collision to it -->
+        <gazebo reference="${prefix}link_1">
+            <static>false</static>
+            <self_collide>true</self_collide>
+        </gazebo>
     <xacro:handle prefix="${prefix}" suffix="1" x="0"  y="0"  z="${height/2}" />
     <!-- <xacro:handle prefix="${prefix}" suffix="2" x="1"  y="1" z="${height/2}" /> -->

File: urdf/uav_cable_assembly.urdf.xacro (robot description, xacro)
@@ -6,6 +6,4 @@
     <xacro:property name="prefix" value="drone${id}_" />
     <xacro:crazy2fly prefix="${prefix}" />
-    <!-- When no panel_link, create a free-floating root link for the cable top -->
-    <xacro:if value="${panel_link == ''}">
         <link name="${prefix}cable_root_link">
             <inertial>
@@ -14,22 +12,26 @@
             </inertial>
         </link>
-        <xacro:property name="cable_parent" value="${prefix}cable_root_link" />
-    </xacro:if>
+        <!-- If panel provided, attach panel to cable root -->
     <xacro:unless value="${panel_link == ''}">
-        <xacro:property name="cable_parent" value="${panel_link}" />
+        <joint name="${prefix}panel_to_cable_joint" type="fixed">
+            <parent link="${panel_link}"/>
+            <child link="${prefix}cable_root_link"/>
+            <origin xyz="${x_off} ${y_off} ${float(z_off)}" rpy="0 0 0"/>
+        </joint>
     </xacro:unless>
+    <!-- Cable hangs from cable_root_link -->
     <xacro:uav_cable
         prefix="${prefix}"
-        parent_link="${cable_parent}"
+        parent_link="${prefix}cable_root_link"
         is_flexible="true"
         segments="${segments}"
         length="${length}"
         radius="0.005" mass="0.01" />
-    <!-- Cable tip attaches to drone base -->
+    <!-- Drone is child of cable tip link_${segments} -->
     <joint name="${prefix}cable_to_drone_joint" type="fixed">
         <parent link="${prefix}link_${segments}"/>
         <child link="${prefix}base_link"/>
-        <origin xyz="${x_off} ${y_off} ${float(z_off)}" rpy="0 0 0"/>
+        <origin xyz="0 0 0" rpy="0 0 0"/>
     </joint>
-</xacro:macro>
+    </xacro:macro>
 </robot>
