Commit message: Receive drones infos from json file

File: urdf/acts.urdf.xacro (robot description, xacro)
@@ -3,19 +3,32 @@
   <xacro:include filename="panel.urdf.xacro" />
   <xacro:include filename="uav_cable_assembly.urdf.xacro" />
+  <xacro:arg name="drone1_id" default="1"/>
+  <xacro:arg name="drone1_x" default="0.0"/>
+  <xacro:arg name="drone1_y" default="0.0"/>
+  <xacro:arg name="drone1_z" default="0.0"/>
+  <!-- TODO: implement the platform receiving these values -->
+  <xacro:arg name="drone1_attach_x" default="0.0"/>
+  <xacro:arg name="drone1_attach_y" default="0.0"/>
+  <xacro:arg name="drone1_attach_z" default="0.0"/>
+  <xacro:arg name="drone1_panel_link" default="main_panel_handle_1"/>
+  <xacro:arg name="drone1_len" default="1.0"/>
+  <xacro:arg name="drone1_roll" default="0.0"/>
+  <xacro:arg name="drone1_pitch" default="0.0"/>
+  <xacro:arg name="drone1_yaw" default="0.0"/>
   <xacro:panel_platform
-    prefix="main_panel_"
-    mass="0.001"
-    radius="0.5"
-    height="0.2" />
+  prefix="main_panel_"
+  mass="0.001"
+  radius="0.7"
+  height="0.2" />
   <xacro:add_drone
-    id="1"
+    id="$(arg drone1_id)"
     segments="10"
-    length="1.0"
-    panel_link="main_panel_handle_1"
-    x_off="0.0"
-    y_off="0.0"
-    z_off="0.0"/>
-  <gazebo>
-    <self_collide>true</self_collide>
-  </gazebo>
-</robot>
+    length="$(arg drone1_len)"
+    panel_link="$(arg drone1_panel_link)"
+    x_off="$(arg drone1_x)"
+    y_off="$(arg drone1_y)"
+    z_off="$(arg drone1_z)"
+    cable_roll="$(arg drone1_roll)"
+    cable_pitch="$(arg drone1_pitch)"
+    cable_yaw="$(arg drone1_yaw)"/>
+  </robot>

File: urdf/components/ugv_component.xacro (robot description, xacro)
@@ -9,5 +9,5 @@
       <visual>
         <origin xyz="${x} ${y} ${z}" rpy="0 0 0"/>
-        <geometry><box size="0.5 0.5 0.2"/></geometry>
+        <geometry><box size="0.2 0.2 0.2"/></geometry>
         <material name="blue"><color rgba="0 0 1 1"/></material>
       </visual>

File: urdf/crazy2fly.urdf.xacro (robot description, xacro)
@@ -90,4 +90,8 @@
 		<joint_name>${prefix}right_ccw_propeller_joint</joint_name>
 		<joint_name>${prefix}left_ccw_propeller_joint</joint_name>
+		<!-- <joint_name>${prefix}joint_x_1</joint_name>
+		<joint_name>${prefix}joint_y_1</joint_name>
+		<joint_name>${prefix}joint_x_2</joint_name>
+		<joint_name>${prefix}joint_y_2</joint_name> -->
 	</plugin>
 		<!-- ODOMETRY PUBLISHER -->

File: urdf/panel.urdf.xacro (robot description, xacro)
@@ -54,6 +54,6 @@
             <self_collide>true</self_collide>
         </gazebo>
-    <xacro:handle prefix="${prefix}" suffix="1" x="0"  y="0"  z="${height/2}" />
-    <!-- <xacro:handle prefix="${prefix}" suffix="2" x="1"  y="1" z="${height/2}" /> -->
+    <xacro:handle prefix="${prefix}" suffix="1" x="0"  y="0"  z="0" />
+    <xacro:handle prefix="${prefix}" suffix="2" x="0"  y="0" z="0" />
     <!--
     <xacro:handle prefix="${prefix}" suffix="3" x="-0.2" y="-0.2" z="${height/2}" />

File: urdf/track.xacro (robot description, xacro)
@@ -5,7 +5,7 @@
   <xacro:ugv_component
     prefix="obstacle_"
-    x="1.0"
-    y="1.0"
-    z="5.0"
+    x="2.0"
+    y="2.0"
+    z="2.0"
   />
   <joint name="ref_joint" type="fixed">

File: urdf/uav_cable_assembly.urdf.xacro (robot description, xacro)
@@ -3,5 +3,5 @@
   <xacro:include filename="$(find acts_simulator)/urdf/crazy2fly.urdf.xacro" />
   <xacro:include filename="$(find acts_simulator)/urdf/components/cable_component.xacro" />
-  <xacro:macro name="add_drone" params="id segments length x_off y_off z_off panel_link:=''">
+<xacro:macro name="add_drone" params="id segments length x_off y_off z_off cable_roll:=0 cable_pitch:=0 cable_yaw:=0 panel_link:=''">
     <xacro:property name="prefix" value="drone${id}_" />
     <xacro:crazy2fly prefix="${prefix}" />
