Commit message: UAV connected to the ground working for forces directed along y and z

File: urdf/crazy2fly.urdf.xacro (robot description, xacro)
@@ -90,11 +90,7 @@
 		<joint_name>${prefix}right_ccw_propeller_joint</joint_name>
 		<joint_name>${prefix}left_ccw_propeller_joint</joint_name>
-		<!-- <joint_name>${prefix}joint_x_1</joint_name>
-		<joint_name>${prefix}joint_y_1</joint_name>
-		<joint_name>${prefix}joint_x_2</joint_name>
-		<joint_name>${prefix}joint_y_2</joint_name> -->
 	</plugin>
 		<!-- ODOMETRY PUBLISHER -->
-		<plugin name="gz::sim::systems::OdometryPublisher" filename="gz-sim-odometry-publisher-system">
+		<!-- <plugin name="gz::sim::systems::OdometryPublisher" filename="gz-sim-odometry-publisher-system">
 			<odom_publish_frequency>100</odom_publish_frequency>
 			<dimensions>3</dimensions>
@@ -103,4 +99,15 @@
 			<odom_topic>${ns}${prefix}mocap/odom</odom_topic>
 			<tf_topic>${ns}${prefix}tf</tf_topic>
+		</plugin> -->
+		<plugin filename="gz-sim-pose-publisher-system"
+				name="gz::sim::systems::PosePublisher">
+			<publish_link_pose>true</publish_link_pose>
+			<publish_sensor_pose>false</publish_sensor_pose>
+			<publish_collision_pose>false</publish_collision_pose>
+			<publish_visual_pose>false</publish_visual_pose>
+			<publish_nested_model_pose>false</publish_nested_model_pose>
+			<use_pose_vector_msg>true</use_pose_vector_msg>
+			<static_publisher>false</static_publisher>
+			<publish_frequency>100</publish_frequency>
 		</plugin>
 		<!-- DETACHABLE JOINT -->

File: urdf/uav_cable_assembly.urdf.xacro (robot description, xacro)
@@ -31,5 +31,4 @@
         cable_yaw="${cable_yaw}"
         radius="0.005" mass="0.01" />
-    <!-- Drone is child of cable tip link_${segments} -->
     <joint name="${prefix}cable_to_drone_joint" type="fixed">
         <parent link="${prefix}link_${segments}"/>
@@ -37,4 +36,35 @@
         <origin xyz="0 0 0" rpy="0 0 0"/>
     </joint>
+    <!-- <link name="${prefix}cable_drone_virtual">
+        <inertial>
+            <mass value="0.0001"/>
+            <inertia ixx="1e-6" ixy="0" ixz="0" iyy="1e-6" iyz="0" izz="1e-6"/>
+        </inertial>
+    </link>
+    <joint name="${prefix}cable_to_drone_joint_x" type="continuous">
+        <parent link="${prefix}link_${segments}"/>
+        <child link="${prefix}cable_drone_virtual"/>
+        <origin xyz="0 0 0" rpy="0 0 0"/>
+        <axis xyz="1 0 0"/>
+        <dynamics damping="10.0" friction="0.01"/>
+    </joint>
+    <joint name="${prefix}cable_to_drone_joint_y" type="continuous">
+        <parent link="${prefix}cable_drone_virtual"/>
+        <child link="${prefix}base_link"/>
+        <axis xyz="0 1 0"/>
+        <dynamics damping="10.0" friction="0.01"/>
+    </joint> -->
+    <gazebo reference="${prefix}base_link">
+    <plugin filename="gz-sim-pose-publisher-system" name="gz::sim::systems::PosePublisher">
+        <publish_link_pose>true</publish_link_pose>
+        <publish_sensor_pose>false</publish_sensor_pose>
+        <publish_collision_pose>false</publish_collision_pose>
+        <publish_visual_pose>false</publish_visual_pose>
+        <publish_nested_model_pose>false</publish_nested_model_pose>
+        <use_pose_vector_msg>true</use_pose_vector_msg>
+        <static_publisher>false</static_publisher>
+        <publish_frequency>100</publish_frequency>
+    </plugin>
+</gazebo>
     </xacro:macro>
 </robot>

Commit message: Receiving imu values and correct loading simple.world

File: urdf/crazy2fly.urdf.xacro (robot description, xacro)
@@ -61,5 +61,5 @@
 	</xacro:core>
 	<!-- IMU SENSOR -->
-	<xacro:imu parent_link="${prefix}c2f" drone_prefix="${prefix}" sensor="px4">
+	<xacro:imu parent_link="${prefix}c2f" drone_prefix="${prefix}" sensor="px4" ns="${ns}">
 		<origin xyz="0 0 0.0315" rpy="0 0 0" />
 	</xacro:imu>

File: urdf/sensors/imu.xacro (robot description, xacro)
@@ -15,5 +15,5 @@
 -->
 <robot xmlns:xacro="http://www.ros.org/wiki/xacro">
-	<xacro:macro name="imu" params="parent_link drone_prefix:='' prefix:='' sensor *joint_pose">
+	<xacro:macro name="imu" params="parent_link drone_prefix:='' prefix:='' sensor ns:='' *joint_pose">
 		<xacro:property name="imu_yaml_file" value="${BASE_CONFIG_PATH}/sensors/imu.yaml" />
 		<xacro:property name="props" value="${xacro.load_yaml(imu_yaml_file)}" />
@@ -113,5 +113,5 @@
 					</linear_acceleration>
 				</imu>
-				<topic>${ns}${drone_prefix}${props.topic}</topic>
+				<topic>${drone_prefix}/${props.topic}</topic>
 				<gz_frame_id>${resolved_prefix}_link</gz_frame_id>
 			</sensor>

Commit message: Trying to connect the drone to cable through spherical joint

File: urdf/crazy2fly.urdf.xacro (robot description, xacro)
@@ -91,5 +91,5 @@
 		<joint_name>${prefix}left_ccw_propeller_joint</joint_name>
 	</plugin>
-		<!-- ODOMETRY PUBLISHER -->
+		<!-- ODOMETRY PUBLISHER --> POSITION CONTROL -- TURN IT ON WHEN USING POSITION CONTROL NODE
 		<!-- <plugin name="gz::sim::systems::OdometryPublisher" filename="gz-sim-odometry-publisher-system">
 			<odom_publish_frequency>100</odom_publish_frequency>

File: urdf/uav_cable_assembly.urdf.xacro (robot description, xacro)
@@ -31,28 +31,38 @@
         cable_yaw="${cable_yaw}"
         radius="0.005" mass="0.01" />
-    <joint name="${prefix}cable_to_drone_joint" type="fixed">
-        <parent link="${prefix}link_${segments}"/>
-        <child link="${prefix}base_link"/>
-        <origin xyz="0 0 0" rpy="0 0 0"/>
-    </joint>
-    <!-- <link name="${prefix}cable_drone_virtual">
+    <link name="${prefix}cable_drone_virtualXY">
         <inertial>
-            <mass value="0.0001"/>
-            <inertia ixx="1e-6" ixy="0" ixz="0" iyy="1e-6" iyz="0" izz="1e-6"/>
+            <mass value="0.1"/>
+            <inertia ixx="0.001" ixy="0" ixz="0"
+                 iyy="0.001" iyz="0"
+                 izz="0.001"/>
+        </inertial>
+    </link>
+    <link name="${prefix}cable_drone_virtualYZ">
+        <inertial>
+            <mass value="0.1"/>
+            <inertia ixx="0.001" ixy="0" ixz="0"
+                 iyy="0.001" iyz="0"
+                 izz="0.001"/>
         </inertial>
     </link>
     <joint name="${prefix}cable_to_drone_joint_x" type="continuous">
         <parent link="${prefix}link_${segments}"/>
-        <child link="${prefix}cable_drone_virtual"/>
+        <child link="${prefix}cable_drone_virtualXY"/>
         <origin xyz="0 0 0" rpy="0 0 0"/>
-        <axis xyz="1 0 0"/>
-        <dynamics damping="10.0" friction="0.01"/>
+        <axis xyz="0 0 1" />
     </joint>
     <joint name="${prefix}cable_to_drone_joint_y" type="continuous">
-        <parent link="${prefix}cable_drone_virtual"/>
+        <parent link="${prefix}cable_drone_virtualXY"/>
+        <child link="${prefix}cable_drone_virtualYZ"/>
+        <origin xyz="0 0 0" rpy="0 0 0"/>
+        <axis xyz="0 1 0" />
+    </joint>
+    <joint name="${prefix}cable_to_drone_joint_z" type="continuous">
+        <parent link="${prefix}cable_drone_virtualYZ"/>
         <child link="${prefix}base_link"/>
-        <axis xyz="0 1 0"/>
-        <dynamics damping="10.0" friction="0.01"/>
-    </joint> -->
+        <origin xyz="0 0 0" rpy="0 ${0} 0"/>
+        <axis xyz="1 0 0" />
+    </joint>
     <model>
     <gazebo reference="${prefix}base_link">
