Commit message: XYZ cable extreme movement

File: urdf/adaptable_cable.xacro (robot description, xacro)
@@ -3,37 +3,49 @@
   <xacro:include filename="$(find acts_simulator)/urdf/components/cable_component.xacro" />
   <link name="world"/>
-  <xacro:uav_cable
-    prefix=""
-    parent_link="world"
-    is_flexible="true"
-    segments="20"
-    length="10"
-    radius="0.01"
-    mass="0.1"
-    orientation="0" />
-<ros2_control name="GazeboSimSystem" type="system">
-  <hardware>
-    <plugin>gz_ros2_control/GazeboSimSystem</plugin>
-  </hardware>
-  <joint name="joint_pulley">
-    <command_interface name="position">
-      <param name="min">-10</param>
-      <param name="max">10</param>
-    </command_interface>
-    <state_interface name="position"/>
-    <state_interface name="velocity"/>
+  <link name="base_x_link"><inertial><mass value="0.01"/>
+    <inertia ixx="1e-5" ixy="0" ixz="0" iyy="1e-5" iyz="0" izz="1e-5"/> </inertial>
+  </link>
+  <joint name="joint_pulley_x" type="prismatic">
+    <parent link="world"/>
+    <child link="base_x_link"/>
+    <origin xyz="0 0 1.2" rpy="0 0 0"/><axis xyz="1 0 0"/>
+    <limit effort="1000.0" lower="-10.0" upper="10.0" velocity="2.0"/>
   </joint>
-</ros2_control>
-<gazebo>
-  <plugin name="gz_ros2_control::GazeboSimROS2ControlPlugin" filename="libgz_ros2_control-system.so">
-    <parameters>$(find acts_simulator)/config/cable_controller.yaml</parameters>
-  </plugin>
-  <plugin
-    filename="gz-sim-joint-controller-system"
-    name="gz::sim::systems::JointController">
-    <joint_name>joint_pulley</joint_name>
-    <initial_position>0.0</initial_position>
-    <topic>/model/cable/joint/joint_pulley/0/cmd_pos</topic>
-  </plugin>
-</gazebo>
+  <link name="base_y_link">
+    <inertial>
+      <mass value="0.01"/>
+      <inertia ixx="1e-5" ixy="0" ixz="0" iyy="1e-5" iyz="0" izz="1e-5"/>
+    </inertial>
+  </link>
+  <joint name="joint_pulley_y" type="prismatic">
+    <parent link="base_x_link"/>
+    <child link="base_y_link"/>
+    <origin xyz="0 0 0" rpy="0 0 0"/><axis xyz="0 1 0"/>
+    <limit effort="1000.0" lower="-10.0" upper="10.0" velocity="2.0"/>
+  </joint>
+  <link name="base_z_link">
+    <inertial>
+      <mass value="0.01"/>
+      <inertia ixx="1e-5" ixy="0" ixz="0" iyy="1e-5" iyz="0" izz="1e-5"/>
+    </inertial>
+  </link>
+  <joint name="joint_pulley_z" type="prismatic">
+    <parent link="base_y_link"/>
+    <child link="base_z_link"/>
+    <origin xyz="0 0 0" rpy="0 0 0"/>
+    <axis xyz="0 0 1"/>
+    <limit effort="1000.0" lower="-1.2" upper="10.0" velocity="2.0"/>
+  </joint>
+  <xacro:uav_cable prefix="" parent_link="base_z_link" is_flexible="true" segments="20" length="10" radius="0.01" mass="0.1" orientation="0" />
+  <ros2_control name="GazeboSimSystem" type="system">
+    <hardware><plugin>gz_ros2_control/GazeboSimSystem</plugin></hardware>
+    <joint name="joint_pulley_x"><command_interface name="position"/><state_interface name="position"/></joint>
+    <joint name="joint_pulley_y"><command_interface name="position"/><state_interface name="position"/></joint>
+    <joint name="joint_pulley_z"><command_interface name="position"/><state_interface name="position"/></joint>
+  </ros2_control>
+  <gazebo>
+    <plugin name="gz_ros2_control::GazeboSimROS2ControlPlugin" filename="libgz_ros2_control-system.so">
+      <parameters>$(find acts_simulator)/config/cable_controller.yaml</parameters>
+    </plugin>
+  </gazebo>
 </robot>

File: urdf/components/cable_component.xacro (robot description, xacro)
@@ -37,11 +37,8 @@
     </link>
     <xacro:if value="${current_num == 1}">
-      <joint name="${prefix}joint_pulley" type="prismatic">
+      <joint name="${prefix}joint_fixed_root" type="fixed">
         <parent link="${parent}"/>
         <child link="${prefix}virtual_${current_num}"/>
         <origin xyz="0 0 0" rpy="0 ${theta} 0"/>
-        <axis xyz="1 0 0"/>
-        <limit effort="10000.0" lower="-10.0" upper="10.0" velocity="5.0"/>
-        <dynamics damping="0.01" friction="0.01"/>
       </joint>
     </xacro:if>

Commit message: pulley working

File: urdf/adaptable_cable.xacro (robot description, xacro)
@@ -2,4 +2,5 @@
 <robot xmlns:xacro="http://www.ros.org/wiki/xacro" name="acts_system">
   <xacro:include filename="$(find acts_simulator)/urdf/components/cable_component.xacro" />
+  <xacro:include filename="$(find acts_simulator)/urdf/components/cable_guide.xacro" />
   <link name="world"/>
   <link name="base_x_link"><inertial><mass value="0.01"/>

File: urdf/components/cable_component.xacro (robot description, xacro)
@@ -49,5 +49,5 @@
         <origin xyz="0 0 ${cable_len}" rpy="0 0 0"/>
         <axis xyz="1 0 0"/>
-        <dynamics damping="0.01" friction="0.001"/>
+        <dynamics damping="2.0" friction="1.0"/>
       </joint>
     </xacro:unless>

Commit message: making the position-pulley scalable

File: urdf/adaptable_cable.xacro (robot description, xacro)
@@ -2,47 +2,24 @@
 <robot xmlns:xacro="http://www.ros.org/wiki/xacro" name="acts_system">
   <xacro:include filename="$(find acts_simulator)/urdf/components/cable_component.xacro" />
-  <xacro:include filename="$(find acts_simulator)/urdf/components/cable_guide.xacro" />
+  <xacro:include filename="$(find acts_simulator)/urdf/components/pulley.xacro" />
   <link name="world"/>
-  <link name="base_x_link"><inertial><mass value="0.01"/>
-    <inertia ixx="1e-5" ixy="0" ixz="0" iyy="1e-5" iyz="0" izz="1e-5"/> </inertial>
-  </link>
-  <joint name="joint_pulley_x" type="prismatic">
-    <parent link="world"/>
-    <child link="base_x_link"/>
-    <origin xyz="0 0 1.2" rpy="0 0 0"/><axis xyz="1 0 0"/>
-    <limit effort="1000.0" lower="-10.0" upper="10.0" velocity="2.0"/>
-  </joint>
-  <link name="base_y_link">
-    <inertial>
-      <mass value="0.01"/>
-      <inertia ixx="1e-5" ixy="0" ixz="0" iyy="1e-5" iyz="0" izz="1e-5"/>
-    </inertial>
-  </link>
-  <joint name="joint_pulley_y" type="prismatic">
-    <parent link="base_x_link"/>
-    <child link="base_y_link"/>
-    <origin xyz="0 0 0" rpy="0 0 0"/><axis xyz="0 1 0"/>
-    <limit effort="1000.0" lower="-10.0" upper="10.0" velocity="2.0"/>
-  </joint>
-  <link name="base_z_link">
-    <inertial>
-      <mass value="0.01"/>
-      <inertia ixx="1e-5" ixy="0" ixz="0" iyy="1e-5" iyz="0" izz="1e-5"/>
-    </inertial>
-  </link>
-  <joint name="joint_pulley_z" type="prismatic">
-    <parent link="base_y_link"/>
-    <child link="base_z_link"/>
-    <origin xyz="0 0 0" rpy="0 0 0"/>
-    <axis xyz="0 0 1"/>
-    <limit effort="1000.0" lower="-1.2" upper="10.0" velocity="2.0"/>
-  </joint>
-  <xacro:uav_cable prefix="" parent_link="base_z_link" is_flexible="true" segments="20" length="10" radius="0.01" mass="0.1" orientation="0" />
-  <ros2_control name="GazeboSimSystem" type="system">
-    <hardware><plugin>gz_ros2_control/GazeboSimSystem</plugin></hardware>
-    <joint name="joint_pulley_x"><command_interface name="position"/><state_interface name="position"/></joint>
-    <joint name="joint_pulley_y"><command_interface name="position"/><state_interface name="position"/></joint>
-    <joint name="joint_pulley_z"><command_interface name="position"/><state_interface name="position"/></joint>
-  </ros2_control>
+  <xacro:position_controlled_pulley prefix="pulley_A" parent_link="world" />
+  <xacro:arg name="x" default="0.0"/>
+  <xacro:arg name="y" default="0.0"/>
+  <xacro:arg name="z" default="0.0"/>
+  <xacro:arg name="length" default="5.0"/>
+  <xacro:uav_cable
+    prefix=""
+    parent_link="base_pulley_A_z_link"
+    is_flexible="true"
+    x="$(arg x)"
+    y="$(arg y)"
+    z="$(arg z)"
+    segments="20"
+    length="$(arg length)"
+    radius="0.01"
+    mass="0.1"
+    orientation="3.1415" />
+  <!-- <xacro:position_controlled_pulley prefix="pulley_B" parent_link="link_20" /> -->
   <gazebo>
     <plugin name="gz_ros2_control::GazeboSimROS2ControlPlugin" filename="libgz_ros2_control-system.so">

File: urdf/components/cable_component.xacro (robot description, xacro)
@@ -29,5 +29,5 @@
   </xacro:macro>
 <!-- ____________   Flexible cable  _______________________-->
-  <xacro:macro name="flexible_chain_generator" params="prefix parent current_num total_num cable_len rad m theta">
+  <xacro:macro name="flexible_chain_generator" params="prefix parent current_num x y z total_num cable_len rad m theta">
     <link name="${prefix}virtual_${current_num}">
       <inertial>
@@ -43,5 +43,5 @@
         <parent link="${parent}"/>
         <child link="${prefix}virtual_${current_num}"/>
-        <origin xyz="0 0 0" rpy="0 ${theta} 0"/>
+        <origin xyz="${x} ${y} ${z}" rpy="0 ${theta} 0"/>
       </joint>
     </xacro:if>
@@ -88,4 +88,5 @@
         parent="${prefix}link_${current_num}"
         current_num="${current_num + 1}"
+        x="0" y="0" z="0"
         total_num="${total_num}"
         cable_len="${cable_len}" rad="${rad}" m="${m}"
@@ -93,8 +94,9 @@
     </xacro:if>
   </xacro:macro>
-  <xacro:macro name="uav_cable" params="prefix parent_link is_flexible segments length radius mass orientation">
+  <xacro:macro name="uav_cable" params="prefix parent_link is_flexible x y z segments length radius mass orientation">
     <xacro:if value="${is_flexible}">
       <xacro:flexible_chain_generator
         prefix="${prefix}" parent="${parent_link}" current_num="1"
+        x="${x}" y="${y}" z="${z}"
         total_num="${segments}" cable_len="${length/segments}" rad="${radius}" m="${mass/segments}" theta="${orientation}" />
     </xacro:if>

File: urdf/components/cable_guide.xacro (robot description, xacro)
@@ -37,4 +37,24 @@
     <xacro:pulley_wall wall_name="e" wx="0.03" wy="0"    wsx="0.02" wsy="0.04"/>
     <xacro:pulley_wall wall_name="w" wx="-0.03" wy="0"    wsx="0.02" wsy="0.04"/>
+    <gazebo reference="${prefix}_link">
+      <collision name="${prefix}_collision">
+        <surface>
+          <contact>
+            <ode>
+              <kp>10000.0</kp>
+              <kd>100.0</kd>
+              <min_depth>0.005</min_depth>
+              <max_vel>0.1</max_vel>
+            </ode>
+          </contact>
+          <friction>
+            <ode>
+              <mu>0.05</mu>
+              <mu2>0.05</mu2>
+            </ode>
+          </friction>
+        </surface>
+      </collision>
+    </gazebo>
   </xacro:macro>
 </robot>

Commit message: Making the orientation of the pulley up/down scalable and WIND/UNWINDING

File: urdf/adaptable_cable.xacro (robot description, xacro)
@@ -9,4 +9,5 @@
   <xacro:arg name="z" default="0.0"/>
   <xacro:arg name="length" default="5.0"/>
+  <xacro:arg name="orientation" default="0.0"/>
   <xacro:uav_cable
     prefix=""
@@ -20,6 +21,6 @@
     radius="0.01"
     mass="0.1"
-    orientation="3.1415" />
-  <!-- <xacro:position_controlled_pulley prefix="pulley_B" parent_link="link_20" /> -->
+    orientation="$(arg orientation)" />
+  <xacro:position_controlled_pulley prefix="pulley_B" parent_link="link_20" />
   <gazebo>
     <plugin name="gz_ros2_control::GazeboSimROS2ControlPlugin" filename="libgz_ros2_control-system.so">

File: urdf/components/pulley.xacro (robot description, xacro)
@@ -34,5 +34,5 @@
     <origin xyz="0 0 0" rpy="0 0 0"/>
     <axis xyz="0 0 1"/>
-    <limit effort="1000.0" lower="-1.2" upper="10.0" velocity="2.0"/>
+    <limit lower="-100.0" upper="100.0" effort="1000" velocity="2.0"/>
   </joint>
   </xacro:macro>

Commit message: Torque pulley working but not controllable

File: urdf/adaptable_cable.xacro (robot description, xacro)
@@ -22,5 +22,5 @@
     mass="0.1"
     orientation="$(arg orientation)" />
-  <xacro:position_controlled_pulley prefix="pulley_B" parent_link="link_20" />
+  <xacro:forceTorque_controlled_pulley prefix="pulley_B" parent_link="link_20" />
   <gazebo>
     <plugin name="gz_ros2_control::GazeboSimROS2ControlPlugin" filename="libgz_ros2_control-system.so">

File: urdf/components/pulley.xacro (robot description, xacro)
@@ -9,5 +9,5 @@
     <child link="base_${prefix}_x_link"/>
     <origin xyz="0 0 0" rpy="0 0 0"/><axis xyz="1 0 0"/>
-    <limit effort="1000.0" lower="-10.0" upper="10.0" velocity="2.0"/>
+    <limit effort="1000.0" lower="-100.0" upper="100.0" velocity="5.0"/>
   </joint>
   <link name="base_${prefix}_y_link">
@@ -21,5 +21,5 @@
     <child link="base_${prefix}_y_link"/>
     <origin xyz="0 0 0" rpy="0 0 0"/><axis xyz="0 1 0"/>
-    <limit effort="1000.0" lower="-10.0" upper="10.0" velocity="2.0"/>
+    <limit effort="1000.0" lower="-100.0" upper="100.0" velocity="5.0"/>
   </joint>
   <link name="base_${prefix}_z_link">
@@ -34,5 +34,5 @@
     <origin xyz="0 0 0" rpy="0 0 0"/>
     <axis xyz="0 0 1"/>
-    <limit lower="-100.0" upper="100.0" effort="1000" velocity="2.0"/>
+    <limit lower="-100.0" upper="100.0" effort="1000" velocity="5.0"/>
   </joint>
   </xacro:macro>
@@ -46,3 +46,23 @@
     </ros2_control>
   </xacro:macro>
+   <xacro:macro name="forceTorque_controlled_pulley" params="prefix parent_link">
+    <xacro:pulley prefix="${prefix}" parent_link="${parent_link}"/>
+    <ros2_control name="ControlSystem_${prefix}" type="system">
+      <hardware> <plugin>gz_ros2_control/GazeboSimSystem</plugin> </hardware>
+      <joint name="joint_${prefix}_x">
+        <command_interface name="position"/>
+        <state_interface name="position"/>
+      </joint>
+      <joint name="joint_${prefix}_y">
+        <command_interface name="position"/>
+        <state_interface name="position"/>
+      </joint>
+      <joint name="joint_${prefix}_z">
+        <command_interface name="effort"/>
+        <state_interface name="position"/>
+        <state_interface name="velocity"/>
+        <state_interface name="effort"/>
+      </joint>
+    </ros2_control>
+  </xacro:macro>
 </robot>

Commit message: Torque pulley not working

File: urdf/adaptable_cable.xacro (robot description, xacro)
@@ -10,4 +10,5 @@
   <xacro:arg name="length" default="5.0"/>
   <xacro:arg name="orientation" default="0.0"/>
+  <xacro:arg name="segments" default="20.0"/>
   <xacro:uav_cable
     prefix=""
@@ -17,10 +18,11 @@
     y="$(arg y)"
     z="$(arg z)"
-    segments="20"
+    segments="$(arg segments)"
     length="$(arg length)"
     radius="0.01"
     mass="0.1"
     orientation="$(arg orientation)" />
-  <xacro:forceTorque_controlled_pulley prefix="pulley_B" parent_link="link_20" />
+  <xacro:forceTorque_controlled_pulley prefix="pulley_B" parent_link="link_$(arg segments)" />
+  <!-- <xacro:forceTorque_controlled_pulley prefix="pulley_B" parent_link="world" /> -->
   <gazebo>
     <plugin name="gz_ros2_control::GazeboSimROS2ControlPlugin" filename="libgz_ros2_control-system.so">

File: urdf/cable_guide.urdf.xacro (robot description, xacro)
@@ -3,11 +3,11 @@
   <xacro:include filename="$(find acts_simulator)/urdf/components/cable_guide.xacro" />
   <link name="world"/>
-  <xacro:cable_guide prefix="winding_pulley"
+  <xacro:cable_guide prefix="pulleyA"
     parent_link="world"
-    x="0" y="0" z="5"
+    x="0" y="0" z="11"
   />
-  <xacro:cable_guide prefix="unwinding_pulley"
+  <xacro:cable_guide prefix="pulleyB"
     parent_link="world"
-    x="0" y="0" z="2"
+    x="0" y="0" z="8"
   />
 </robot>

File: urdf/components/cable_component.xacro (robot description, xacro)
@@ -31,8 +31,5 @@
   <xacro:macro name="flexible_chain_generator" params="prefix parent current_num x y z total_num cable_len rad m theta">
     <link name="${prefix}virtual_${current_num}">
-      <inertial>
-        <mass value="0.0001"/>
-        <inertia ixx="1e-8" ixy="0" ixz="0" iyy="1e-8" iyz="0" izz="1e-8"/>
-      </inertial>
+      <xacro:cylinder_inertia m="${m}" r="${rad}" h="${cable_len}" />
       <visual name="visual">
         <geometry><sphere radius="0.001"/></geometry>
@@ -44,4 +41,5 @@
         <child link="${prefix}virtual_${current_num}"/>
         <origin xyz="${x} ${y} ${z}" rpy="0 ${theta} 0"/>
+        <dynamics damping="2.0" friction="1.0"/>
       </joint>
     </xacro:if>

File: urdf/components/pulley.xacro (robot description, xacro)
@@ -1,7 +1,15 @@
 <?xml version="1.0"?>
 <robot xmlns:xacro="http://www.ros.org/wiki/xacro">
+  <xacro:macro name="pulley_inertia" params="m inertia">
+    <inertial>
+      <mass value="${m}"/>
+      <inertia ixx="${inertia}" ixy="0.0" ixz="0.0"
+               iyy="${inertia}" iyz="0.0"
+               izz="${inertia}"/>
+    </inertial>
+  </xacro:macro>
   <xacro:macro name="pulley" params="prefix parent_link">
-    <link name="base_${prefix}_x_link"><inertial><mass value="0.01"/>
-    <inertia ixx="1e-5" ixy="0" ixz="0" iyy="1e-5" iyz="0" izz="1e-5"/> </inertial>
+    <link name="base_${prefix}_x_link">
+    <xacro:pulley_inertia m="0.01" inertia="1e-5" />
   </link>
   <joint name="joint_${prefix}_x" type="prismatic">
@@ -9,11 +17,9 @@
     <child link="base_${prefix}_x_link"/>
     <origin xyz="0 0 0" rpy="0 0 0"/><axis xyz="1 0 0"/>
-    <limit effort="1000.0" lower="-100.0" upper="100.0" velocity="5.0"/>
+    <limit effort="1000.0" lower="-100.0" upper="100.0" velocity="100.0"/>
+    <dynamics damping="0.1" friction="0.01"/>
   </joint>
   <link name="base_${prefix}_y_link">
-    <inertial>
-      <mass value="0.01"/>
-      <inertia ixx="1e-5" ixy="0" ixz="0" iyy="1e-5" iyz="0" izz="1e-5"/>
-    </inertial>
+    <xacro:pulley_inertia m="0.01" inertia="1e-5" />
   </link>
   <joint name="joint_${prefix}_y" type="prismatic">
@@ -21,11 +27,9 @@
     <child link="base_${prefix}_y_link"/>
     <origin xyz="0 0 0" rpy="0 0 0"/><axis xyz="0 1 0"/>
-    <limit effort="1000.0" lower="-100.0" upper="100.0" velocity="5.0"/>
+    <limit effort="1000.0" lower="-100.0" upper="100.0" velocity="100.0"/>
+    <dynamics damping="0.1" friction="0.01"/>
   </joint>
   <link name="base_${prefix}_z_link">
-    <inertial>
-      <mass value="0.01"/>
-      <inertia ixx="1e-5" ixy="0" ixz="0" iyy="1e-5" iyz="0" izz="1e-5"/>
-    </inertial>
+    <xacro:pulley_inertia m="0.01" inertia="1e-5" />
   </link>
   <joint name="joint_${prefix}_z" type="prismatic">
@@ -34,5 +38,6 @@
     <origin xyz="0 0 0" rpy="0 0 0"/>
     <axis xyz="0 0 1"/>
-    <limit lower="-100.0" upper="100.0" effort="1000" velocity="5.0"/>
+    <limit lower="-100.0" upper="100.0" effort="1000" velocity="100.0"/>
+    <dynamics damping="0.1" friction="0.01"/>
   </joint>
   </xacro:macro>
@@ -40,9 +45,24 @@
     <xacro:pulley prefix="${prefix}" parent_link="${parent_link}"/>
     <ros2_control name="ControlSystem_${prefix}" type="system">
-      <hardware> <plugin>gz_ros2_control/GazeboSimSystem</plugin></hardware>
-      <joint name="joint_${prefix}_x"> <command_interface name="position"/><state_interface name="position"/> </joint>
-      <joint name="joint_${prefix}_y"> <command_interface name="position"/><state_interface name="position"/> </joint>
-      <joint name="joint_${prefix}_z"> <command_interface name="position"/><state_interface name="position"/> </joint>
-    </ros2_control>
+      <hardware><plugin>gz_ros2_control/GazeboSimSystem</plugin></hardware>
+      <joint name="joint_${prefix}_x">
+        <command_interface name="position"/>
+        <state_interface name="position"/>
+        <state_interface name="velocity"/>
+        <state_interface name="effort"/>
+      </joint>
+      <joint name="joint_${prefix}_y">
+        <command_interface name="position"/>
+        <state_interface name="position"/>
+        <state_interface name="velocity"/>
+        <state_interface name="effort"/>
+      </joint>
+      <joint name="joint_${prefix}_z">
+        <command_interface name="position"/>
+        <state_interface name="position"/>
+        <state_interface name="velocity"/>
+        <state_interface name="effort"/>
+      </joint>
+      </ros2_control>
   </xacro:macro>
    <xacro:macro name="forceTorque_controlled_pulley" params="prefix parent_link">
@@ -51,13 +71,16 @@
       <hardware> <plugin>gz_ros2_control/GazeboSimSystem</plugin> </hardware>
       <joint name="joint_${prefix}_x">
-        <command_interface name="position"/>
-        <state_interface name="position"/>
+        <command_interface name="effort"/> <state_interface name="position"/>
+        <state_interface name="velocity"/>
+        <state_interface name="effort"/>
       </joint>
       <joint name="joint_${prefix}_y">
-        <command_interface name="position"/>
-        <state_interface name="position"/>
+        <command_interface name="effort"/> <state_interface name="position"/>
+        <state_interface name="velocity"/>
+        <state_interface name="effort"/>
       </joint>
       <joint name="joint_${prefix}_z">
         <command_interface name="effort"/>
+        <dynamics damping="0.1" friction="0.01"/>
         <state_interface name="position"/>
         <state_interface name="velocity"/>

Commit message: Cable to extremity  update working

File: urdf/adaptable_cable.xacro (robot description, xacro)
@@ -9,5 +9,5 @@
     <parent link="world"/>
     <child link="base_x_link"/>
-    <origin xyz="0 0 1.2" rpy="0 0 0"/><axis xyz="1 0 0"/>
+    <origin xyz="0 0 0.0" rpy="0 0 0"/><axis xyz="1 0 0"/>
     <limit effort="1000.0" lower="-10.0" upper="10.0" velocity="2.0"/>
   </joint>
