Commit message: Rigth heigth

File: urdf/acts_model.xacro (robot description, xacro)
@@ -6,4 +6,5 @@
   <xacro:property name="sqrt3" value="${3**0.5}"/>
   <xacro:property name="cable_segments" value="5"/>
+  <xacro:property name="system_heigth" value="1.5"/>
   <xacro:property name="hook1_x" value="0.0"/>
   <xacro:property name="hook1_y" value="${sqrt3 / 3}"/>
@@ -25,5 +26,8 @@
     link_name="chassis_link"
     mass="1.0"
-    x="2" y="2" z="0.2"
+    width="2"
+    length="2"
+    heigth="0.2"
+    x="0" y="0" z="${system_heigth}"
     material_name="Blue"
     material_color="0.0 0.0 0.8 0.0" />
@@ -40,5 +44,5 @@
     x_off="${ground_anchor_x}"
     y_off="${ground_anchor_y}"
-    z_off="${ground_anchor_z}"
+    z_off="${ground_anchor_z+system_heigth}"
     cable_roll="0.0" cable_pitch="0" cable_yaw="0" />
   <xacro:add_drone
@@ -49,5 +53,5 @@
     x_off="${hook1_x}"
     y_off="${hook1_y}"
-    z_off="${hook1_z}"
+    z_off="${hook1_z+system_heigth}"
     cable_roll="0" cable_pitch="0" cable_yaw="0" />
   <xacro:add_drone
@@ -58,5 +62,5 @@
     x_off="${hook2_x}"
     y_off="${hook2_y}"
-    z_off="${hook2_z}"
+    z_off="${hook2_z+system_heigth}"
     cable_roll="0" cable_pitch="0" cable_yaw="0" />
   <xacro:add_drone
@@ -67,5 +71,5 @@
     x_off="${hook3_x}"
     y_off="${hook3_y}"
-    z_off="${hook3_z}"
+    z_off="${hook3_z+system_heigth}"
     cable_roll="0" cable_pitch="0" cable_yaw="0" />
 </robot>

File: urdf/components/panel.xacro (robot description, xacro)
@@ -1,18 +1,18 @@
 <?xml version="1.0"?>
 <robot xmlns:xacro="http://www.ros.org/wiki/xacro">
-  <xacro:macro name="panel" params="link_name mass x y z material_name material_color">
+  <xacro:macro name="panel" params="link_name mass width length heigth x y z material_name material_color">
     <link name="${link_name}">
       <inertial>
-        <origin xyz="0 0 0" rpy="0 0 0"/>
+        <origin xyz="${x} ${y} ${z}" rpy="0 0 0"/>
         <mass value="${mass}"/>
         <inertia
-          ixx="${(1/12) * mass * (y*y + z*z)}" ixy="0.0" ixz="0.0"
-          iyy="${(1/12) * mass * (x*x + z*z)}" iyz="0.0"
-          izz="${(1/12) * mass * (x*x + y*y)}"/>
+          ixx="${(1/12) * mass * (length*length + heigth*heigth)}" ixy="0.0" ixz="0.0"
+          iyy="${(1/12) * mass * (width*width + heigth*heigth)}" iyz="0.0"
+          izz="${(1/12) * mass * (width*width + length*length)}"/>
       </inertial>
       <visual>
-        <origin xyz="0 0 0" rpy="0 0 0"/>
+        <origin xyz="${x} ${y} ${z}" rpy="0 0 0"/>
         <geometry>
-          <box size="${x} ${y} ${z}"/>
+          <box size="${width} ${length} ${heigth}"/>
         </geometry>
         <material name="${material_name}">
@@ -23,5 +23,5 @@
         <origin xyz="0 0 0" rpy="0 0 0"/>
         <geometry>
-          <box size="${x} ${y} ${z}"/>
+          <box size="${width} ${length} ${heigth}"/>
         </geometry>
       </collision>

Commit message: Initializing setting ugv to right position

File: urdf/acts_model.xacro (robot description, xacro)
@@ -38,5 +38,5 @@
   </joint>
   <xacro:add_ugv
-    id="4"
+    id="1"
     segments="${cable_segments}"
     length="1.5"
@@ -45,5 +45,16 @@
     y_off="${ground_anchor_y}"
     z_off="${ground_anchor_z+system_heigth}"
-    cable_roll="0.0" cable_pitch="0" cable_yaw="0" />
+    cable_roll="0.0" cable_pitch="0" cable_yaw="0"
+    target_hook="hook1" />
+    <xacro:add_ugv
+    id="2"
+    segments="${cable_segments}"
+    length="1.5"
+    panel_link="chassis_link"
+    x_off="${ground_anchor_x+0.5}"
+    y_off="${ground_anchor_y+0.5}"
+    z_off="${ground_anchor_z+system_heigth}"
+    cable_roll="0.0" cable_pitch="0" cable_yaw="0"
+    target_hook="hook2" />
   <xacro:add_drone
     id="1"
@@ -73,3 +84,12 @@
     z_off="${hook3_z+system_heigth}"
     cable_roll="0" cable_pitch="0" cable_yaw="0" />
+    <!-- <gazebo>
+    <plugin name="gz_ros2_control::GazeboSimROS2ControlPlugin" filename="libgz_ros2_control-system.so">
+      <parameters>$(find acts_simulator)/config/cable_controller.yaml</parameters>
+    </plugin>
+  </gazebo> -->
+<!--
+    <gazebo>
+    <plugin filename="gz-sim-apply-link-wrench-system" name="gz::sim::systems::ApplyLinkWrench"/>
+  </gazebo> -->
 </robot>

File: urdf/ugv_cable_assembly.urdf.xacro (robot description, xacro)
@@ -3,12 +3,6 @@
   <xacro:include filename="$(find acts_simulator)/urdf/components/cable_component.xacro" />
   <xacro:include filename="$(find acts_simulator)/urdf/components/ugv_component.xacro" />
-  <xacro:macro name="add_ugv" params="id segments length x_off:=0 y_off:=0 z_off:=0 cable_roll:=0 cable_pitch:=0 cable_yaw:=0 panel_link:=''">
+  <xacro:macro name="add_ugv" params="id segments length x_off:=0 y_off:=0 z_off:=0 cable_roll:=0 cable_pitch:=0 cable_yaw:=0 panel_link:='' target_hook:='hook1'">
     <xacro:property name="prefix" value="ugv${id}_" />
-    <xacro:ugv_component
-    prefix="${prefix}"
-    x="0"
-    y="0"
-    z="0"
-    />
     <link name="${prefix}cable_root_link">
         <inertial>
@@ -34,44 +28,39 @@
         cable_yaw="${cable_yaw}"
         radius="0.005" mass="0.01" />
-       <link name="${prefix}virtual_cable_to_ugv_joint">
+   <link name="${prefix}virtual_extreme_link">
         <inertial>
-            <mass value="0.0001"/>
-            <inertia ixx="1e-6" ixy="0" ixz="0" iyy="1e-6" iyz="0" izz="1e-6"/>
+            <mass value="0.01"/>
+            <inertia ixx="1e-5" ixy="0" ixz="0" iyy="1e-5" iyz="0" izz="1e-5"/>
         </inertial>
+        <visual>
+            <geometry>
+                <sphere radius="0.02"/>
+            </geometry>
+            <material name="Red">
+                <color rgba="1.0 0.0 0.0 1.0"/>
+            </material>
+        </visual>
+        <collision>
+            <geometry>
+                <sphere radius="0.02"/>
+            </geometry>
+        </collision>
     </link>
-    <link name="${prefix}cable_attach_link">
-    <inertial>
-        <mass value="0.0001"/>
-        <inertia ixx="1e-6" ixy="0" ixz="0" iyy="1e-6" iyz="0" izz="1e-6"/>
-    </inertial>
-    </link>
-    <!-- Fix the attachment link to the ugv's base_link -->
-    <joint name="${prefix}cable_attach_fixed" type="fixed">
-    <parent link="${prefix}cable_attach_link"/>
-    <child link="${prefix}base_link"/>
-    <origin xyz="0 0 0" rpy="0 0 0"/>
+    <joint name="${prefix}extreme_motor_joint" type="fixed">
+        <parent link="${prefix}link_${segments}"/>
+        <child link="${prefix}virtual_extreme_link"/>
+        <origin xyz="0 0 0" rpy="0 0 0"/>
     </joint>
-    <!-- joint_x: last cable segment to virtual -->
-    <joint name="${prefix}joint_x_cable_to_ugv_joint" type="revolute">
-    <parent link="${prefix}link_${segments}"/>
-    <child link="${prefix}virtual_cable_to_ugv_joint"/>
-    <axis xyz="1 0 0"/>
-    <limit lower="-1.5708" upper="1.5708" effort="10" velocity="1.0"/>
-    <dynamics damping="0.05" friction="0.01"/>
-    </joint>
-    <!-- joint_y: virtual to cable_attach_link  -->
-    <joint name="${prefix}joint_y_cable_to_ugv_joint" type="revolute">
-    <parent link="${prefix}virtual_cable_to_ugv_joint"/>
-    <child link="${prefix}cable_attach_link"/>
-    <axis xyz="0 1 0"/>
-    <limit lower="-1.5708" upper="1.5708" effort="10" velocity="1.0"/>
-    <dynamics damping="0.05" friction="0.01"/>
-    </joint>
-    <gazebo reference="${prefix}base_link">
+    <gazebo reference="${prefix}extreme_motor_joint">
         <preserveFixedJoint>true</preserveFixedJoint>
     </gazebo>
-    <gazebo reference="${prefix}cable_attach_link">
-        <preserveFixedJoint>true</preserveFixedJoint>
-    </gazebo>
+    <!-- <gazebo>
+        <plugin filename="gz-sim-pose-publisher-system" name="gz::sim::systems::PosePublisher">
+            <publish_link_pose>true</publish_link_pose>
+            <publish_nested_model_pose>true</publish_nested_model_pose>
+            <use_pose_vector_msg>true</use_pose_vector_msg>
+            <update_rate>50</update_rate>
+        </plugin>
+    </gazebo> -->
   </xacro:macro>
 </robot>

Commit message: joint moving, but wrong extremity

File: urdf/acts_model.xacro (robot description, xacro)
@@ -4,4 +4,5 @@
   <xacro:include filename="uav_cable_assembly.urdf.xacro" />
   <xacro:include filename="ugv_cable_assembly.urdf.xacro" />
+  <xacro:arg name="controller_config" default=""/>
   <xacro:property name="sqrt3" value="${3**0.5}"/>
   <xacro:property name="cable_segments" value="5"/>
@@ -22,4 +23,22 @@
   <xacro:property name="target1_y" value="0.0"/>
   <xacro:property name="target1_z" value="0.0"/>
+  <xacro:macro name="ros2_control_ugv_joint" params="prefix">
+    <joint name="${prefix}joint_x_cable_to_ugv">
+      <command_interface name="position">
+        <param name="min">-1.5708</param>
+        <param name="max"> 1.5708</param>
+      </command_interface>
+      <state_interface name="position"/>
+      <state_interface name="velocity"/>
+    </joint>
+    <joint name="${prefix}joint_y_cable_to_ugv">
+      <command_interface name="position">
+        <param name="min">-1.5708</param>
+        <param name="max"> 1.5708</param>
+      </command_interface>
+      <state_interface name="position"/>
+      <state_interface name="velocity"/>
+    </joint>
+  </xacro:macro>
   <link name="base_link"/>
   <xacro:panel
@@ -45,6 +64,5 @@
     y_off="${ground_anchor_y}"
     z_off="${ground_anchor_z+system_heigth}"
-    cable_roll="0.0" cable_pitch="0" cable_yaw="0"
-    target_hook="hook1" />
+    cable_roll="0.0" cable_pitch="0" cable_yaw="0"/>
     <xacro:add_ugv
     id="2"
@@ -55,6 +73,5 @@
     y_off="${ground_anchor_y+0.5}"
     z_off="${ground_anchor_z+system_heigth}"
-    cable_roll="0.0" cable_pitch="0" cable_yaw="0"
-    target_hook="hook2" />
+    cable_roll="0.0" cable_pitch="0" cable_yaw="0"/>
   <xacro:add_drone
     id="1"
@@ -84,12 +101,19 @@
     z_off="${hook3_z+system_heigth}"
     cable_roll="0" cable_pitch="0" cable_yaw="0" />
-    <!-- <gazebo>
-    <plugin name="gz_ros2_control::GazeboSimROS2ControlPlugin" filename="libgz_ros2_control-system.so">
-      <parameters>$(find acts_simulator)/config/cable_controller.yaml</parameters>
+    <ros2_control name="CableSystem" type="system">
+    <hardware>
+      <plugin>gz_ros2_control/GazeboSimSystem</plugin>
+    </hardware>
+    <xacro:ros2_control_ugv_joint prefix="ugv1_" />
+    <xacro:ros2_control_ugv_joint prefix="ugv2_" />
+    <!-- add ugv3...ugv6 tip joints here, same pattern -->
+  </ros2_control>
+  <gazebo>
+    <plugin filename="gz_ros2_control-system"
+            name="gz_ros2_control::GazeboSimROS2ControlPlugin">
+      <robot_param>robot_description</robot_param>
+      <robot_param_node>robot_state_publisher</robot_param_node>
+      <parameters>$(arg controller_config)</parameters>
     </plugin>
-  </gazebo> -->
-<!--
-    <gazebo>
-    <plugin filename="gz-sim-apply-link-wrench-system" name="gz::sim::systems::ApplyLinkWrench"/>
-  </gazebo> -->
+  </gazebo>
 </robot>

File: urdf/components/ugv_component.xacro (robot description, xacro)
@@ -10,6 +10,9 @@
       <visual>
         <geometry>
-        <box size="0.2 0.2 0.1"/>
+            <sphere radius="0.02"/>
         </geometry>
+        <material name="Red">
+            <color rgba="1.0 0.0 0.0 1.0"/>
+        </material>
       </visual>
 		<!-- <collision name="${prefix}base_collision">

File: urdf/uav_cable_assembly.urdf.xacro (robot description, xacro)
@@ -1,6 +1,6 @@
 <?xml version="1.0"?>
 <robot xmlns:xacro="http://www.ros.org/wiki/xacro">
-  <xacro:include filename="$(find acts_simulator)/urdf/crazy2fly.urdf.xacro" />
-  <xacro:include filename="$(find acts_simulator)/urdf/components/cable_component.xacro" />
+  <xacro:include filename="crazy2fly.urdf.xacro" />
+  <xacro:include filename="components/cable_component.xacro" />
 <xacro:macro name="add_drone" params="id segments length x_off:=0 y_off:=0 z_off:=0 cable_roll:=0 cable_pitch:=0 cable_yaw:=0 panel_link:=''">
     <xacro:property name="prefix" value="drone${id}_" />

File: urdf/ugv_cable_assembly.urdf.xacro (robot description, xacro)
@@ -1,66 +1,63 @@
 <?xml version="1.0"?>
 <robot xmlns:xacro="http://www.ros.org/wiki/xacro">
-  <xacro:include filename="$(find acts_simulator)/urdf/components/cable_component.xacro" />
-  <xacro:include filename="$(find acts_simulator)/urdf/components/ugv_component.xacro" />
-  <xacro:macro name="add_ugv" params="id segments length x_off:=0 y_off:=0 z_off:=0 cable_roll:=0 cable_pitch:=0 cable_yaw:=0 panel_link:='' target_hook:='hook1'">
+  <xacro:include filename="components/cable_component.xacro" />
+  <xacro:include filename="components/ugv_component.xacro" />
+  <xacro:macro name="add_ugv" params="id segments length x_off:=0 y_off:=0 z_off:=0
+                                       cable_roll:=0 cable_pitch:=0 cable_yaw:=0 panel_link:=''">
     <xacro:property name="prefix" value="ugv${id}_" />
+    <!-- UGV body -->
+    <xacro:ugv_component prefix="${prefix}" x="0" y="0" z="0" />
+    <!-- Cable attachment point at the top (fixed to panel) -->
     <link name="${prefix}cable_root_link">
-        <inertial>
-            <mass value="0.0001"/>
-            <inertia ixx="1e-6" ixy="0" ixz="0" iyy="1e-6" iyz="0" izz="1e-6"/>
-        </inertial>
+      <inertial>
+        <mass value="0.0001"/>
+        <inertia ixx="1e-6" ixy="0" ixz="0" iyy="1e-6" iyz="0" izz="1e-6"/>
+      </inertial>
     </link>
     <xacro:unless value="${panel_link == ''}">
-        <joint name="${prefix}panel_to_cable_joint" type="fixed">
-            <parent link="${panel_link}"/>
-            <child link="${prefix}cable_root_link"/>
-            <origin xyz="${x_off} ${y_off} ${z_off}" rpy="0 0 0"/>
-        </joint>
+      <joint name="${prefix}panel_to_cable_joint" type="fixed">
+        <parent link="${panel_link}"/>
+        <child link="${prefix}cable_root_link"/>
+        <origin xyz="${x_off} ${y_off} ${z_off}" rpy="0 0 0"/>
+      </joint>
     </xacro:unless>
+    <!-- Cable chain: cable_root_link → link_1 → ... → link_N -->
     <xacro:ugv_cable
-        prefix="${prefix}"
-        parent_link="${prefix}cable_root_link"
-        is_flexible="true"
-        segments="${segments}"
-        length="${length}"
-        cable_roll="${cable_roll}"
-        cable_pitch="${cable_pitch}"
-        cable_yaw="${cable_yaw}"
-        radius="0.005" mass="0.01" />
-   <link name="${prefix}virtual_extreme_link">
-        <inertial>
-            <mass value="0.01"/>
-            <inertia ixx="1e-5" ixy="0" ixz="0" iyy="1e-5" iyz="0" izz="1e-5"/>
-        </inertial>
-        <visual>
-            <geometry>
-                <sphere radius="0.02"/>
-            </geometry>
-            <material name="Red">
-                <color rgba="1.0 0.0 0.0 1.0"/>
-            </material>
-        </visual>
-        <collision>
-            <geometry>
-                <sphere radius="0.02"/>
-            </geometry>
-        </collision>
+      prefix="${prefix}"
+      parent_link="${prefix}cable_root_link"
+      is_flexible="true"
+      segments="${segments}"
+      length="${length}"
+      cable_roll="${cable_roll}"
+      cable_pitch="${cable_pitch}"
+      cable_yaw="${cable_yaw}"
+      radius="0.005" mass="0.01" />
+    <!-- Virtual intermediate link for the 2-axis joint at the tip -->
+    <link name="${prefix}virtual_tip_link">
+      <inertial>
+        <mass value="0.0001"/>
+        <inertia ixx="1e-6" ixy="0" ixz="0" iyy="1e-6" iyz="0" izz="1e-6"/>
+      </inertial>
     </link>
-    <joint name="${prefix}extreme_motor_joint" type="fixed">
-        <parent link="${prefix}link_${segments}"/>
-        <child link="${prefix}virtual_extreme_link"/>
-        <origin xyz="0 0 0" rpy="0 0 0"/>
+    <!-- joint_x: last cable segment → virtual tip (rotation around X) -->
+    <joint name="${prefix}joint_x_cable_to_ugv" type="revolute">
+      <parent link="${prefix}link_${segments}"/>
+      <child link="${prefix}virtual_tip_link"/>
+      <axis xyz="1 0 0"/>
+      <limit lower="-1.5708" upper="1.5708" effort="10" velocity="1.0"/>
+      <dynamics damping="0.05" friction="0.01"/>
     </joint>
-    <gazebo reference="${prefix}extreme_motor_joint">
-        <preserveFixedJoint>true</preserveFixedJoint>
+    <!-- joint_y: virtual tip → base_link (rotation around Y) -->
+    <joint name="${prefix}joint_y_cable_to_ugv" type="revolute">
+      <parent link="${prefix}virtual_tip_link"/>
+      <child link="${prefix}base_link"/>
+      <axis xyz="0 1 0"/>
+      <limit lower="-1.5708" upper="1.5708" effort="10" velocity="1.0"/>
+      <dynamics damping="0.05" friction="0.01"/>
+    </joint>
+    <!-- Keep fixed joints from being welded by Gazebo -->
+    <gazebo reference="${prefix}panel_to_cable_joint">
+      <preserveFixedJoint>true</preserveFixedJoint>
     </gazebo>
-    <!-- <gazebo>
-        <plugin filename="gz-sim-pose-publisher-system" name="gz::sim::systems::PosePublisher">
-            <publish_link_pose>true</publish_link_pose>
-            <publish_nested_model_pose>true</publish_nested_model_pose>
-            <use_pose_vector_msg>true</use_pose_vector_msg>
-            <update_rate>50</update_rate>
-        </plugin>
-    </gazebo> -->
   </xacro:macro>
 </robot>
