Commit message: Effort controller [DOESN'T WORK]

File: urdf/acts_model.xacro (robot description, xacro)
@@ -25,7 +25,7 @@
   <xacro:macro name="ros2_control_ugv_joint" params="prefix">
     <joint name="${prefix}joint_x_cable_to_ugv">
-      <command_interface name="position">
-        <param name="min">-1.5708</param>
-        <param name="max"> 1.5708</param>
+      <command_interface name="effort">
+        <param name="min">-20.0</param>
+        <param name="max"> 20.0</param>
       </command_interface>
       <state_interface name="position"/>
@@ -33,7 +33,7 @@
     </joint>
     <joint name="${prefix}joint_y_cable_to_ugv">
-      <command_interface name="position">
-        <param name="min">-1.5708</param>
-        <param name="max"> 1.5708</param>
+      <command_interface name="effort">
+        <param name="min">-20.0</param>
+        <param name="max"> 20.0</param>
       </command_interface>
       <state_interface name="position"/>

File: urdf/components/ugv_component.xacro (robot description, xacro)
@@ -4,5 +4,5 @@
     <link name="${prefix}base_link">
       <inertial>
-        <mass value="10.0" />
+        <mass value="0.001" />
         <origin xyz="0 0 0" rpy="0 0 0" />
         <inertia ixx="0.01" ixy="0" ixz="0" iyy="0.01" iyz="0" izz="0.02" />

File: urdf/ground_hooks.xacro (robot description, xacro)
@@ -14,29 +14,8 @@
     </link>
     <joint name="base_link_to_${prefix}" type="fixed">
-      <parent link="base_link"/>   <!-- was: world -->
+      <parent link="world"/>   <!-- was: world -->
       <child link="${prefix}"/>
       <origin xyz="${x} ${y} ${z}" rpy="0 0 0"/>
     </joint>
-    <ros2_control name="ControlSystem_${prefix}" type="system">
-      <hardware><plugin>gz_ros2_control/GazeboSimSystem</plugin></hardware>
-      <joint name="joint_${prefix}_x">
-        <command_interface name="position"/>
-        <state_interface name="position"/>
-        <state_interface name="velocity"/>
-        <state_interface name="effort"/>
-      </joint>
-      <joint name="joint_${prefix}_y">
-        <command_interface name="position"/>
-        <state_interface name="position"/>
-        <state_interface name="velocity"/>
-        <state_interface name="effort"/>
-      </joint>
-      <joint name="joint_${prefix}_z">
-        <command_interface name="position"/>
-        <state_interface name="position"/>
-        <state_interface name="velocity"/>
-        <state_interface name="effort"/>
-      </joint>
-    </ros2_control>
   </xacro:macro>
   <link name="world"/>

File: urdf/ugv_cable_assembly.urdf.xacro (robot description, xacro)
@@ -1,12 +1,10 @@
 <?xml version="1.0"?>
 <robot xmlns:xacro="http://www.ros.org/wiki/xacro">
-  <xacro:include filename="components/cable_component.xacro" />
-  <xacro:include filename="components/ugv_component.xacro" />
+  <xacro:include filename="$(find acts_simulator)/urdf/components/cable_component.xacro" />
+  <xacro:include filename="$(find acts_simulator)/urdf/components/ugv_component.xacro" />
   <xacro:macro name="add_ugv" params="id segments length x_off:=0 y_off:=0 z_off:=0
                                        cable_roll:=0 cable_pitch:=0 cable_yaw:=0 panel_link:=''">
     <xacro:property name="prefix" value="ugv${id}_" />
-    <!-- UGV body -->
     <xacro:ugv_component prefix="${prefix}" x="0" y="0" z="0" />
-    <!-- Cable attachment point at the top (fixed to panel) -->
     <link name="${prefix}cable_root_link">
       <inertial>
@@ -22,8 +20,35 @@
       </joint>
     </xacro:unless>
-    <!-- Cable chain: cable_root_link → link_1 → ... → link_N -->
+    <link name="${prefix}virtual_top_link">
+      <inertial>
+        <mass value="0.0001"/>
+        <inertia ixx="1e-6" ixy="0" ixz="0" iyy="1e-6" iyz="0" izz="1e-6"/>
+      </inertial>
+    </link>
+    <joint name="${prefix}joint_x_cable_to_ugv" type="revolute">
+      <parent link="${prefix}cable_root_link"/>
+      <child link="${prefix}virtual_top_link"/>
+      <origin xyz="0 0 0" rpy="0 0 0"/>
+      <axis xyz="1 0 0"/>
+      <limit lower="-1.5708" upper="1.5708" effort="20" velocity="2.0"/>
+      <dynamics damping="0.1" friction="0.01"/>
+    </joint>
+    <link name="${prefix}actuated_cable_base_link">
+      <inertial>
+        <mass value="0.0001"/>
+        <inertia ixx="1e-6" ixy="0" ixz="0" iyy="1e-6" iyz="0" izz="1e-6"/>
+      </inertial>
+    </link>
+    <joint name="${prefix}joint_y_cable_to_ugv" type="revolute">
+      <parent link="${prefix}virtual_top_link"/>
+      <child link="${prefix}actuated_cable_base_link"/>
+      <origin xyz="0 0 0" rpy="0 0 0"/>
+      <axis xyz="0 1 0"/>
+      <limit lower="-1.5708" upper="1.5708" effort="20" velocity="2.0"/>
+      <dynamics damping="0.1" friction="0.01"/>
+    </joint>
     <xacro:ugv_cable
       prefix="${prefix}"
-      parent_link="${prefix}cable_root_link"
+      parent_link="${prefix}actuated_cable_base_link"
       is_flexible="true"
       segments="${segments}"
@@ -33,29 +58,13 @@
       cable_yaw="${cable_yaw}"
       radius="0.005" mass="0.01" />
-    <!-- Virtual intermediate link for the 2-axis joint at the tip -->
-    <link name="${prefix}virtual_tip_link">
-      <inertial>
-        <mass value="0.0001"/>
-        <inertia ixx="1e-6" ixy="0" ixz="0" iyy="1e-6" iyz="0" izz="1e-6"/>
-      </inertial>
-    </link>
-    <!-- joint_x: last cable segment → virtual tip (rotation around X) -->
-    <joint name="${prefix}joint_x_cable_to_ugv" type="revolute">
+    <joint name="${prefix}cable_to_base_fixed_joint" type="fixed">
       <parent link="${prefix}link_${segments}"/>
-      <child link="${prefix}virtual_tip_link"/>
-      <axis xyz="1 0 0"/>
-      <limit lower="-1.5708" upper="1.5708" effort="10" velocity="1.0"/>
-      <dynamics damping="0.05" friction="0.01"/>
+      <child link="${prefix}base_link"/>
+      <origin xyz="0 0 0" rpy="0 0 0"/>
     </joint>
-    <!-- joint_y: virtual tip → base_link (rotation around Y) -->
-    <joint name="${prefix}joint_y_cable_to_ugv" type="revolute">
-      <parent link="${prefix}virtual_tip_link"/>
-      <child link="${prefix}base_link"/>
-      <axis xyz="0 1 0"/>
-      <limit lower="-1.5708" upper="1.5708" effort="10" velocity="1.0"/>
-      <dynamics damping="0.05" friction="0.01"/>
-    </joint>
-    <!-- Keep fixed joints from being welded by Gazebo -->
     <gazebo reference="${prefix}panel_to_cable_joint">
+      <preserveFixedJoint>true</preserveFixedJoint>
+    </gazebo>
+    <gazebo reference="${prefix}cable_to_base_fixed_joint">
       <preserveFixedJoint>true</preserveFixedJoint>
     </gazebo>

Commit message: Last try

File: urdf/acts_model.xacro (robot description, xacro)
@@ -6,6 +6,6 @@
   <xacro:arg name="controller_config" default=""/>
   <xacro:property name="sqrt3" value="${3**0.5}"/>
-  <xacro:property name="cable_segments" value="5"/>
-  <xacro:property name="system_heigth" value="1.0"/>
+  <xacro:property name="cable_segments" value="10"/>
+  <xacro:property name="system_heigth" value="2.0"/>
   <xacro:property name="hook1_x" value="0.0"/>
   <xacro:property name="hook1_y" value="${sqrt3 / 3}"/>
@@ -26,5 +26,5 @@
   <xacro:panel
     link_name="chassis_link"
-    mass="1.0"
+    mass="0.001"
     width="2"
     length="2"
@@ -56,5 +56,5 @@
     z_off="${ground_anchor_z+system_heigth}"
     cable_roll="0.0" cable_pitch="0" cable_yaw="0"/>
-  <xacro:add_drone
+  <!-- <xacro:add_drone
     id="1"
     segments="${cable_segments}"
@@ -82,5 +82,5 @@
     y_off="${hook3_y}"
     z_off="${hook3_z+system_heigth}"
-    cable_roll="0" cable_pitch="0" cable_yaw="0" />
+    cable_roll="0" cable_pitch="0" cable_yaw="0" /> -->
     <gazebo>
     <plugin name="gz_ros2_control::GazeboSimROS2ControlPlugin" filename="libgz_ros2_control-system.so">

File: urdf/adaptable_cable.xacro (robot description, xacro)
@@ -2,10 +2,14 @@
 <robot xmlns:xacro="http://www.ros.org/wiki/xacro" name="acts_system">
   <xacro:include filename="$(find acts_simulator)/urdf/components/cable_component.xacro" />
+  <xacro:include filename="components/pulley.xacro" />
   <link name="world"/>
+  <xacro:pulley
+    prefix="cable1_"
+    parent_link="world" />
   <link name="base_x_link"><inertial><mass value="0.01"/>
     <inertia ixx="1e-5" ixy="0" ixz="0" iyy="1e-5" iyz="0" izz="1e-5"/> </inertial>
   </link>
   <joint name="joint_pulley_x" type="prismatic">
-    <parent link="world"/>
+    <parent link="cable1_base_z_link"/>
     <child link="base_x_link"/>
     <origin xyz="0 0 0.0" rpy="0 0 0"/><axis xyz="1 0 0"/>
@@ -37,5 +41,5 @@
     <limit effort="1000.0" lower="-1.2" upper="10.0" velocity="2.0"/>
   </joint>
-  <xacro:uav_cable prefix="" parent_link="base_z_link" is_flexible="true" segments="20" length="10" radius="0.01" mass="0.1" orientation="0" />
+  <xacro:uav_cable prefix="" parent_link="base_z_link" is_flexible="true" segments="20" length="10" radius="0.01" mass="0.1" />
   <ros2_control name="GazeboSimSystem" type="system">
     <hardware><plugin>gz_ros2_control/GazeboSimSystem</plugin></hardware>

File: urdf/components/panel.xacro (robot description, xacro)
@@ -21,5 +21,5 @@
       </visual>
       <collision>
-        <origin xyz="0 0 0" rpy="0 0 0"/>
+        <origin xyz="${x} ${y} ${z}" rpy="0 0 0"/>
         <geometry>
           <box size="${width} ${length} ${heigth}"/>

File: urdf/components/pulley.xacro (robot description, xacro)
@@ -4,4 +4,12 @@
 <link name="${prefix}base_x_link"><inertial><mass value="0.01"/>
     <inertia ixx="1e-5" ixy="0" ixz="0" iyy="1e-5" iyz="0" izz="1e-5"/> </inertial>
+    <visual>
+        <geometry>
+            <sphere radius="0.1"/>
+        </geometry>
+        <material name="blue">
+            <color rgba="1.0 0.0 0.0 1.0"/>
+        </material>
+      </visual>
   </link>
   <joint name="${prefix}joint_pulley_x" type="prismatic">
@@ -36,13 +44,31 @@
     <origin xyz="0 0 0" rpy="0 0 0"/>
     <axis xyz="0 0 1"/>
-    <limit effort="1000.0" lower="-1.2" upper="10.0" velocity="2.0"/>
+    <limit effort="1000.0" lower="-20" upper="20.0" velocity="2.0"/>
     <dynamics damping="10.0" friction="0.5"/>
   </joint>
     <ros2_control name="${prefix}GazeboSimSystem" type="system">
-        <hardware><plugin>gz_ros2_control/GazeboSimSystem</plugin></hardware>
-        <joint name="${prefix}joint_pulley_x"><command_interface name="position"/><state_interface name="position"/></joint>
-        <joint name="${prefix}joint_pulley_y"><command_interface name="position"/><state_interface name="position"/></joint>
-        <joint name="${prefix}joint_pulley_z"><command_interface name="position"/><state_interface name="position"/></joint>
-    </ros2_control>
+    <hardware>
+      <plugin>gz_ros2_control/GazeboSimSystem</plugin>
+    </hardware>
+    <joint name="${prefix}joint_pulley_x">
+      <command_interface name="position"/>
+      <state_interface name="position"/>
+      <state_interface name="velocity"/>
+    </joint>
+    <joint name="${prefix}joint_pulley_y">
+      <command_interface name="position"/>
+      <state_interface name="position"/>
+      <state_interface name="velocity"/>
+    </joint>
+    <joint name="${prefix}joint_pulley_z">
+      <command_interface name="position"/>
+      <state_interface name="position"/>
+      <state_interface name="velocity"/>
+    </joint>
+  </ros2_control>
+  <gazebo>
+    <plugin filename="gz_ros2_control-system" name="gz_ros2_control::GazeboSimROS2ControlPlugin">
+      </plugin>
+  </gazebo>
 </xacro:macro>
 </robot>
