Commit message: Cable moveable correctly along one axis

File: urdf/components/cable_component.xacro (robot description, xacro)
@@ -29,60 +29,66 @@
   </xacro:macro>
 <!-- ____________   Flexible cable  _______________________-->
-  <xacro:macro name="flexible_chain_generator" params="prefix parent current_num total_num cable_len rad m">
-  <link name="${prefix}virtual_${current_num}">
-    <inertial>
-      <mass value="0.0001"/> <inertia ixx="1e-8" ixy="0" ixz="0" iyy="1e-8" iyz="0" izz="1e-8"/>
-    </inertial>
-  </link>
-  <joint name="${prefix}joint_x_${current_num}" type="continuous">
-    <parent link="${parent}"/>
-    <child link="${prefix}virtual_${current_num}"/>
+  <xacro:macro name="flexible_chain_generator" params="prefix parent current_num total_num cable_len rad m theta">
+    <link name="${prefix}virtual_${current_num}">
+      <inertial>
+        <mass value="0.0001"/>
+        <inertia ixx="1e-8" ixy="0" ixz="0" iyy="1e-8" iyz="0" izz="1e-8"/>
+      </inertial>
+    </link>
     <xacro:if value="${current_num == 1}">
-      <origin xyz="0 0 0" rpy="0 0 0"/> </xacro:if>
+      <joint name="${prefix}joint_pulley" type="prismatic">
+        <parent link="${parent}"/>
+        <child link="${prefix}virtual_${current_num}"/>
+        <origin xyz="0 0 0" rpy="0 ${theta} 0"/>
+        <axis xyz="1 0 0"/>
+        <limit effort="10000.0" lower="-10.0" upper="10.0" velocity="5.0"/>
+        <dynamics damping="0.01" friction="0.01"/>
+      </joint>
+    </xacro:if>
     <xacro:unless value="${current_num == 1}">
-      <origin xyz="0 0 ${cable_len}" rpy="0 0 0"/>
+      <joint name="${prefix}joint_x_${current_num}" type="continuous">
+        <parent link="${parent}"/>
+        <child link="${prefix}virtual_${current_num}"/>
+        <origin xyz="0 0 ${cable_len}" rpy="0 0 0"/>
+        <axis xyz="1 0 0"/>
+        <dynamics damping="0.01" friction="0.001"/>
+      </joint>
     </xacro:unless>
-    <axis xyz="1 0 0"/>
-    <dynamics damping="0.01" friction="0.001"/>
-  </joint>
-  <link name="${prefix}link_${current_num}">
-    <xacro:cylinder_inertia m="${m}" r="${rad}" h="${cable_len}" />
-    <visual>
-      <origin xyz="0 0 ${cable_len/2.0}"/>
-      <geometry><cylinder radius="${rad}" length="${cable_len}"/></geometry>
-    </visual>
-    <collision>
-      <origin xyz="0 0 ${cable_len/2.0}"/>
-      <geometry><cylinder radius="${rad}" length="${cable_len}"/></geometry>
-    </collision>
-    <self_collide>false</self_collide>
-  </link>
-  <joint name="${prefix}joint_y_${current_num}" type="continuous">
-    <parent link="${prefix}virtual_${current_num}"/>
-    <child link="${prefix}link_${current_num}"/>
-    <origin xyz="0 0 0" rpy="0 0 0"/>
-    <axis xyz="0 1 0"/>
-    <dynamics damping="0.01" friction="0.001"/>
-  </joint>
-  <xacro:if value="${current_num &lt; total_num}">
-    <xacro:flexible_chain_generator
-      prefix="${prefix}"
-      parent="${prefix}link_${current_num}"
-      current_num="${current_num + 1}"
-      total_num="${total_num}"
-      cable_len="${cable_len}" rad="${rad}" m="${m}" />
-  </xacro:if>
-</xacro:macro>
-<!-- ____________   Cable macro  _______________________-->
-  <xacro:macro name="uav_cable" params="prefix parent_link is_flexible segments length radius mass">
+    <link name="${prefix}link_${current_num}">
+      <xacro:cylinder_inertia m="${m}" r="${rad}" h="${cable_len}" />
+      <visual>
+        <origin xyz="0 0 ${cable_len/2.0}"/>
+        <geometry><cylinder radius="${rad}" length="${cable_len}"/></geometry>
+      </visual>
+      <collision>
+        <origin xyz="0 0 ${cable_len/2.0}"/>
+        <geometry><cylinder radius="${rad}" length="${cable_len}"/></geometry>
+      </collision>
+    </link>
+    <joint name="${prefix}joint_y_${current_num}" type="continuous">
+      <parent link="${prefix}virtual_${current_num}"/>
+      <child link="${prefix}link_${current_num}"/>
+      <origin xyz="0 0 0" rpy="0 0 0"/>
+      <axis xyz="0 1 0"/>
+      <dynamics damping="0.01" friction="0.001"/>
+    </joint>
+    <xacro:if value="${current_num &lt; total_num}">
+      <xacro:flexible_chain_generator
+        prefix="${prefix}"
+        parent="${prefix}link_${current_num}"
+        current_num="${current_num + 1}"
+        total_num="${total_num}"
+        cable_len="${cable_len}" rad="${rad}" m="${m}"
+        theta="${theta}" />
+    </xacro:if>
+  </xacro:macro>
+  <xacro:macro name="uav_cable" params="prefix parent_link is_flexible segments length radius mass orientation">
     <xacro:if value="${is_flexible}">
       <xacro:flexible_chain_generator
         prefix="${prefix}" parent="${parent_link}" current_num="1"
-        total_num="${segments}" cable_len="${length/segments}" rad="${radius}" m="${mass/segments}" />
+        total_num="${segments}" cable_len="${length/segments}" rad="${radius}" m="${mass/segments}" theta="${orientation}" />
     </xacro:if>
     <xacro:unless value="${is_flexible}">
-      <xacro:rigid_cable prefix="${prefix}" parent_link="${parent_link}"
-        length="${length}" radius="${radius}" mass="${mass}" />
-    </xacro:unless>
+      </xacro:unless>
   </xacro:macro>
 </robot>

Commit message: Change of cable visibility [NOT WORKING]

File: urdf/components/cable_component.xacro (robot description, xacro)
@@ -35,4 +35,7 @@
         <inertia ixx="1e-8" ixy="0" ixz="0" iyy="1e-8" iyz="0" izz="1e-8"/>
       </inertial>
+      <visual name="visual">
+        <geometry><sphere radius="0.001"/></geometry>
+      </visual>
     </link>
     <xacro:if value="${current_num == 1}">
@@ -54,13 +57,23 @@
     <link name="${prefix}link_${current_num}">
       <xacro:cylinder_inertia m="${m}" r="${rad}" h="${cable_len}" />
-      <visual>
+      <visual name="visual">
         <origin xyz="0 0 ${cable_len/2.0}"/>
         <geometry><cylinder radius="${rad}" length="${cable_len}"/></geometry>
+        <material name="gray"><color rgba="0.5 0.5 0.5 1.0"/></material>
       </visual>
-      <collision>
+      <collision name="collision">
         <origin xyz="0 0 ${cable_len/2.0}"/>
         <geometry><cylinder radius="${rad}" length="${cable_len}"/></geometry>
       </collision>
     </link>
+    <gazebo reference="${prefix}link_${current_num}">
+      <visual>
+        <material>
+          <ambient>0.5 0.5 0.5 1.0</ambient>
+          <diffuse>0.5 0.5 0.5 1.0</diffuse>
+        </material>
+          <transparency>0</transparency>
+      </visual>
+    </gazebo>
     <joint name="${prefix}joint_y_${current_num}" type="continuous">
       <parent link="${prefix}virtual_${current_num}"/>

Commit message: inclined cable at spawn

File: urdf/components/cable_component.xacro (robot description, xacro)
@@ -10,5 +10,5 @@
   </xacro:macro>
 <!-- ____________   Flexible cable  _______________________-->
-  <xacro:macro name="flexible_chain_generator" params="prefix parent current_num total_num cable_len rad m">
+  <xacro:macro name="flexible_chain_generator" params="prefix parent cable_roll:=0 cable_pitch:=0 cable_yaw:=0 current_num total_num cable_len rad m">
   <link name="${prefix}virtual_${current_num}">
     <inertial>
@@ -18,10 +18,13 @@
   </link>
   <joint name="${prefix}joint_x_${current_num}" type="continuous">
-    <parent link="${parent}"/>
-    <child link="${prefix}virtual_${current_num}"/>
-    <origin xyz="0 0 ${current_num == 1 and 0 or cable_len}" rpy="0 0 0"/>
-    <axis xyz="1 0 0"/>
-    <dynamics damping="0.05" friction="0.01"/>
-  </joint>
+  <parent link="${parent}"/>
+  <child link="${prefix}virtual_${current_num}"/>
+  <origin xyz="0 0 ${current_num == 1 and 0 or cable_len}"
+          rpy="${current_num == 1 and cable_roll or 0}
+               ${current_num == 1 and cable_pitch or 0}
+               ${current_num == 1 and cable_yaw or 0}"/>
+  <axis xyz="1 0 0"/>
+  <dynamics damping="0.05" friction="0.01"/>
+</joint>
   <link name="${prefix}link_${current_num}">
     <xacro:cylinder_inertia m="${m}" r="${rad}" h="${cable_len}" />
@@ -44,24 +47,29 @@
   </gazebo>
   <xacro:if value="${current_num &lt; total_num}">
-    <xacro:flexible_chain_generator
-      prefix="${prefix}"
-      parent="${prefix}link_${current_num}"
-      current_num="${current_num + 1}"
-      total_num="${total_num}"
-      cable_len="${cable_len}" rad="${rad}" m="${m}" />
+  <xacro:flexible_chain_generator
+    prefix="${prefix}"
+    parent="${prefix}link_${current_num}"
+    cable_roll="0" cable_pitch="0" cable_yaw="0"
+    current_num="${current_num + 1}"
+    total_num="${total_num}"
+    cable_len="${cable_len}" rad="${rad}" m="${m}" />
   </xacro:if>
 </xacro:macro>
 <!-- ____________   Cable macro  _______________________-->
-  <xacro:macro name="uav_cable" params="prefix parent_link is_flexible segments length radius mass">
-    <xacro:if value="${is_flexible}">
-      <xacro:flexible_chain_generator
-        prefix="${prefix}" parent="${parent_link}" current_num="1"
-        total_num="${segments}" cable_len="${length/segments}" rad="${radius}" m="${mass/segments}" />
-    </xacro:if>
-    <xacro:unless value="${is_flexible}">
-      <xacro:flexible_chain_generator
-      prefix="${prefix}" parent="${parent_link}" current_num="1"
-      total_num="1" cable_len="${length}" rad="${radius}" m="${mass}" />
-    </xacro:unless>
-  </xacro:macro>
+<xacro:macro name="uav_cable" params="prefix parent_link is_flexible segments length radius mass cable_roll:=0 cable_pitch:=0 cable_yaw:=0">
+  <xacro:if value="${is_flexible}">
+    <xacro:flexible_chain_generator
+      prefix="${prefix}" parent="${parent_link}"
+      cable_roll="${cable_roll}" cable_pitch="${cable_pitch}" cable_yaw="${cable_yaw}"
+      current_num="1" total_num="${segments}"
+      cable_len="${length/segments}" rad="${radius}" m="${mass/segments}" />
+  </xacro:if>
+  <xacro:unless value="${is_flexible}">
+    <xacro:flexible_chain_generator
+      prefix="${prefix}" parent="${parent_link}"
+      cable_roll="${cable_roll}" cable_pitch="${cable_pitch}" cable_yaw="${cable_yaw}"
+      current_num="1" total_num="1"
+      cable_len="${length}" rad="${radius}" m="${mass}" />
+  </xacro:unless>
+</xacro:macro>
 </robot>

File: urdf/uav_cable_assembly.urdf.xacro (robot description, xacro)
@@ -3,5 +3,5 @@
   <xacro:include filename="$(find acts_simulator)/urdf/crazy2fly.urdf.xacro" />
   <xacro:include filename="$(find acts_simulator)/urdf/components/cable_component.xacro" />
-<xacro:macro name="add_drone" params="id segments length x_off y_off z_off cable_roll:=0 cable_pitch:=0 cable_yaw:=0 panel_link:=''">
+<xacro:macro name="add_drone" params="id segments length x_off:=0 y_off:=0 z_off:=0 cable_roll:=0 cable_pitch:=0 cable_yaw:=0 panel_link:=''">
     <xacro:property name="prefix" value="drone${id}_" />
     <xacro:crazy2fly prefix="${prefix}" />
@@ -27,4 +27,7 @@
         segments="${segments}"
         length="${length}"
+        cable_roll="${cable_roll}"
+        cable_pitch="${cable_pitch}"
+        cable_yaw="${cable_yaw}"
         radius="0.005" mass="0.01" />
     <!-- Drone is child of cable tip link_${segments} -->

Commit message: Simulation spawn but wrong high

File: urdf/components/cable_component.xacro (robot description, xacro)
@@ -9,6 +9,6 @@
     </inertial>
   </xacro:macro>
-<!-- ____________   Flexible cable  _______________________-->
-  <xacro:macro name="flexible_chain_generator" params="prefix parent cable_roll:=0 cable_pitch:=0 cable_yaw:=0 current_num total_num cable_len rad m">
+<xacro:macro name="flexible_chain_generator" params="prefix parent cable_roll:=0 cable_pitch:=0 cable_yaw:=0 current_num total_num cable_len rad m type:='uav'">
+  <xacro:property name="dir" value="${-1 if type == 'ugv' else 1}" />
   <link name="${prefix}virtual_${current_num}">
     <inertial>
@@ -18,20 +18,20 @@
   </link>
   <joint name="${prefix}joint_x_${current_num}" type="continuous">
-  <parent link="${parent}"/>
-  <child link="${prefix}virtual_${current_num}"/>
-  <origin xyz="0 0 ${current_num == 1 and 0 or cable_len}"
-          rpy="${current_num == 1 and cable_roll or 0}
-               ${current_num == 1 and cable_pitch or 0}
-               ${current_num == 1 and cable_yaw or 0}"/>
-  <axis xyz="1 0 0"/>
-  <dynamics damping="0.05" friction="0.01"/>
-</joint>
+    <parent link="${parent}"/>
+    <child link="${prefix}virtual_${current_num}"/>
+    <origin xyz="0 0 ${current_num == 1 and 0 or (cable_len * dir)}"
+            rpy="${current_num == 1 and cable_roll or 0}
+                 ${current_num == 1 and cable_pitch or 0}
+                 ${current_num == 1 and cable_yaw or 0}"/>
+    <axis xyz="1 0 0"/>
+    <dynamics damping="0.05" friction="0.01"/>
+  </joint>
   <link name="${prefix}link_${current_num}">
     <xacro:cylinder_inertia m="${m}" r="${rad}" h="${cable_len}" />
     <visual>
-      <origin xyz="0 0 ${-cable_len/2.0}"/>
+      <origin xyz="0 0 ${-cable_len / 2.0 * dir}"/>
       <geometry><cylinder radius="${rad}" length="${cable_len}"/></geometry>
     </visual>
-    </link>
+  </link>
   <joint name="${prefix}joint_y_${current_num}" type="continuous">
     <parent link="${prefix}virtual_${current_num}"/>
@@ -47,18 +47,19 @@
   </gazebo>
   <xacro:if value="${current_num &lt; total_num}">
-  <xacro:flexible_chain_generator
-    prefix="${prefix}"
-    parent="${prefix}link_${current_num}"
-    cable_roll="0" cable_pitch="0" cable_yaw="0"
-    current_num="${current_num + 1}"
-    total_num="${total_num}"
-    cable_len="${cable_len}" rad="${rad}" m="${m}" />
-  </xacro:if>
+    <xacro:flexible_chain_generator
+      prefix="${prefix}"
+      parent="${prefix}link_${current_num}"
+      cable_roll="0" cable_pitch="0" cable_yaw="0"
+      current_num="${current_num + 1}"
+      total_num="${total_num}"
+      cable_len="${cable_len}" rad="${rad}" m="${m}"
+      type="${type}" />
+      </xacro:if>
 </xacro:macro>
-<!-- ____________   Cable macro  _______________________-->
 <xacro:macro name="uav_cable" params="prefix parent_link is_flexible segments length radius mass cable_roll:=0 cable_pitch:=0 cable_yaw:=0">
   <xacro:if value="${is_flexible}">
     <xacro:flexible_chain_generator
       prefix="${prefix}" parent="${parent_link}"
+      type="uav"
       cable_roll="${cable_roll}" cable_pitch="${cable_pitch}" cable_yaw="${cable_yaw}"
       current_num="1" total_num="${segments}"
@@ -68,4 +69,23 @@
     <xacro:flexible_chain_generator
       prefix="${prefix}" parent="${parent_link}"
+      type="uav"
+      cable_roll="${cable_roll}" cable_pitch="${cable_pitch}" cable_yaw="${cable_yaw}"
+      current_num="1" total_num="1"
+      cable_len="${length}" rad="${radius}" m="${mass}" />
+  </xacro:unless>
+</xacro:macro>
+<xacro:macro name="ugv_cable" params="prefix parent_link is_flexible segments length radius mass cable_roll:=0 cable_pitch:=0 cable_yaw:=0">
+  <xacro:if value="${is_flexible}">
+    <xacro:flexible_chain_generator
+      prefix="${prefix}" parent="${parent_link}"
+      type="ugv"
+      cable_roll="${cable_roll}" cable_pitch="${cable_pitch}" cable_yaw="${cable_yaw}"
+      current_num="1" total_num="${segments}"
+      cable_len="${length/segments}" rad="${radius}" m="${mass/segments}" />
+  </xacro:if>
+  <xacro:unless value="${is_flexible}">
+    <xacro:flexible_chain_generator
+      prefix="${prefix}" parent="${parent_link}"
+      type="ugv"
       cable_roll="${cable_roll}" cable_pitch="${cable_pitch}" cable_yaw="${cable_yaw}"
       current_num="1" total_num="1"

File: urdf/components/ugv_component.xacro (robot description, xacro)
@@ -4,18 +4,19 @@
     <link name="${prefix}base_link">
       <inertial>
-        <mass value="2.0"/>
-        <inertia ixx="0.05" ixy="0.0" ixz="0.0" iyy="0.05" iyz="0.0" izz="0.08"/>
+        <mass value="10.0" />
+        <origin xyz="0 0 0" rpy="0 0 0" />
+        <inertia ixx="0.01" ixy="0" ixz="0" iyy="0.01" iyz="0" izz="0.02" />
       </inertial>
       <visual>
-        <origin xyz="${x} ${y} ${z}" rpy="0 0 0"/>
-        <geometry><box size="0.2 0.2 0.2"/></geometry>
-        <material name="blue"><color rgba="0 0 1 1"/></material>
+        <geometry>
+        <box size="0.2 0.2 0.1"/>
+        </geometry>
       </visual>
-      <!-- <collision>
-        <geometry>
-          <box size="0.5 0.5 0.2"/>
-        </geometry>
-      </collision> -->
-    </link>
+		<!-- <collision name="${prefix}base_collision">
+			<geometry>
+			<box size="0.3 0.3 0.15"/>
+			</geometry>
+		</collision> -->
+	</link>
   </xacro:macro>
 </robot>

File: urdf/special_cases/track.xacro (robot description, xacro)
@@ -1,12 +1,16 @@
 <?xml version="1.0"?>
 <robot xmlns:xacro="http://www.ros.org/wiki/xacro" name="reference_marker">
-  <xacro:include filename="components/ugv_component.xacro" />
   <link name="ref_root"/>
-  <xacro:ugv_component
-    prefix="obstacle_"
-    x="2.0"
-    y="2.0"
-    z="2.0"
-  />
+  <link name="obstacle_base_link">
+    <inertial>
+      <mass value="2.0"/>
+      <inertia ixx="0.05" ixy="0.0" ixz="0.0" iyy="0.05" iyz="0.0" izz="0.08"/>
+    </inertial>
+    <visual>
+      <origin xyz="-0.5 0.0 0.1" rpy="0 0 0"/>
+      <geometry><box size="0.1 0.1 0.1"/></geometry>
+      <material name="blue"><color rgba="0 0 1 1"/></material>
+    </visual>
+  </link>
   <joint name="ref_joint" type="fixed">
     <parent link="ref_root"/>

File: urdf/ugv_cable_assembly.urdf.xacro (robot description, xacro)
@@ -1,16 +1,20 @@
 <?xml version="1.0"?>
 <robot xmlns:xacro="http://www.ros.org/wiki/xacro">
-  <xacro:include filename="$(find acts_simulator)/urdf/crazy2fly.urdf.xacro" />
   <xacro:include filename="$(find acts_simulator)/urdf/components/cable_component.xacro" />
-<xacro:macro name="add_drone" params="id segments length x_off:=0 y_off:=0 z_off:=0 cable_roll:=0 cable_pitch:=0 cable_yaw:=0 panel_link:=''">
-    <xacro:property name="prefix" value="drone${id}_" />
-    <xacro:crazy2fly prefix="${prefix}" />
-        <link name="${prefix}cable_root_link">
-            <inertial>
-                <mass value="0.0001"/>
-                <inertia ixx="1e-6" ixy="0" ixz="0" iyy="1e-6" iyz="0" izz="1e-6"/>
-            </inertial>
-        </link>
-        <!-- If panel provided, attach panel to cable root -->
+  <xacro:include filename="$(find acts_simulator)/urdf/components/ugv_component.xacro" />
+  <xacro:macro name="add_ugv" params="id segments length x_off:=0 y_off:=0 z_off:=0 cable_roll:=0 cable_pitch:=0 cable_yaw:=0 panel_link:=''">
+    <xacro:property name="prefix" value="ugv${id}_" />
+    <xacro:ugv_component
+    prefix="${prefix}"
+    x="0"
+    y="0"
+    z="0"
+    />
+    <link name="${prefix}cable_root_link">
+        <inertial>
+            <mass value="0.0001"/>
+            <inertia ixx="1e-6" ixy="0" ixz="0" iyy="1e-6" iyz="0" izz="1e-6"/>
+        </inertial>
+    </link>
     <xacro:unless value="${panel_link == ''}">
         <joint name="${prefix}panel_to_cable_joint" type="fixed">
@@ -20,6 +24,5 @@
         </joint>
     </xacro:unless>
-    <!-- Cable hangs from cable_root_link -->
-    <xacro:uav_cable
+    <xacro:ugv_cable
         prefix="${prefix}"
         parent_link="${prefix}cable_root_link"
@@ -31,7 +34,5 @@
         cable_yaw="${cable_yaw}"
         radius="0.005" mass="0.01" />
-    <!-- virtual -->
-    <!-- Link between joint_x and joint_y -->
-    <link name="${prefix}virtual_cable_to_drone_joint">
+       <link name="${prefix}virtual_cable_to_ugv_joint">
         <inertial>
             <mass value="0.0001"/>
@@ -45,5 +46,5 @@
     </inertial>
     </link>
-    <!-- Fix the attachment link to the drone's base_link -->
+    <!-- Fix the attachment link to the ugv's base_link -->
     <joint name="${prefix}cable_attach_fixed" type="fixed">
     <parent link="${prefix}cable_attach_link"/>
@@ -52,7 +53,7 @@
     </joint>
     <!-- joint_x: last cable segment to virtual -->
-    <joint name="${prefix}joint_x_cable_to_drone_joint" type="revolute">
+    <joint name="${prefix}joint_x_cable_to_ugv_joint" type="revolute">
     <parent link="${prefix}link_${segments}"/>
-    <child link="${prefix}virtual_cable_to_drone_joint"/>
+    <child link="${prefix}virtual_cable_to_ugv_joint"/>
     <axis xyz="1 0 0"/>
     <limit lower="-1.5708" upper="1.5708" effort="10" velocity="1.0"/>
@@ -60,6 +61,6 @@
     </joint>
     <!-- joint_y: virtual to cable_attach_link  -->
-    <joint name="${prefix}joint_y_cable_to_drone_joint" type="revolute">
-    <parent link="${prefix}virtual_cable_to_drone_joint"/>
+    <joint name="${prefix}joint_y_cable_to_ugv_joint" type="revolute">
+    <parent link="${prefix}virtual_cable_to_ugv_joint"/>
     <child link="${prefix}cable_attach_link"/>
     <axis xyz="0 1 0"/>
@@ -73,4 +74,4 @@
         <preserveFixedJoint>true</preserveFixedJoint>
     </gazebo>
-    </xacro:macro>
+  </xacro:macro>
 </robot>
