Commit message: Trying to apply cable movement to the whole system

File: urdf/components/cable_component.xacro (robot description, xacro)
@@ -9,83 +9,81 @@
     </inertial>
   </xacro:macro>
-<!-- ____________   Rigid cable  _______________________-->
-  <xacro:macro name="rigid_cable" params="prefix parent_link length radius mass">
-    <link name="${prefix}rigid_link">
-      <xacro:cylinder_inertia m="${mass}" r="${radius}" h="${length}" />
-      <visual>
-        <origin xyz="0 0 ${-length/2.0}"/>
-        <geometry><cylinder radius="${radius}" length="${length}"/></geometry>
-      </visual>
-      <collision>
-        <origin xyz="0 0 ${-length/2.0}"/>
-        <geometry><cylinder radius="${radius}" length="${length}"/></geometry>
-      </collision>
-    </link>
-    <joint name="${prefix}rigid_joint" type="universal">
-      <parent link="${parent_link}"/>
-      <child link="${prefix}rigid_link"/>
-      <origin xyz="0 0 -0.05" rpy="0 0 0"/>
-    </joint>
-  </xacro:macro>
-<!-- ____________   Flexible cable  _______________________-->
-  <xacro:macro name="flexible_chain_generator" params="prefix parent current_num total_num cable_len rad m theta">
-    <link name="${prefix}virtual_${current_num}">
-      <inertial>
-        <mass value="0.0001"/>
-        <inertia ixx="1e-8" ixy="0" ixz="0" iyy="1e-8" iyz="0" izz="1e-8"/>
-      </inertial>
-    </link>
-    <xacro:if value="${current_num == 1}">
-      <joint name="${prefix}joint_fixed_root" type="fixed">
-        <parent link="${parent}"/>
-        <child link="${prefix}virtual_${current_num}"/>
-        <origin xyz="0 0 0" rpy="0 ${theta} 0"/>
-      </joint>
-    </xacro:if>
-    <xacro:unless value="${current_num == 1}">
-      <joint name="${prefix}joint_x_${current_num}" type="continuous">
-        <parent link="${parent}"/>
-        <child link="${prefix}virtual_${current_num}"/>
-        <origin xyz="0 0 ${cable_len}" rpy="0 0 0"/>
-        <axis xyz="1 0 0"/>
-        <dynamics damping="0.01" friction="0.001"/>
-      </joint>
-    </xacro:unless>
-    <link name="${prefix}link_${current_num}">
-      <xacro:cylinder_inertia m="${m}" r="${rad}" h="${cable_len}" />
-      <visual>
-        <origin xyz="0 0 ${cable_len/2.0}"/>
-        <geometry><cylinder radius="${rad}" length="${cable_len}"/></geometry>
-      </visual>
-      <collision>
-        <origin xyz="0 0 ${cable_len/2.0}"/>
-        <geometry><cylinder radius="${rad}" length="${cable_len}"/></geometry>
-      </collision>
-    </link>
-    <joint name="${prefix}joint_y_${current_num}" type="continuous">
-      <parent link="${prefix}virtual_${current_num}"/>
-      <child link="${prefix}link_${current_num}"/>
-      <origin xyz="0 0 0" rpy="0 0 0"/>
-      <axis xyz="0 1 0"/>
-      <dynamics damping="0.01" friction="0.001"/>
-    </joint>
-    <xacro:if value="${current_num &lt; total_num}">
-      <xacro:flexible_chain_generator
-        prefix="${prefix}"
-        parent="${prefix}link_${current_num}"
-        current_num="${current_num + 1}"
-        total_num="${total_num}"
-        cable_len="${cable_len}" rad="${rad}" m="${m}"
-        theta="${theta}" />
-    </xacro:if>
-  </xacro:macro>
-  <xacro:macro name="uav_cable" params="prefix parent_link is_flexible segments length radius mass orientation">
-    <xacro:if value="${is_flexible}">
-      <xacro:flexible_chain_generator
-        prefix="${prefix}" parent="${parent_link}" current_num="1"
-        total_num="${segments}" cable_len="${length/segments}" rad="${radius}" m="${mass/segments}" theta="${orientation}" />
-    </xacro:if>
-    <xacro:unless value="${is_flexible}">
-      </xacro:unless>
-  </xacro:macro>
+<xacro:macro name="flexible_chain_generator" params="prefix parent cable_roll:=0 cable_pitch:=0 cable_yaw:=0 current_num total_num cable_len rad m type:='uav'">
+  <xacro:property name="dir" value="${-1 if type == 'ugv' else 1}" />
+  <link name="${prefix}virtual_${current_num}">
+    <inertial>
+      <mass value="0.0001"/>
+      <inertia ixx="1e-6" ixy="0" ixz="0" iyy="1e-6" iyz="0" izz="1e-6"/>
+    </inertial>
+  </link>
+  <joint name="${prefix}joint_x_${current_num}" type="continuous">
+    <parent link="${parent}"/>
+    <child link="${prefix}virtual_${current_num}"/>
+    <origin xyz="0 0 ${current_num == 1 and 0 or (cable_len * dir)}"
+            rpy="${current_num == 1 and cable_roll or 0}
+                 ${current_num == 1 and cable_pitch or 0}
+                 ${current_num == 1 and cable_yaw or 0}"/>
+    <axis xyz="1 0 0"/>
+    <dynamics damping="0.01" friction="0.001"/>
+  </joint>
+  <link name="${prefix}link_${current_num}">
+    <xacro:cylinder_inertia m="${m}" r="${rad}" h="${cable_len}" />
+    <visual>
+      <origin xyz="0 0 ${-cable_len / 2.0 * dir}"/>
+      <geometry><cylinder radius="${rad}" length="${cable_len}"/></geometry>
+    </visual>
+  </link>
+  <joint name="${prefix}joint_y_${current_num}" type="continuous">
+    <parent link="${prefix}virtual_${current_num}"/>
+    <child link="${prefix}link_${current_num}"/>
+    <axis xyz="0 1 0"/>
+    <dynamics damping="0.01" friction="0.001"/>
+  </joint>
+  <xacro:if value="${current_num &lt; total_num}">
+    <xacro:flexible_chain_generator
+      prefix="${prefix}"
+      parent="${prefix}link_${current_num}"
+      cable_roll="0" cable_pitch="0" cable_yaw="0"
+      current_num="${current_num + 1}"
+      total_num="${total_num}"
+      cable_len="${cable_len}" rad="${rad}" m="${m}"
+      type="${type}" />
+      </xacro:if>
+</xacro:macro>
+<xacro:macro name="uav_cable" params="prefix parent_link is_flexible segments length radius mass cable_roll:=0 cable_pitch:=0 cable_yaw:=0">
+  <xacro:if value="${is_flexible}">
+    <xacro:flexible_chain_generator
+      prefix="${prefix}" parent="${parent_link}"
+      type="uav"
+      cable_roll="${cable_roll}" cable_pitch="${cable_pitch}" cable_yaw="${cable_yaw}"
+      current_num="1" total_num="${segments}"
+      cable_len="${length/segments}" rad="${radius}" m="${mass/segments}" />
+  </xacro:if>
+  <xacro:unless value="${is_flexible}">
+    <xacro:flexible_chain_generator
+      prefix="${prefix}" parent="${parent_link}"
+      type="uav"
+      cable_roll="${cable_roll}" cable_pitch="${cable_pitch}" cable_yaw="${cable_yaw}"
+      current_num="1" total_num="1"
+      cable_len="${length}" rad="${radius}" m="${mass}" />
+  </xacro:unless>
+</xacro:macro>
+<xacro:macro name="ugv_cable" params="prefix parent_link is_flexible segments length radius mass cable_roll:=0 cable_pitch:=0 cable_yaw:=0">
+  <xacro:if value="${is_flexible}">
+    <xacro:flexible_chain_generator
+      prefix="${prefix}" parent="${parent_link}"
+      type="ugv"
+      cable_roll="${cable_roll}" cable_pitch="${cable_pitch}" cable_yaw="${cable_yaw}"
+      current_num="1" total_num="${segments}"
+      cable_len="${length/segments}" rad="${radius}" m="${mass/segments}" />
+  </xacro:if>
+  <xacro:unless value="${is_flexible}">
+    <xacro:flexible_chain_generator
+      prefix="${prefix}" parent="${parent_link}"
+      type="ugv"
+      cable_roll="${cable_roll}" cable_pitch="${cable_pitch}" cable_yaw="${cable_yaw}"
+      current_num="1" total_num="1"
+      cable_len="${length}" rad="${radius}" m="${mass}" />
+  </xacro:unless>
+</xacro:macro>
 </robot>

File: urdf/components/ugv_component.xacro (robot description, xacro)
@@ -1,23 +1,25 @@
 <?xml version="1.0"?>
 <robot xmlns:xacro="http://www.ros.org/wiki/xacro">
-  <xacro:macro name="ugv_platform" params="prefix">
+  <xacro:macro name="ugv_component" params="prefix x y z">
     <link name="${prefix}base_link">
       <inertial>
-        <mass value="2.0"/>
-        <inertia ixx="0.05" ixy="0.0" ixz="0.0" iyy="0.05" iyz="0.0" izz="0.08"/>
+        <mass value="0.001" />
+        <origin xyz="0 0 0" rpy="0 0 0" />
+        <inertia ixx="0.01" ixy="0" ixz="0" iyy="0.01" iyz="0" izz="0.02" />
       </inertial>
       <visual>
         <geometry>
-          <box size="0.5 0.5 0.2"/> </geometry>
-        <material name="blue">
-            <color rgba="0 0 1 1"/>
+            <sphere radius="0.02"/>
+        </geometry>
+        <material name="Red">
+            <color rgba="1.0 0.0 0.0 1.0"/>
         </material>
       </visual>
-      <collision>
-        <geometry>
-          <box size="0.5 0.5 0.2"/>
-        </geometry>
-      </collision>
-    </link>
+		<!-- <collision name="${prefix}base_collision">
+			<geometry>
+			<box size="0.3 0.3 0.15"/>
+			</geometry>
+		</collision> -->
+	</link>
   </xacro:macro>
 </robot>

File: urdf/uav_cable_assembly.urdf.xacro (robot description, xacro)
@@ -1,28 +1,76 @@
 <?xml version="1.0"?>
 <robot xmlns:xacro="http://www.ros.org/wiki/xacro">
-  <xacro:include filename="$(find acts_simulator)/urdf/crazy2fly.urdf.xacro" />
-  <xacro:include filename="$(find acts_simulator)/urdf/components/cable_component.xacro" />
-  <xacro:macro name="add_drone" params="id segments length panel_link x_off y_off z_off">
+  <xacro:include filename="crazy2fly.urdf.xacro" />
+  <xacro:include filename="components/cable_component.xacro" />
+<xacro:macro name="add_drone" params="id segments length x_off:=0 y_off:=0 z_off:=0 cable_roll:=0 cable_pitch:=0 cable_yaw:=0 panel_link:=''">
     <xacro:property name="prefix" value="drone${id}_" />
     <xacro:crazy2fly prefix="${prefix}" />
+        <link name="${prefix}cable_root_link">
+            <inertial>
+                <mass value="0.0001"/>
+                <inertia ixx="1e-6" ixy="0" ixz="0" iyy="1e-6" iyz="0" izz="1e-6"/>
+            </inertial>
+        </link>
+        <!-- If panel provided, attach panel to cable root -->
+    <xacro:unless value="${panel_link == ''}">
+        <joint name="${prefix}panel_to_cable_joint" type="fixed">
+            <parent link="${panel_link}"/>
+            <child link="${prefix}cable_root_link"/>
+            <origin xyz="${x_off} ${y_off} ${z_off}" rpy="0 0 0"/>
+        </joint>
+    </xacro:unless>
+    <!-- Cable hangs from cable_root_link -->
     <xacro:uav_cable
-      prefix="${prefix}"
-      parent_link="${panel_link}"
-      is_flexible="true"
-      segments="${segments}"
-      length="${length}"
-      radius="0.005" mass="0.01" />
-    <joint name="${prefix}cable_to_drone_joint" type="fixed">
-      <parent link="${prefix}link_${segments}"/>
-      <child link="${prefix}base_link"/>
-      <origin xyz="${x_off} ${y_off} ${float(z_off)}" rpy="0 0 0"/>
+        prefix="${prefix}"
+        parent_link="${prefix}cable_root_link"
+        is_flexible="true"
+        segments="${segments}"
+        length="${length}"
+        cable_roll="${cable_roll}"
+        cable_pitch="${cable_pitch}"
+        cable_yaw="${cable_yaw}"
+        radius="0.005" mass="0.01" />
+    <!-- virtual -->
+    <!-- Link between joint_x and joint_y -->
+    <link name="${prefix}virtual_cable_to_drone_joint">
+        <inertial>
+            <mass value="0.0001"/>
+            <inertia ixx="1e-6" ixy="0" ixz="0" iyy="1e-6" iyz="0" izz="1e-6"/>
+        </inertial>
+    </link>
+    <link name="${prefix}cable_attach_link">
+    <inertial>
+        <mass value="0.0001"/>
+        <inertia ixx="1e-6" ixy="0" ixz="0" iyy="1e-6" iyz="0" izz="1e-6"/>
+    </inertial>
+    </link>
+    <!-- Fix the attachment link to the drone's base_link -->
+    <joint name="${prefix}cable_attach_fixed" type="fixed">
+    <parent link="${prefix}cable_attach_link"/>
+    <child link="${prefix}base_link"/>
+    <origin xyz="0 0 0" rpy="0 0 0"/>
     </joint>
-    <gazebo reference="${prefix}cable_to_drone_joint">
-      <preserveFixedJoint>true</preserveFixedJoint>
-      <disableFixedJointLumping>true</disableFixedJointLumping>
+    <!-- joint_x: last cable segment to virtual -->
+    <joint name="${prefix}joint_x_cable_to_drone_joint" type="revolute">
+    <parent link="${prefix}link_${segments}"/>
+    <child link="${prefix}virtual_cable_to_drone_joint"/>
+    <axis xyz="1 0 0"/>
+    <limit lower="-1.5708" upper="1.5708" effort="10" velocity="1.0"/>
+    <dynamics damping="0.05" friction="0.01"/>
+    </joint>
+    <!-- joint_y: virtual to cable_attach_link  -->
+    <joint name="${prefix}joint_y_cable_to_drone_joint" type="revolute">
+    <parent link="${prefix}virtual_cable_to_drone_joint"/>
+    <child link="${prefix}cable_attach_link"/>
+    <axis xyz="0 1 0"/>
+    <limit lower="-1.5708" upper="1.5708" effort="10" velocity="1.0"/>
+    <dynamics damping="0.05" friction="0.01"/>
+    </joint>
+    <gazebo reference="${prefix}base_link">
+        <preserveFixedJoint>true</preserveFixedJoint>
     </gazebo>
-    <gazebo reference="${prefix}base_link">
-      <self_collide>true</self_collide>
+    <gazebo reference="${prefix}cable_attach_link">
+        <preserveFixedJoint>true</preserveFixedJoint>
     </gazebo>
-  </xacro:macro>
+    </xacro:macro>
 </robot>
